File: designs/ADC_Board_rev3/adc_cap.brd (EAGLE design)
At the start: 81.9 x 76.5 mm, 81 parts, among them J1 22-05-7028-02, J2 22-05-7028-02, J3 22-05-7028-02, J4 22-05-7028-02, J5 22-05-7058-05, Q1 BSS84, Q2 BSS84, Q3 BSS84, Q4 BSS84

Commit message: updeate to values on the ADC cape rev 3
Parts:
- C1, C10, C12, C14, C15, C19, C2, C4, C5, C7: value (none) -> 10uF
- C11, R11, R21, R22, R23, R26, R6, R9: value (none) -> 0K
- C13, C16, C3: value (none) -> 0.1uF
- C17, C18, C8, C9, R1, R2, R3, R4: value (none) -> NC
- C6: value (none) -> 0.1F
- R10: value (none) -> 0k
- R12, R13: value (none) -> 5K
- R14, R15, R16, R17, R18, R19, R20, R24, R25, R27, R28, R29, R30, R31, R8: value (none) -> 10k
- R5, R7: value (none) -> 10K
