File: designs/range_cape/range_cape.brd (EAGLE design)
At the start: 37 parts, among them J1 22-05-7048-04, J10 22-05-7048-04, J11 22-05-7048-04, J12 22-05-7048-04, J2 22-05-7048-04, J3 22-05-7048-04, J4 22-05-7048-04, J5 22-05-7048-04, J6 22-05-7048-04, J7 22-05-7048-04, J8 22-05-7048-04, J9 22-05-7048-04, U5 LMS8117AMP-3.3, U6 MSP430FR5739IDA

Commit message: done with range cape
Parts:
- moved R2 10.4 mm to (41.7, 8.13)
- moved R1 10.4 mm to (46.0, 8.13)
- moved C15 6.15 mm to (46.0, 22.4), turned to 0 degrees
- moved C12 5.43 mm to (43.8, 18.3), turned to 90 degrees
- moved C14 4.84 mm to (46.0, 20.2), turned to 0 degrees
- moved JP1 1.02 mm to (24.6, 21.6)
- renumbered J1 to X4, J10 to X12, J11 to X9, J12 to X8, J2 to X5, J3 to X2, J4 to X3, J5 to X1, J6 to X6, J7 to X11, J8 to X10, J9 to X7
Connections:
- removed net N$10: X11.2
- removed net N$11: X10.2
- removed net N$12: X10.3
- removed net N$18: X7.2
- removed net N$19: X7.3
- removed net N$22: X12.2
- removed net N$23: X12.3
- removed net N$26: X9.2
- removed net N$27: X9.3
- removed net N$30: X8.2
- removed net N$31: X8.3
- removed net N$34: X6.3
- removed net N$35: X6.2
- removed net N$41: X1.3
- removed net N$42: X1.2
- removed net N$43: X3.3
- removed net N$44: X3.2
- removed net N$46: X2.3
- removed net N$47: X2.2
- removed net N$50: X5.3
- removed net N$51: X5.2
- removed net N$54: X4.3
- removed net N$55: X4.2
- removed net N$7: X11.3
- new net MSP_ADC0: U6.5, X10.3
- new net MSP_ADC1: U6.6, X9.3
- new net MSP_ADC12: U6.8, X7.3
- new net MSP_ADC13: U6.9, X6.3
- new net MSP_ADC14: U6.10, X5.3
- new net MSP_ADC15: U6.11, X4.3
- new net MSP_ADC2: U6.7, X8.3
- new net MSP_ADC5: U6.14, X1.3
- new net MSP_ADC6: U6.36, X12.3
- new net MSP_ADC7: U6.37, X11.3
- new net X-1: U6.19, X1.2
- new net X-10: U6.28, X10.2
- new net X-11: U6.27, X11.2
- new net X-12: U6.26, X12.2
- new net X-2: U6.20, X2.2
- new net X-3: U6.2, X3.2
- new net X-4: U6.1, X4.2
- new net X-5: U6.23, X5.2
- new net X-6: U6.24, X6.2
- new net X-7: U6.25, X7.2
- new net X-8: U6.35, X8.2
- new net X-9: U6.29, X9.2
- net MSP_ADC3: now also X3.3
- net MSP_ADC4: now also X2.3
Routing:
- net MSP_ADC2: track 0.00 -> 71.9 mm, vias 0 -> 2
- net MSP_ADC12: track 0.00 -> 62.2 mm, vias 0 -> 1
- net MSP_ADC1: track 0.00 -> 57.4 mm, vias 0 -> 2
- net MSP_ADC14: track 0.00 -> 57.0 mm
- net X-5: track 0.00 -> 55.2 mm, vias 0 -> 2
- net X-7: track 0.00 -> 52.3 mm, vias 0 -> 5
- net MSP_ADC6: track 0.00 -> 51.8 mm, vias 0 -> 2
- net X-8: track 0.00 -> 50.9 mm, vias 0 -> 6
- net X-6: track 0.00 -> 50.2 mm, vias 0 -> 3
- net X-9: track 0.00 -> 49.0 mm, vias 0 -> 6
- net MSP_ADC7: track 0.00 -> 45.4 mm, vias 0 -> 2
- net MSP_ADC0: track 0.00 -> 44.8 mm, vias 0 -> 2
- net MSP_ADC15: track 0.00 -> 44.4 mm
- net MSP_ADC13: track 0.00 -> 44.4 mm, vias 0 -> 1
- net X-10: track 0.00 -> 38.3 mm, vias 0 -> 4
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Other:
- board outline added: 86.4 x 67.2 mm

Commit message: pushing up frist rev of some capes
Parts:
- removed C12: 40nF, SparkFun-Capacitors:0805
- removed D1: 3_3V_PWR, SparkFun-LED:FKIT-LED-1206
- removed D2: 5V_PWR, SparkFun-LED:FKIT-LED-1206
- removed D3: 1N4004, diode:DO41-10
- removed JP1: 2514-6002UB, msp_jtag:3M_2514-6002UB
- removed PL6: (no value), con-molex-2:5569-2
- removed R10: 330, rcl:R0805W
- removed U6: MSP430FR5739IDA, TI-MSP430FR5739:SOP65P810X120-38N
- removed X1, X10, X11, X12, X2, X3, X4, X5, X6, X7, X8, X9: 22-05-7048-04, con-molex:7395-04
- added AUX1, AUX2, AUX3, AUX4, AUX5, AUX6, AUX7, AUX8: (no value), SparkFun-Connectors:1X03_LOCK
- added C1, C7: .1uF, 3-3_fixed:1206
- added C13, C17, C18, C2, C3, C4, C5, C6, C8, C9: 10uF, 3-3_fixed:1206
- added C19, C20, C21, C26, C27, C28: 10uF, 5v_fixed:1206
- added C23, C24, C29, C30, C31: 3.3uF, 5v_fixed:C3216X7R1E335K
- added C25: 620pF, 5v_fixed:0402
- added C32: 100nF, 3-3_fixed:0603
- added C33: 390pF, 3-3_fixed:0805
- added J1, J10, J2, J3, J4, J5, J6, J7, J8, J9: 22-05-7048-04, con-molex:7395-04
- added J11: 22-05-7028-02, con-molex:7395-02
- added J12: EXTERNAL_DEBUG_CON, jtag_interface:EXTERNAL_DEBUG
- added L1, L2: 2.2uH, 5v_fixed:IHLP-1212BZ
- added R12, R13, R14, R15, R16, R17, R18, R19, R20, R21, R22, R23, R24, R25, R26, R27: (no value), rcl:R0402
- added R3, R4: 100k, 5v_fixed:CRCW0402100KFKED
- added U$2: IEEE, TIparts:IEEE
- added U1, U4: SN74CBT3383PW, range_cape:SOP65P640X120-24N
- added U2: TPS62143RGTR, 5v_fixed:S-PVQFN-N16
- added U3: TPS62132RGTR, 3-3_fixed:S-PVQFN-N16
- C10, C11: device SparkFun-Capacitors:EIA3216 -> rcl:C0805
- C14, C15: device SparkFun-Capacitors:0805 -> rcl:C0805
- C16: device SparkFun-Capacitors:0805 -> rcl:C0603
- C22: value 100uF -> 3.3uF; device SparkFun-Capacitors:EIA7343 -> 5v_fixed:C3216X7R1E335K
- R5: value 330 -> 200k; device rcl:R0805W -> rcl:R0603
- R6: value 220 -> 200k; device rcl:R0805W -> rcl:R0603
- R7, R8, R9: device rcl:R0805W -> rcl:R0603
- U$3: value NANO_FUSE -> MSP430FR5969; device custom_fuses:NANO_FUSE -> range_cape:QFN50P700X700X100-49N
- U5: value LMS8117AMP-3.3 -> DRV8830DGQR; device NSC-LMS8117AMP:SOT230P696X180-4N -> Texas Instruments_By_element14_Batch_1:SOP65P640X110-15N
- moved S1 123.1 mm to (131.2, 14.8)
- moved R6 94.4 mm to (117.7, 41.4), turned to 0 degrees
- moved R7 86.9 mm to (105.7, 24.2), turned to 0 degrees
- moved C16 85.8 mm to (105.2, 21.4), turned to 270 degrees
- moved C11 81.4 mm to (123.1, 41.0), flipped to the bottom
- moved R8 79.2 mm to (102.3, 24.2), turned to 0 degrees
- moved R9 68.5 mm to (92.1, 20.4), flipped to the top, turned to 180 degrees
- moved R5 65.7 mm to (74.4, 23.2), flipped to the bottom, turned to 0 degrees
- moved C15 59.0 mm to (99.8, 46.5), flipped to the bottom, turned to 90 degrees
- moved C14 57.9 mm to (97.5, 46.5), flipped to the bottom, turned to 90 degrees
- moved U$1 50.5 mm to (50.4, 3.17)
- moved U5 49.9 mm to (60.7, 57.0), turned to 270 degrees
- moved R1 48.9 mm to (94.9, 10.4)
- moved R2 48.2 mm to (89.8, 10.4)
- moved C10 46.0 mm to (77.2, 22.4), flipped to the bottom
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Connections:
- removed net MSP_ADC0: U6.5, X10.3
- removed net MSP_ADC1: U6.6, X9.3
- removed net MSP_ADC12: U6.8, X7.3
- removed net MSP_ADC13: U6.9, X6.3
- removed net MSP_ADC14: U6.10, X5.3
- removed net MSP_ADC15: U6.11, X4.3
- removed net MSP_ADC2: U6.7, X8.3
- removed net MSP_ADC3: U6.12, X3.3
- removed net MSP_ADC4: U6.13, X2.3
- removed net MSP_ADC5: U6.14, X1.3
- removed net MSP_ADC6: U6.36, X12.3
- removed net MSP_ADC7: U6.37, X11.3
- removed net N$13: D2.A, R10.1
- removed net N$6: D1.A, R5.2
- removed net VCORE: C12.2, U6.32
- removed net X-1: U6.19, X1.2
- removed net X-10: U6.28, X10.2
- removed net X-11: U6.27, X11.2
- removed net X-12: U6.26, X12.2
- removed net X-2: U6.20, X2.2
- removed net X-3: U6.2, X3.2
- removed net X-4: U6.1, X4.2
- removed net X-5: U6.23, X5.2
- removed net X-6: U6.24, X6.2
- removed net X-7: U6.25, X7.2
- removed net X-8: U6.35, X8.2
- removed net X-9: U6.29, X9.2
- new net DVCC: C14.1, C15.1, U$3.37, U$3.48
- new net ECHO1: U4.7
- new net ECHO10: U4.12
- new net ECHO2: U4.6
- new net ECHO3: U4.5
- new net ECHO4: U4.4
- new net ECHO5: U4.3
- new net ECHO6: U4.8
- new net ECHO7: U4.9
- new net ECHO8: U4.10
- new net ECHO9: U4.11
- new net N$12: C10.1, R5.1, U4.23, U4.24
- new net N$2: L2.1, U3.1
- new net N$20: C33.1, U3.9
- new net N$5: L1.1, U2.1
- new net N$7: C25.1, U2.9
- new net PWM_C1: R12.2, U1.3
- new net PWM_C2: R13.2, U1.4
- new net PWM_C3: R14.2, U1.5
- new net PWM_C4: R15.2, U1.6
- new net PWM_C5: R16.2, U1.7
- new net PWM_C6: R17.2, U1.8
- new net PWM_C7: R18.2, U1.9
- new net PWM_C8: R19.2, U1.10
- new net PWM_IN_1: AUX1.1, R20.1, U1.22
- new net PWM_IN_2: AUX2.1, R21.1, U1.21
- new net PWM_IN_3: AUX3.1, R22.1, U1.20
- new net PWM_IN_4: AUX4.1, R23.1, U1.19
- new net PWM_OUT_1: AUX5.1, R24.1, U1.18
- new net PWM_OUT_2: AUX6.1, R25.1, U1.17
- new net PWM_OUT_3: AUX7.1, R26.1, U1.16
- new net PWM_OUT_4: AUX8.1, R27.1, U1.15
- new net TRIG_J1: J1.2
- new net TRIG_J10: J10.2
- new net TRIG_J2: J2.2
- new net TRIG_J3: J3.2
- new net TRIG_J4: J4.2, J5.2
- new net TRIG_J6: J6.2, J7.2
- new net TRIG_J8: J8.2
- new net TRIG_J9: J9.2
- new net VCC: C22.1, C23.1, C24.1, C29.1, C30.1, C31.1, C32.1, J11.1, U2.10, U2.11, U2.13, U3.10, U3.11, U3.13, U5.4
- new net X1: J1.3, U4.13
- new net X10: J10.3, U4.18
- new net X2: J2.3, U4.14
- new net X3: J3.3, U4.15
- new net X4: J4.3, U4.16
- new net X5: J5.3, U4.17
- new net X6: J6.3, U4.22
- new net X7: J7.3, U4.21
- new net X8: J8.3, U4.20
- new net X9: J9.3, U4.19
- net +3V3: now also C26.1, C27.1, C28.1, L2.2, R12.1, R13.1, R14.1, R15.1, R16.1, R17.1, R18.1, R19.1, R4.1, U1.2, U3.14, U3.7, U4.2; no longer C11.A, C14.1, C15.1, R5.1, R6.2, U5.4, U6.34, U6.4
- net +5V: now also AUX1.2, AUX2.2, AUX3.2, AUX4.2, AUX5.2, AUX6.2, AUX7.2, AUX8.2, C1.1, C13.1, C17.1, C18.1, C19.1, C2.1, C20.1, C21.1, C3.1, C4.1, C5.1, C6.1, C7.1, C8.1, C9.1, J1.1, J10.1, J2.1, J3.1, J4.1, J5.1, J6.1, J7.1, J8.1, J9.1, L1.2, R20.2, R21.2, R22.2, R23.2, R24.2, R25.2, R26.2, R27.2, R3.1, R5.2, R6.2, U$1.P9.5, U$1.P9.6, U2.14, U2.7; no longer C10.A, C22.A, D3.C, R10.2, U5.3, X1.1, X10.1, X11.1, X12.1, X2.1, X3.1, X4.1, X5.1, X6.1, X7.1, X8.1, X9.1
- net GND: now also AUX1.3, AUX2.3, AUX3.3, AUX4.3, AUX5.3, AUX6.3, AUX7.3, AUX8.3, C1.2, C10.2, C11.2, C13.2, C17.2, C18.2, C19.2, C2.2, C20.2, C21.2, C22.2, C23.2, C24.2, C25.2, C26.2, C27.2, C28.2, C29.2, C3.2, C30.2, C31.2, C32.2, C33.2, C4.2, C5.2, C6.2, C7.2, C8.2, C9.2, J1.4, J10.4, J11.2, J12.10, J2.4, J3.4, J4.4, J5.4, J6.4, J7.4, J8.4, J9.4, U1.1, U2.15, U2.17, U2.5, U2.6, U2.8, U3.15, U3.17, U3.5, U3.6, U3.8, U4.1; no longer C10.C, C11.C, C12.1, C22.C, D1.C, D2.C, JP1.9, PL6.1, U5.1, U6.3, U6.33, U6.38, X1.4, X10.4, X11.4, X12.4, X2.4, X3.4, X4.4, X5.4, X6.4, X7.4, X8.4, X9.4
- net N$14: now also R3.2, U2.4; no longer D3.A, U$3.2
- net N$15: now also R4.2, U3.4; no longer PL6.2, U$3.1
- net N$4: now also C11.1, U1.23, U1.24; no longer JP1.4
- net N$8: now also J12.12; no longer JP1.11
- net N$9: now also J12.1; no longer JP1.2
- net RESET: no longer U6.22
- net SCL: no longer U6.31
- net SDA: no longer U6.30
- net TCK: now also J12.8; no longer JP1.7, U6.18
- net TDI: now also J12.4; no longer JP1.3, U6.16
- net TDO: now also J12.2; no longer JP1.1, U6.15
- net TEST: now also J12.7; no longer JP1.8, U6.21
- net TMS: now also J12.6; no longer JP1.5, U6.17
Routing:
- net GND: track 0.00 -> 145.6 mm, vias 10 -> 21
- net X6: track 0.00 -> 77.9 mm
- net MSP_ADC2: track 71.9 -> 0.00 mm, vias 2 -> 0
- net X5: track 0.00 -> 69.2 mm
- net X7: track 0.00 -> 67.1 mm
- net MSP_ADC12: track 62.2 -> 0.00 mm, vias 1 -> 0
- net +5V: track 326.7 -> 386.8 mm, vias 0 -> 7
- net MSP_ADC1: track 57.4 -> 0.00 mm, vias 2 -> 0
- net MSP_ADC14: track 57.0 -> 0.00 mm
- net X8: track 0.00 -> 56.6 mm
- net TRIG_J4: track 0.00 -> 56.4 mm, vias 0 -> 4
- net X4: track 0.00 -> 55.8 mm
- net X-5: track 55.2 -> 0.00 mm, vias 2 -> 0
- net TRIG_J6: track 0.00 -> 54.1 mm, vias 0 -> 1
- net X-7: track 52.3 -> 0.00 mm, vias 5 -> 0
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- added copper zone on layer 1, net +3V3
- added copper zone on layer 1, net +5V
- added copper zone on layer 1, net VCC
- added copper zone on layer 16, net VCC
Other:
- outline, holes or cut-outs redrawn
- board text added: "Range Cape"
