File: designs/range_cape/range_cape.sch (EAGLE design)
At the start: 37 parts, among them J1 22-05-7048-04, J10 22-05-7048-04, J11 22-05-7048-04, J12 22-05-7048-04, J2 22-05-7048-04, J3 22-05-7048-04, J4 22-05-7048-04, J5 22-05-7048-04, J6 22-05-7048-04, J7 22-05-7048-04, J8 22-05-7048-04, J9 22-05-7048-04, U5 LMS8117AMP-3.3, U6 MSP430FR5739IDA

Commit message: done with range cape
Parts:
- renumbered J1 to X4, J10 to X12, J11 to X9, J12 to X8, J2 to X5, J3 to X2, J4 to X3, J5 to X1, J6 to X6, J7 to X11, J8 to X10, J9 to X7
Connections:
- removed net N$10: X11-2.S
- removed net N$11: X10-2.S
- removed net N$12: X10-3.S
- removed net N$18: X7-2.S
- removed net N$19: X7-3.S
- removed net N$22: X12-2.S
- removed net N$23: X12-3.S
- removed net N$26: X9-2.S
- removed net N$27: X9-3.S
- removed net N$30: X8-2.S
- removed net N$31: X8-3.S
- removed net N$34: X6-3.S
- removed net N$35: X6-2.S
- removed net N$41: X1-3.S
- removed net N$42: X1-2.S
- removed net N$43: X3-3.S
- removed net N$44: X3-2.S
- removed net N$46: X2-3.S
- removed net N$47: X2-2.S
- removed net N$50: X5-3.S
- removed net N$51: X5-2.S
- removed net N$54: X4-3.S
- removed net N$55: X4-2.S
- removed net N$7: X11-3.S
- new net MSP_ADC0: U6.P1.0, X10-3.S
- new net MSP_ADC1: U6.P1.1, X9-3.S
- new net MSP_ADC12: U6.P3.0, X7-3.S
- new net MSP_ADC13: U6.P3.1, X6-3.S
- new net MSP_ADC14: U6.P3.2, X5-3.S
- new net MSP_ADC15: U6.P3.3, X4-3.S
- new net MSP_ADC2: U6.P1.2, X8-3.S
- new net MSP_ADC5: U6.P1.5, X1-3.S
- new net MSP_ADC6: U6.P2.3, X12-3.S
- new net MSP_ADC7: U6.P2.4, X11-3.S
- new net X-1: U6.P2.5, X1-2.S
- new net X-10: U6.P3.6, X10-2.S
- new net X-11: U6.P3.5, X11-2.S
- new net X-12: U6.P3.4, X12-2.S
- new net X-2: U6.P2.6, X2-2.S
- new net X-3: U6.PJ.5/XOUT, X3-2.S
- new net X-4: U6.PJ.4/XIN, X4-2.S
- new net X-5: U6.P2.0, X5-2.S
- new net X-6: U6.P2.1, X6-2.S
- new net X-7: U6.P2.2, X7-2.S
- new net X-8: U6.P2.7, X8-2.S
- new net X-9: U6.P3.7, X9-2.S
- net MSP_ADC3: now also X3-3.S
- net MSP_ADC4: now also X2-3.S

Commit message: pushing up frist rev of some capes
Parts:
- removed C12: 40nF, SparkFun-Capacitors:CAP0805
- removed D1: 3_3V_PWR, SparkFun-LED:LED-FKIT-1206
- removed D2: 5V_PWR, SparkFun-LED:LED-FKIT-1206
- removed D3: 1N4004, diode:1N4004
- removed JP1: 2514-6002UB, msp_jtag:2514-6002UB
- removed PL6: (no value), con-molex-2:555X-2H
- removed R10: 330, rcl:R-US_R0805W
- removed U6: MSP430FR5739IDA, TI-MSP430FR5739:MSP430FR5739IDA
- removed X11, X4: 22-05-7048-04, con-molex:22-05-7048-04
- added AUX1, AUX2, AUX3, AUX4, AUX5, AUX6, AUX7, AUX8: (no value), SparkFun-Connectors:M03LOCK
- added C1, C7: .1uF, 3-3_fixed:C3216X5R1A106K
- added C13, C17, C18, C2, C3, C4, C5, C6, C8, C9: 10uF, 3-3_fixed:C3216X5R1A106K
- added C19, C20, C21, C26, C27, C28: 10uF, 5v_fixed:C3216X5R1A106K
- added C23, C24, C29, C30, C31: 3.3uF, 5v_fixed:C3216X7R1E335K
- added C25: 620pF, 5v_fixed:GRM1555C1E621JA01D
- added C32: 100nF, 3-3_fixed:C0603C104K3RACTU
- added C33: 390pF, 3-3_fixed:08055C391KAT2A
- added J11: 22-05-7028-02, con-molex:22-05-7028-02
- added J12: EXTERNAL_DEBUG_CON, jtag_interface:EXTERNAL_DEBUG_CON
- added L1, L2: 2.2uH, 5v_fixed:IHLP1212BZER2R2M11
- added R12, R13, R14, R15, R16, R17, R18, R19, R20, R21, R22, R23, R24, R25, R26, R27: (no value), rcl:R-US_R0402
- added R3, R4: 100k, 5v_fixed:CRCW0402100KFKED
- added U$2: IEEE, TIparts:IEEE
- added U1, U4: SN74CBT3383PW, range_cape:SN74CBT3383PW
- added U2: TPS62143RGTR, 5v_fixed:TPS62143RGTR
- added U3: TPS62132RGTR, 3-3_fixed:TPS62132RGTR
- C10, C11: device SparkFun-Capacitors:10UF-16V-10%(TANT) -> rcl:C-USC0805
- C14, C15: device SparkFun-Capacitors:CAP0805 -> rcl:C-USC0805
- C16: device SparkFun-Capacitors:CAP0805 -> rcl:C-USC0603
- C22: value 100uF -> 3.3uF; device SparkFun-Capacitors:100UF-10V-10%(TANT) -> 5v_fixed:C3216X7R1E335K
- R5: value 330 -> 200k; device rcl:R-US_R0805W -> rcl:R-US_R0603
- R6: value 220 -> 200k; device rcl:R-US_R0805W -> rcl:R-US_R0603
- R7, R8, R9: device rcl:R-US_R0805W -> rcl:R-US_R0603
- U$3: value NANO_FUSE -> MSP430FR5969; device custom_fuses:NANO_FUSE -> range_cape:MSP430FR5969
- U5: value LMS8117AMP-3.3 -> DRV8830DGQR; device NSC-LMS8117AMP:LMS8117AMP-3.3 -> Texas Instruments_By_element14_Batch_1:DRV8830DGQR
- renumbered X1 to J9, X10 to J5, X12 to J3, X2 to J7, X3 to J8, X5 to J6, X6 to J10, X7 to J4, X8 to J1, X9 to J2
Connections:
- removed net MSP_ADC0: J5-3.S, U6.P1.0
- removed net MSP_ADC1: J2-3.S, U6.P1.1
- removed net MSP_ADC12: J4-3.S, U6.P3.0
- removed net MSP_ADC13: J10-3.S, U6.P3.1
- removed net MSP_ADC14: J6-3.S, U6.P3.2
- removed net MSP_ADC15: U6.P3.3, X4-3.S
- removed net MSP_ADC2: J1-3.S, U6.P1.2
- removed net MSP_ADC3: J8-3.S, U6.P1.3
- removed net MSP_ADC4: J7-3.S, U6.P1.4
- removed net MSP_ADC5: J9-3.S, U6.P1.5
- removed net MSP_ADC6: J3-3.S, U6.P2.3
- removed net MSP_ADC7: U6.P2.4, X11-3.S
- removed net N$13: D2.A, R10.1
- removed net N$6: D1.A, R5.2
- removed net VCORE: C12.2, U6.VCORE
- removed net X-1: J9-2.S, U6.P2.5
- removed net X-10: J5-2.S, U6.P3.6
- removed net X-11: U6.P3.5, X11-2.S
- removed net X-12: J3-2.S, U6.P3.4
- removed net X-2: J7-2.S, U6.P2.6
- removed net X-3: J8-2.S, U6.PJ.5/XOUT
- removed net X-4: U6.PJ.4/XIN, X4-2.S
- removed net X-5: J6-2.S, U6.P2.0
- removed net X-6: J10-2.S, U6.P2.1
- removed net X-7: J4-2.S, U6.P2.2
- removed net X-8: J1-2.S, U6.P2.7
- removed net X-9: J2-2.S, U6.P3.7
- new net DVCC: C14.1, C15.1, U$3.AVCC, U$3.DVCC
- new net ECHO1: U4.S5
- new net ECHO10: U4.S10
- new net ECHO2: U4.S4
- new net ECHO3: U4.S3
- new net ECHO4: U4.S2
- new net ECHO5: U4.S1
- new net ECHO6: U4.S6
- new net ECHO7: U4.S7
- new net ECHO8: U4.S8
- new net ECHO9: U4.S9
- new net N$12: C10.1, R5.1, U4.DREF, U4.GREF
- new net N$2: L2.1, U3.SW_2
- new net N$20: C33.1, U3.SS_TR
- new net N$5: L1.1, U2.SW_2
- new net N$7: C25.1, U2.SS_TR
- new net PWM_C1: R12.2, U1.S1
- new net PWM_C2: R13.2, U1.S2
- new net PWM_C3: R14.2, U1.S3
- new net PWM_C4: R15.2, U1.S4
- new net PWM_C5: R16.2, U1.S5
- new net PWM_C6: R17.2, U1.S6
- new net PWM_C7: R18.2, U1.S7
- new net PWM_C8: R19.2, U1.S8
- new net PWM_IN_1: AUX1.1, R20.1, U1.D1
- new net PWM_IN_2: AUX2.1, R21.1, U1.D2
- new net PWM_IN_3: AUX3.1, R22.1, U1.D3
- new net PWM_IN_4: AUX4.1, R23.1, U1.D4
- new net PWM_OUT_1: AUX5.1, R24.1, U1.D5
- new net PWM_OUT_2: AUX6.1, R25.1, U1.D6
- new net PWM_OUT_3: AUX7.1, R26.1, U1.D7
- new net PWM_OUT_4: AUX8.1, R27.1, U1.D8
- new net TRIG_J1: J1-2.S
- new net TRIG_J10: J10-2.S
- new net TRIG_J2: J2-2.S
- new net TRIG_J3: J3-2.S
- new net TRIG_J4: J4-2.S, J5-2.S
- new net TRIG_J6: J6-2.S, J7-2.S
- new net TRIG_J8: J8-2.S
- new net TRIG_J9: J9-2.S
- new net VCC: C22.1, C23.1, C24.1, C29.1, C30.1, C31.1, C32.1, J11-1.S, U2.AVIN, U2.EN, U2.PVIN_2, U3.AVIN, U3.EN, U3.PVIN_2
- new net X1: J1-3.S, U4.D10
- new net X10: J10-3.S, U4.D5
- new net X2: J2-3.S, U4.D9
- new net X3: J3-3.S, U4.D8
- new net X4: J4-3.S, U4.D7
- new net X5: J5-3.S, U4.D6
- new net X6: J6-3.S, U4.D1
- new net X7: J7-3.S, U4.D2
- new net X8: J8-3.S, U4.D3
- new net X9: J9-3.S, U4.D4
- net +3V3: now also C26.1, C27.1, C28.1, L2.2, R12.1, R13.1, R14.1, R15.1, R16.1, R17.1, R18.1, R19.1, R4.1, U1.SREF, U3.FSW, U3.VOS, U4.SREF; no longer C11.+, C14.1, C15.1, R5.1, R6.2, U5.VOUT, U6.AVCC, U6.DVCC
- net +5V: now also AUX1.2, AUX2.2, AUX3.2, AUX4.2, AUX5.2, AUX6.2, AUX7.2, AUX8.2, C1.1, C13.1, C17.1, C18.1, C19.1, C2.1, C20.1, C21.1, C3.1, C4.1, C5.1, C6.1, C7.1, C8.1, C9.1, L1.2, R20.2, R21.2, R22.2, R23.2, R24.2, R25.2, R26.2, R27.2, R3.1, R5.2, R6.2, U$1P9.VDD_5V@1, U$1P9.VDD_5V@2, U2.FSW, U2.VOS; no longer C10.+, C22.+, D3.C, R10.2, U5.IN, X11-1.S, X4-1.S
- net GND: now also AUX1.3, AUX2.3, AUX3.3, AUX4.3, AUX5.3, AUX6.3, AUX7.3, AUX8.3, C1.2, C10.2, C11.2, C13.2, C17.2, C18.2, C19.2, C2.2, C20.2, C21.2, C22.2, C23.2, C24.2, C25.2, C26.2, C27.2, C28.2, C29.2, C3.2, C30.2, C31.2, C32.2, C33.2, C4.2, C5.2, C6.2, C7.2, C8.2, C9.2, J11-2.S, J12.10, U1.GND, U2.AGND, U2.DEF, U2.EP, U2.FB, U2.PGND_2, U3.AGND, U3.DEF, U3.EP, U3.FB, U3.PGND_2, U4.GND; no longer C10.-, C11.-, C12.1, C22.-, D1.C, D2.C, JP1.9, PL6-1.S, U5.GND, U6.AVSS, U6.AVSS_2, U6.DVSS, X11-4.S, X4-4.S
- net N$14: now also R3.2, U2.PG; no longer D3.A, U$3.2
- net N$15: now also R4.2, U3.PG; no longer PL6-2.S, U$3.1
- net N$4: now also C11.1, U1.DREF, U1.GREF; no longer JP1.4
- net N$8: now also J12.12; no longer JP1.11
- net N$9: now also J12.1; no longer JP1.2
- net RESET: no longer U6.!RST!/NMI/SBWTDIO
- net SCL: no longer U6.P1.7
- net SDA: no longer U6.P1.6
- net TCK: now also J12.8; no longer JP1.7, U6.PJ.3
- net TDI: now also J12.4; no longer JP1.3, U6.PJ.1
- net TDO: now also J12.2; no longer JP1.1, U6.PJ.0
- net TEST: now also J12.7; no longer JP1.8, U6.TEST/SBWTCK
- net TMS: now also J12.6; no longer JP1.5, U6.PJ.2
