File: designs/Servo cape/servo_cape.brd (EAGLE design)
At the start: 160 x 100 mm, 47 parts, among them J1 22-05-7038-03, J10 22-05-7038-03, J2 22-05-7038-03, J3 22-05-7038-03, J4 22-05-7038-03, J5 22-05-7038-03, J6 22-05-7038-03, J7 22-05-7038-03, J8 22-05-7038-03, J9 22-05-7038-03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

Commit message: servo cape
Parts:
- removed J10, J8, J9: 22-05-7038-03, con-molex:7395-03
- moved J5 232.7 mm to (84.1, 15.0), turned to 90 degrees
- moved J7 222.7 mm to (84.1, 6.10), turned to 90 degrees
- moved J4 222.7 mm to (84.1, 23.6), turned to 90 degrees
- moved J3 213.2 mm to (84.1, 32.5), turned to 90 degrees
- moved U$12 208.7 mm to (53.3, 9.40)
- moved J2 204.0 mm to (84.1, 41.1), turned to 90 degrees
- moved J1 195.3 mm to (84.1, 49.8), turned to 90 degrees
- moved J6 165.3 mm to (8.89, 46.5), turned to 270 degrees
- moved S1 146.0 mm to (70.9, 12.7), turned to 180 degrees
- moved U$3 132.0 mm to (29.2, 9.14)
- moved U6 115.6 mm to (57.4, 25.9)
- moved D3 102.7 mm to (29.2, 13.5)
- moved DATA_POWER 100.4 mm to (5.08, 5.08)
- moved SERVO_PWR1 100.4 mm to (5.08, 11.4)
- moved SERVO_PWR2 100.4 mm to (5.08, 17.8)
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Connections:
- net +5V_SUPPLY2: no longer J10.2, J8.2, J9.2
- net GND_SUPPLY2: no longer J10.3, J8.3, J9.3
- net SERVO_10: no longer J10.1
- net SERVO_8: no longer J8.1
- net SERVO_9: no longer J9.1
Other:
- outline, holes or cut-outs redrawn
