File: designs/Servo cape/servo_cape.sch (EAGLE design)
At the start: 47 parts, among them J1 22-05-7038-03, J10 22-05-7038-03, J2 22-05-7038-03, J3 22-05-7038-03, J4 22-05-7038-03, J5 22-05-7038-03, J6 22-05-7038-03, J7 22-05-7038-03, J8 22-05-7038-03, J9 22-05-7038-03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

Commit message: servo cape
Parts:
- removed J10, J8, J9: 22-05-7038-03, con-molex:22-05-7038-03
Connections:
- net +5V_SUPPLY2: no longer J10-2.S, J8-2.S, J9-2.S
- net GND_SUPPLY2: no longer J10-3.S, J8-3.S, J9-3.S
- net SERVO_10: no longer J10-1.S
- net SERVO_8: no longer J8-1.S
- net SERVO_9: no longer J9-1.S
Changed lines of the file:
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@@
 <?xml version="1.0" encoding="utf-8"?>
 <!DOCTYPE eagle SYSTEM "eagle.dtd">
-<eagle version="7.3.0">
+<eagle version="7.2.0">
 <drawing>
 <settings>
@@
 <part name="J5" library="con-molex" deviceset="22-?-03" device="05-7038"/>
 <part name="J6" library="con-molex" deviceset="22-?-03" device="05-7038"/>
-<part name="J7" library="con-molex" deviceset="22-?-03" device="05-7038"/>
-<part name="J8" library="con-molex" deviceset="22-?-03" device="05-7038"/>
-<part name="J9" library="con-molex" deviceset="22-?-03" device="05-7038"/>
-<part name="J10" library="con-molex" deviceset="22-?-03" device="05-7038"/>
 <part name="U$12" library="range_cape" deviceset="DEBUG_CON" device=""/>
 <part name="SERVO_PWR1" library="con-molex" deviceset="22-?-02" device="05-7028"/>
@@
 <part name="R14" library="rcl" deviceset="R-US_" device="R0805W" value="330"/>
 <part name="GND4" library="SparkFun-Aesthetics" deviceset="GND" device=""/>
+<part name="J7" library="con-molex" deviceset="22-?-03" device="05-7038"/>
 </parts>
 <sheets>
@@
 <instance part="J6" gate="-2" x="167.64" y="157.48"/>
 <instance part="J6" gate="-3" x="167.64" y="152.4"/>
-<instance part="J7" gate="-1" x="167.64" y="144.78"/>
-<instance part="J7" gate="-2" x="167.64" y="139.7"/>
-<instance part="J7" gate="-3" x="167.64" y="134.62"/>
-<instance part="J8" gate="-1" x="167.64" y="127"/>
-<instance part="J8" gate="-2" x="167.64" y="121.92"/>
-<instance part="J8" gate="-3" x="167.64" y="116.84"/>
-<instance part="J9" gate="-1" x="167.64" y="109.22"/>
-<instance part="J9" gate="-2" x="167.64" y="104.14"/>
-<instance part="J9" gate="-3" x="167.64" y="99.06"/>
-<instance part="J10" gate="-1" x="167.64" y="91.44"/>
-<instance part="J10" gate="-2" x="167.64" y="86.36"/>
-<instance part="J10" gate="-3" x="167.64" y="81.28"/>
 <instance part="SERVO_PWR1" gate="-1" x="66.04" y="170.18"/>
 <instance part="SERVO_PWR1" gate="-2" x="66.04" y="165.1"/>
@@
 <instance part="D5" gate="G$1" x="215.9" y="58.42" rot="R270"/>
 <instance part="R12" gate="G$1" x="220.98" y="68.58" rot="R90"/>
+<instance part="J7" gate="-1" x="167.64" y="144.78"/>
+<instance part="J7" gate="-2" x="167.64" y="139.7"/>
+<instance part="J7" gate="-3" x="167.64" y="134.62"/>
 </instances>
 <busses>
@@
 </segment>
 <segment>
-<wire x1="157.48" y1="86.36" x2="157.48" y2="104.14" width="0.1524" layer="91"/>
-<wire x1="157.48" y1="104.14" x2="157.48" y2="121.92" width="0.1524" layer="91"/>
-<wire x1="157.48" y1="121.92" x2="157.48" y2="139.7" width="0.1524" layer="91"/>
+<wire x1="157.48" y1="76.2" x2="157.48" y2="139.7" width="0.1524" layer="91"/>
 <wire x1="157.48" y1="139.7" x2="157.48" y2="157.48" width="0.1524" layer="91"/>
 <wire x1="157.48" y1="157.48" x2="157.48" y2="172.72" width="0.1524" layer="91"/>
@@
 <wire x1="165.1" y1="157.48" x2="157.48" y2="157.48" width="0.1524" layer="91"/>
 <junction x="157.48" y="157.48"/>
+<pinref part="R11" gate="G$1" pin="2"/>
 <pinref part="J7" gate="-2" pin="S"/>
 <wire x1="165.1" y1="139.7" x2="157.48" y2="139.7" width="0.1524" layer="91"/>
 <junction x="157.48" y="139.7"/>
-<pinref part="J8" gate="-2" pin="S"/>
-<wire x1="165.1" y1="121.92" x2="157.48" y2="121.92" width="0.1524" layer="91"/>
-<junction x="157.48" y="121.92"/>
-<pinref part="J9" gate="-2" pin="S"/>
-<wire x1="165.1" y1="104.14" x2="157.48" y2="104.14" width="0.1524" layer="91"/>
-<junction x="157.48" y="104.14"/>
-<pinref part="J10" gate="-2" pin="S"/>
-<wire x1="165.1" y1="86.36" x2="157.48" y2="86.36" width="0.1524" layer="91"/>
-<pinref part="R11" gate="G$1" pin="2"/>
-<wire x1="157.48" y1="76.2" x2="157.48" y2="86.36" width="0.1524" layer="91"/>
-<junction x="157.48" y="86.36"/>
 </segment>
 </net>
@@
 </segment>
 <segment>
-<pinref part="J10" gate="-3" pin="S"/>
-<wire x1="152.4" y1="81.28" x2="165.1" y2="81.28" width="0.1524" layer="91"/>
-<pinref part="J9" gate="-3" pin="S"/>
-<wire x1="165.1" y1="99.06" x2="152.4" y2="99.06" width="0.1524" layer="91"/>
-<wire x1="152.4" y1="99.06" x2="152.4" y2="81.28" width="0.1524" layer="91"/>
-<pinref part="J8" gate="-3" pin="S"/>
-<wire x1="165.1" y1="116.84" x2="152.4" y2="116.84" width="0.1524" layer="91"/>
-<wire x1="152.4" y1="116.84" x2="152.4" y2="99.06" width="0.1524" layer="91"/>
-<junction x="152.4" y="99.06"/>
-<pinref part="J7" gate="-3" pin="S"/>
-<wire x1="165.1" y1="134.62" x2="152.4" y2="134.62" width="0.1524" layer="91"/>
-<wire x1="152.4" y1="134.62" x2="152.4" y2="116.84" width="0.1524" layer="91"/>
-<junction x="152.4" y="116.84"/>
+<wire x1="152.4" y1="152.4" x2="152.4" y2="134.62" width="0.1524" layer="91"/>
 <pinref part="J6" gate="-3" pin="S"/>
+<wire x1="152.4" y1="134.62" x2="152.4" y2="81.28" width="0.1524" layer="91"/>
 <wire x1="165.1" y1="152.4" x2="152.4" y2="152.4" width="0.1524" layer="91"/>
-<wire x1="152.4" y1="152.4" x2="152.4" y2="134.62" width="0.1524" layer="91"/>
-<junction x="152.4" y="134.62"/>
 <wire x1="152.4" y1="81.28" x2="144.78" y2="81.28" width="0.1524" layer="91"/>
-<junction x="152.4" y="81.28"/>
 <label x="142.24" y="81.28" size="1.27" layer="95" rot="R180" xref="yes"/>
 <pinref part="D4" gate="G$1" pin="C"/>
@@
 <wire x1="144.78" y1="71.12" x2="144.78" y2="81.28" width="0.1524" layer="91"/>
 <junction x="144.78" y="81.28"/>
+<pinref part="J7" gate="-3" pin="S"/>
+<wire x1="165.1" y1="134.62" x2="152.4" y2="134.62" width="0.1524" layer="91"/>
+<junction x="152.4" y="134.62"/>
 </segment>
 </net>
@@
 </segment>
 </net>
-<net name="SERVO_9" class="0">
-<segment>
-<pinref part="J9" gate="-1" pin="S"/>
-<wire x1="165.1" y1="109.22" x2="144.78" y2="109.22" width="0.1524" layer="91"/>
-<label x="144.78" y="109.22" size="1.27" layer="95" rot="R180" xref="yes"/>
-</segment>
-</net>
-<net name="SERVO_8" class="0">
-<segment>
-<pinref part="J8" gate="-1" pin="S"/>
-<wire x1="165.1" y1="127" x2="144.78" y2="127" width="0.1524" layer="91"/>
-<label x="144.78" y="127" size="1.27" layer="95" rot="R180" xref="yes"/>
-</segment>
-</net>
-<net name="SERVO_7" class="0">
-<segment>
-<pinref part="J7" gate="-1" pin="S"/>
-<wire x1="165.1" y1="144.78" x2="144.78" y2="144.78" width="0.1524" layer="91"/>
-<label x="144.78" y="144.78" size="1.27" layer="95" rot="R180" xref="yes"/>
-</segment>
-</net>
 <net name="SERVO_6" class="0">
 <segment>
@@
 <wire x1="165.1" y1="162.56" x2="144.78" y2="162.56" width="0.1524" layer="91"/>
 <label x="144.78" y="162.56" size="1.27" layer="95" rot="R180" xref="yes"/>
-</segment>
-</net>
-<net name="SERVO_10" class="0">
-<segment>
-<pinref part="J10" gate="-1" pin="S"/>
-<wire x1="165.1" y1="91.44" x2="144.78" y2="91.44" width="0.1524" layer="91"/>
-<label x="144.78" y="91.44" size="1.27" layer="95" rot="R180" xref="yes"/>
 </segment>
 </net>
@@
 </segment>
 </net>
+<net name="SERVO_7" class="0">
+<segment>
+<pinref part="J7" gate="-1" pin="S"/>
+<wire x1="165.1" y1="144.78" x2="142.24" y2="144.78" width="0.1524" layer="91"/>
+<label x="142.24" y="144.78" size="1.778" layer="95" rot="R180"/>
+</segment>
+</net>
