File: designs/Servo cape/ServoCape_Rev2.sch (EAGLE design)
At the start: 31 parts, among them J1 Servo 2, J2 Servo 1, J3 Servo 3, J4 Servo 4, J5 Servo 5, J6 Servo 6, J7 Power Input, U5 LMS8117AMP-3.3

Commit message: Updating servo cape
Parts:
- removed C8: 10uF, SparkFun-Capacitors:10UF-16V-10%(TANT)
- removed D3: 1N4004, diode:1N4004
- removed JP1: (no value), jumper:JP1Q
- removed U$3: NANO_FUSE, custom_fuses:NANO_FUSE
- added IC1: PIC24FJ64GB202, microchip:ENC28J60SP
- added J8: Power Input, con-molex:22-05-7028-02
- added LED1, LED2, LED3, LED4, LED5: (no value), motherboard_i_autoroute:LED_LEDCHIPLED_1206
- added LOGICINPUT: 22-05-7028-02, con-molex:22-05-7028-02
- added R11, R12, R13, R8, R9: (no value), rcl:R-US_M0805
- added R14: Not Installed, rcl:R-US_R0402
- added R7: 4.7k, rcl:R-US_R0805
- added U$4: Switch1, Parts4Class:MC32882_SW
- added U$5: Switch2, Parts4Class:MC32882_SW
- C1, C2, C3: device rcl:C-USC0805K -> rcl:C-USC0805
- C4: value .1uF -> 10uF; device rcl:C-USC0805K -> rcl:C-USC0805
- C6: value 100uF -> 10uF; device SparkFun-Capacitors:100UF-10V-10%(TANT) -> SparkFun-Capacitors:10UF-16V-10%(TANT)
- R10, R5: value 330 -> (none)
- R6: value 0 -> 4.7k; device rcl:R-US_R0402 -> rcl:R-US_R0805
- U$1: value PIC24FJ64GB202 -> Switch3; device ServoCape:PIC24FJ64GB202 -> Parts4Class:MC32882_SW
- renumbered U5 to U2
Connections:
- removed net +5V_SUPPLY2: J1-2.S
- removed net +5V_SUPPLY3: J3-2.S
- removed net +5V_SUPPLY5: J5-2.S
- removed net +5V_SUPPLY6: J6-2.S
- removed net 6V: C6.+, C7.+, D3.C, J2-2.S, J4-2.S, R10.2, U2.IN
- removed net 6V_INPUT: J7-1.S, U$3.1
- removed net AVDD: C2.1, R6.2, U$1.AVDD
- removed net AVSS: C2.2, U$1.AVSS
- removed net GND: C1.2, C3.2, C4.2, C5.2, C6.-, C7.-, C8.-, D1.C, D2.C, J3-3.S, J6-3.S, J7-2.S, PROGRAMMING.P$10, PROGRAMMING.P$9, U$1.VSS1, U$1.VSS2, U$2P8.DGND@1, U$2P8.DGND@2, U$2P9.DGND@1, U$2P9.DGND@2, U$2P9.DGND@3, U$2P9.DGND@4, U$2P9.DGND@5, U$2P9.DGND@6, U2.GND
- removed net GND_SUPPLY1: J2-3.S
- removed net GND_SUPPLY2: J1-3.S
- removed net GND_SUPPLY4: J4-3.S
- removed net GND_SUPPLY5: J5-3.S
- removed net N$14: D3.A, U$3.2
- removed net N$2: R1.1, U$1.MCLR
- removed net N$4: C5.1, JP1.1
- removed net VDD: R3.2, R4.2
- new net +5V: C7.+, LOGICINPUT-1.S, R10.2, R14.1, U2.IN
- new net 6V_INPUT1: C4.1, J4-2.S, J5-2.S, J6-2.S, J8-1.S, R14.2
- new net 6V_INPUT2: C3.1, J1-2.S, J2-2.S, J3-2.S, J7-1.S
- new net IO1: IC1.!CS, R6.1, U$4.P2, U$4.P3
- new net IO2: IC1.VSS, R7.1, U$5.P2, U$5.P3
- new net IO3: IC1.VDDTX, R8.2
- new net IO4: IC1.CLKOUT, R13.2
- new net IO5: IC1.!RESET, R12.2
- new net IO6: IC1.RBIAS, R9.2
- new net IO7: IC1.TPOUT-, R11.2
- new net IO8: IC1.TPOUT+
- new net MCLR': IC1.VCAP, R1.1
- new net N$5: LED3.A, R11.1
- new net N$7: LED4.A, R12.1
- new net N$8: LED5.A, R13.1
- new net VSS: C1.2, C2.2, C3.2, C4.2, C5.2, C6.-, C7.-, D1.C, D2.C, IC1.LEDA, IC1.SCK, J1-3.S, J2-3.S, J3-3.S, J4-3.S, J5-3.S, J6-3.S, J7-2.S, J8-2.S, LED1.C, LED2.C, LED3.C, LED4.C, LED5.C, LOGICINPUT-2.S, PROGRAMMING.P$10, PROGRAMMING.P$9, R6.2, R7.2, U$1.P1, U$1.P4, U$2P8.DGND@1, U$2P8.DGND@2, U$2P9.DGND@1, U$2P9.DGND@2, U$2P9.DGND@3, U$2P9.DGND@4, U$2P9.DGND@5, U$2P9.DGND@6, U2.GND
- net 3.3V: now also C2.1, C6.+, IC1.TPIN+, IC1.VDD, R3.2, R4.2, U$4.P1, U$4.P4, U$5.P1, U$5.P4; no longer C4.1, C8.+, R6.1, U$1.VDD1
- net MCLR: now also C5.1, R1.2, R2.1, U$1.P2, U$1.P3
- net N$1: now also LED1.A, R8.1; no longer JP1.2, R1.2, R2.1
- net N$3: now also LED2.A, R9.1; no longer C3.1, U$1.VDDCORE
- net OC1: now also IC1.VDDOSC; no longer U$1.RB13
- net OC2: now also IC1.LEDB; no longer U$1.TMS
- net OC3: now also IC1.OSC2; no longer U$1.TDI
- net OC4: now also IC1.VSSOSC; no longer U$1.RB6
- net OC5: now also IC1.VSSPLL; no longer U$1.RA1
- net OC6: now also IC1.VSSTX; no longer U$1.RA0
- net PGC1: now also IC1.NC*; no longer U$1.RB1
- net PGD1: now also IC1.!INT; no longer U$1.RB0
- net SCL: now also IC1.SI; no longer U$1.RB3
- net SDA: now also IC1.SO; no longer U$1.RB2
Other:
- moved on the sheet: C1, C2, C5, C6, R6
