File: designs/Son_of_Dark_Power/Son_of_Dark_Powersch.sch (EAGLE design)
At the start: 74 parts, among them IC2 TS5205, J1 22-05-7048-04, J2 22-05-7028-02, J3 22-05-7028-02, J4 22-05-7028-02, J5 22-05-7028-02, J6 22-05-7028-02, J7 22-05-7028-02, J8 22-05-7028-02, J9 22-05-7028-02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

Commit message: servo cape
Parts:
- R1: value (none) -> 0 ohm
Changed lines of the file:
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@@
 <?xml version="1.0" encoding="utf-8"?>
 <!DOCTYPE eagle SYSTEM "eagle.dtd">
-<eagle version="7.3.0">
+<eagle version="7.2.0">
 <drawing>
 <settings>
@@
 <part name="C1" library="3-3_fixed" deviceset="C3216X5R1A106K" device="" value=".1uF"/>
 <part name="P+18" library="supply1" deviceset="+5V" device=""/>
-<part name="R1" library="rcl" deviceset="R-US_" device="R1206"/>
+<part name="R1" library="rcl" deviceset="R-US_" device="R1206" value="0 ohm"/>
 <part name="FRAME2" library="frames" deviceset="DINA5_L" device=""/>
 <part name="U$2" library="5v" deviceset="TPS5450DDAR" device=""/>

Commit message: Need to add switch
Parts:
- removed R13: 220, rcl:R-US_R0603
- removed R20: 49.9k, rcl:R-US_R0603
- removed S1: POWER ON, smd-special:SWS001
- removed U$12: DEBUG_CON, range_cape:DEBUG_CON
- removed U$5: MSP430F20X3, TIparts:MSP430F20X3
- added J11: PIN-CONNECTOR74089, Mother-Board-rev5:PIN-CONNECTOR74089
- added U$6: PIC16F676-I/ST, Microchip_By_element14_Batch_1:PIC16F676-I/ST
Connections:
- removed net LDS_RX: U$1P9.GPIO_15
- removed net LDS_TX: U$1P9.GPIO_14
- removed net LIDAR_DIR: U$1P9.GPIO_49
- removed net LIDAR_PWM: U$1P9.GPIO_2
- removed net N$11: C21.1, C22.1, IC2.VOUT, R11.2, R12.2, R14.2, U$5.VCC
- removed net POWER_EN: Q2.G, S1.2
- removed net RESET: C20.1, R12.1, R13.2, U$5.RTS
- removed net SCL: U$1P9.I2C2_SCL
- removed net SDA: U$1P9.I2C2_SDA
- removed net SIMO: U$1P9.GPIO_122
- removed net SOMI: U$1P9.GPIO_121
- removed net SPI_CLK: U$1P9.GPIO_120
- removed net SPI_SL0: U$1P9.GPIO_123
- removed net SPI_SL1: U$1P9.GPIO_7
- removed net TCK: U$12.7, U$5.P1.4
- removed net TDI/VPP: U$12.3, U$5.P1.6
- removed net TDO/TDI: U$12.1, U$5.P1.7
- removed net TEST/VPP: U$5.TEST
- removed net TMS: U$12.5, U$5.P1.5
- new net +3V3: C21.1, C22.1, IC2.VOUT, J11.P$1, J11.P$2, R11.2, R12.2, U$6.VDD
- new net BB_PWR_SW: U$1P9.PWR_BUT, U$6.RC5
- new net ICSPCLK: J11.P$3, J11.P$4, U$6.RA1/AN1/CIN-/VREF/ICSPCLK
- new net ICSPDAT: J11.P$5, J11.P$6, U$6.RA0/AN0/CIN+/ICSPDAT
- new net N$15: U$6.RC1/AN5
- new net N$16: U$6.RC0/AN4
- new net N$17: U$6.RA4/~T1G/OSC2/AN3/CLKOUT
- new net POWER_SIG: SPDT.C1, U$6.RC3/AN7
- new net VPP/MCLR: J11.P$7, J11.P$8, R14.2, U$6.RA3/~MCLR/VPP
- net +5V: no longer C23.1, IC2.CE, IC2.VIN
- net EN: now also Q2.G, U$6.RC4; no longer R20.2, SPDT.C1, U$5.P2.7
- net GND: now also J11.P$10, J11.P$9, U$1P9.DGND@3, U$1P9.DGND@4, U$1P9.DGND@5, U$1P9.DGND@6, U$6.VSS; no longer R20.1, S1.1, U$12.9, U$5.VSS
- net N$5: now also U$6.RC2/AN6; no longer R13.1, U$12.10, U$12.11, U$12.12
- net N$6: now also C20.1, R12.1; no longer U$12.4
- net N$8: now also U$6.RA2/AN2/COUT/T0CKI/INT; no longer U$5.P1.3
- net N$9: now also U$6.RA5/T1CKI/OSC1/CLKIN; no longer U$5.P2.6
- net VCC: now also C23.1, IC2.CE, IC2.VIN
Other:
- note added: "ICSP"
- note removed: "NOT Installed"
- moved on the sheet: C20, LED5, R12, R14, R15, R16, R17

Commit message: Done with rev 2
Parts:
- added POWER: SPST-2_5X4, ultrasonic_mount:SPST-2_5X4
Connections:
- removed net N$17: U$6.RA4/~T1G/OSC2/AN3/CLKOUT
- new net N$11: POWER.P$1, U$6.RA4/~T1G/OSC2/AN3/CLKOUT
- net GND: now also POWER.P$2
Other:
- moved on the sheet: R16, R17
Changed lines of the file:
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@@
 <?xml version="1.0" encoding="utf-8"?>
 <!DOCTYPE eagle SYSTEM "eagle.dtd">
-<eagle version="7.4.0">
+<eagle version="7.3.0">
 <drawing>
 <settings>
@@
 <part name="GND6" library="SparkFun-Aesthetics" deviceset="GND" device=""/>
 <part name="GND7" library="SparkFun-Aesthetics" deviceset="GND" device=""/>
+<part name="POWER" library="ultrasonic_mount" deviceset="SPST-2_5X4" device=""/>
+<part name="GND8" library="supply1" deviceset="GND" device=""/>
 </parts>
 <sheets>
@@
 <instance part="C21" gate="G$1" x="134.62" y="35.56"/>
 <instance part="C22" gate="G$1" x="142.24" y="35.56"/>
-<instance part="GND1" gate="1" x="27.94" y="142.24"/>
-<instance part="R16" gate="G$1" x="27.94" y="154.94" rot="R270"/>
-<instance part="R17" gate="G$1" x="27.94" y="170.18" rot="R270"/>
+<instance part="GND1" gate="1" x="17.78" y="142.24"/>
+<instance part="R16" gate="G$1" x="17.78" y="154.94" rot="R270"/>
+<instance part="R17" gate="G$1" x="17.78" y="170.18" rot="R270"/>
 <instance part="R12" gate="G$1" x="198.12" y="175.26" rot="R90"/>
 <instance part="C20" gate="G$1" x="198.12" y="157.48"/>
@@
 <instance part="J11" gate="G$1" x="365.76" y="81.28"/>
 <instance part="GND5" gate="1" x="198.12" y="144.78"/>
+<instance part="POWER" gate="G$1" x="27.94" y="132.08" rot="R270"/>
+<instance part="GND8" gate="1" x="27.94" y="116.84"/>
 </instances>
 <busses>
@@
 <pinref part="GND1" gate="1" pin="GND"/>
 <pinref part="R16" gate="G$1" pin="2"/>
-<wire x1="27.94" y1="149.86" x2="27.94" y2="144.78" width="0.1524" layer="91"/>
+<wire x1="17.78" y1="149.86" x2="17.78" y2="144.78" width="0.1524" layer="91"/>
 </segment>
 <segment>
@@
 <wire x1="198.12" y1="147.32" x2="198.12" y2="152.4" width="0.1524" layer="91"/>
 </segment>
+<segment>
+<pinref part="POWER" gate="G$1" pin="P$2"/>
+<pinref part="GND8" gate="1" pin="GND"/>
+<wire x1="27.94" y1="124.46" x2="27.94" y2="119.38" width="0.1524" layer="91"/>
+</segment>
 </net>
 <net name="VCC" class="0">
@@
 <segment>
 <pinref part="R17" gate="G$1" pin="1"/>
-<wire x1="27.94" y1="175.26" x2="27.94" y2="185.42" width="0.1524" layer="91"/>
-<label x="27.94" y="185.42" size="1.778" layer="95" rot="R270"/>
+<wire x1="17.78" y1="175.26" x2="17.78" y2="185.42" width="0.1524" layer="91"/>
+<label x="17.78" y="185.42" size="1.778" layer="95" rot="R270"/>
 </segment>
 <segment>
@@
 <pinref part="R17" gate="G$1" pin="2"/>
 <pinref part="R16" gate="G$1" pin="1"/>
-<wire x1="27.94" y1="160.02" x2="27.94" y2="162.56" width="0.1524" layer="91"/>
+<wire x1="17.78" y1="160.02" x2="17.78" y2="162.56" width="0.1524" layer="91"/>
 <pinref part="U$6" gate="A" pin="RA2/AN2/COUT/T0CKI/INT"/>
-<wire x1="27.94" y1="162.56" x2="27.94" y2="165.1" width="0.1524" layer="91"/>
-<wire x1="68.58" y1="162.56" x2="27.94" y2="162.56" width="0.1524" layer="91"/>
-<junction x="27.94" y="162.56"/>
+<wire x1="17.78" y1="162.56" x2="17.78" y2="165.1" width="0.1524" layer="91"/>
+<wire x1="68.58" y1="162.56" x2="17.78" y2="162.56" width="0.1524" layer="91"/>
+<junction x="17.78" y="162.56"/>
 </segment>
 </net>
@@
 </segment>
 </net>
-<net name="N$17" class="0">
-<segment>
-<pinref part="U$6" gate="A" pin="RA4/~T1G/OSC2/AN3/CLKOUT"/>
-<wire x1="68.58" y1="157.48" x2="63.5" y2="157.48" width="0.1524" layer="91"/>
-<label x="63.5" y="157.48" size="1.27" layer="95" rot="R180" xref="yes"/>
-</segment>
-</net>
 <net name="POWER_SIG" class="0">
 <segment>
@@
 </segment>
 </net>
+<net name="N$11" class="0">
+<segment>
+<pinref part="U$6" gate="A" pin="RA4/~T1G/OSC2/AN3/CLKOUT"/>
+<pinref part="POWER" gate="G$1" pin="P$1"/>
+<wire x1="68.58" y1="157.48" x2="27.94" y2="157.48" width="0.1524" layer="91"/>
+<wire x1="27.94" y1="157.48" x2="27.94" y2="137.16" width="0.1524" layer="91"/>
+</segment>
+</net>
