File: designs/Son_of_Dark_Power/Son_of_Dark_Power.brd (EAGLE design)
At the start: 89.4 x 55.5 mm, 73 parts, among them IC2 TS5205, J1 22-05-7048-04, J11 PIN-CONNECTOR74089, J2 22-05-7028-02, J3 22-05-7028-02, J4 22-05-7028-02, J5 22-05-7028-02, J6 22-05-7028-02, J7 22-05-7028-02, J8 22-05-7028-02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

Commit message: reverting changes back to rev 1
Parts:
- removed J11: PIN-CONNECTOR74089, Mother-Board-rev5:10-PIN-SMD
- removed POWER: SPST-2_5X4, ultrasonic_mount:SPST-TAC-4X2_5MM
- removed U$6: PIC16F676-I/ST, Microchip_By_element14_Batch_1:SOP65P640X120-14N
- added R13: 220, rcl:R0603
- added R20: 49.9k, rcl:R0603
- added S1: POWER ON, smd-special:SMS-001
- added U$12: DEBUG_CON, range_cape:DEBUG_SM
- PL5: device Son_of_Dark_Powersch:5569-2 -> con-molex-2:5569-2
- R1: value 0 ohm -> (none)
- U$5: value LOGO-IEEE -> MSP430F20X3; device Son_of_Dark_Powersch:LOGO -> TIparts:TSSOP-14
- moved U$5 40.6 mm to (20.7, 44.5), turned to 0 degrees
- moved LED5 6.45 mm to (11.7, 46.2), turned to 90 degrees
- moved C20 0.89 mm to (22.5, 37.8)
- turned R12 to 180 degrees
- turned R14 to 0 degrees
Connections:
- removed net +3V3: C21.1, C22.1, IC2.5, J11.1, J11.2, R11.2, R12.2, U$6.1
- removed net BB_PWR_SW: U$1.P9.9, U$6.5
- removed net ICSPCLK: J11.3, J11.4, U$6.12
- removed net ICSPDAT: J11.5, J11.6, U$6.13
- removed net N$15: U$6.9
- removed net N$16: U$6.10
- removed net POWER_SIG: SPDT.2, U$6.7
- removed net VPP/MCLR: J11.7, J11.8, R14.2, U$6.4
- new net LDS_RX: U$1.P9.24
- new net LDS_TX: U$1.P9.26
- new net LIDAR_DIR: U$1.P9.23
- new net LIDAR_PWM: U$1.P9.22
- new net POWER_EN: Q2.1, S1.2
- new net RESET: C20.1, R12.1, R13.2, U$5.10
- new net SCL: U$1.P9.19
- new net SDA: U$1.P9.20
- new net SIMO: U$1.P9.30
- new net SOMI: U$1.P9.29
- new net SPI_CLK: U$1.P9.31
- new net SPI_SL0: U$1.P9.28
- new net SPI_SL1: U$1.P9.42
- new net TCK: U$12.7, U$5.6
- new net TDI/VPP: U$12.3, U$5.8
- new net TDO/TDI: U$12.1, U$5.9
- new net TEST/VPP: U$5.11
- new net TMS: U$12.5, U$5.7
- net +5V: now also C23.1, IC2.1, IC2.3
- net EN: now also R20.2, SPDT.2, U$5.12; no longer Q2.1, U$6.6
- net GND: now also R20.1, S1.1, U$12.9, U$5.14; no longer J11.10, J11.9, POWER.P$2, U$1.P9.43, U$1.P9.44, U$1.P9.45, U$1.P9.46, U$6.14
- net N$11: now also C21.1, C22.1, IC2.5, R11.2, R12.2, R14.2, U$5.1; no longer POWER.P$1, U$6.3
- net N$5: now also R13.1, U$12.10, U$12.11, U$12.12; no longer U$6.8
- net N$6: now also U$12.4; no longer C20.1, R12.1
- net N$8: now also U$5.5; no longer U$6.11
- net N$9: now also U$5.13; no longer U$6.2
- net VCC: no longer C23.1, IC2.1, IC2.3
Routing:
- net BB_PWR_SW: track 94.5 -> 0.00 mm, vias 2 -> 0
- net POWER_EN: track 0.00 -> 51.5 mm, vias 0 -> 1
- net +5V: track 105.0 -> 147.7 mm, vias 4 -> 5
- net +3V3: track 39.0 -> 0.00 mm, vias 3 -> 0
- net EN: track 75.5 -> 49.3 mm
- net RESET: track 0.00 -> 23.8 mm, vias 0 -> 1
- net VPP/MCLR: track 15.9 -> 0.00 mm, vias 2 -> 0
- net N$11: track 18.0 -> 30.9 mm, vias 3 -> 2
- net N$5: track 0.00 -> 12.4 mm
- net GND: track 116.8 -> 106.0 mm
- net VCC: track 20.5 -> 11.8 mm
- net ICSPDAT: track 8.05 -> 0.00 mm, vias 1 -> 0
- net TDO/TDI: track 0.00 -> 7.77 mm, vias 0 -> 1
- net TMS: track 0.00 -> 6.65 mm, vias 0 -> 1
- net POWER_SIG: track 5.43 -> 0.00 mm
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Other:
- outline, holes or cut-outs redrawn
