File: designs/Son_of_Dark_Power/Son_of_Dark_Power.sch (EAGLE design)
At the start: 73 parts, among them IC2 TS5205, J1 22-05-7048-04, J11 PIN-CONNECTOR74089, J2 22-05-7028-02, J3 22-05-7028-02, J4 22-05-7028-02, J5 22-05-7028-02, J6 22-05-7028-02, J7 22-05-7028-02, J8 22-05-7028-02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

Commit message: reverting changes back to rev 1
Parts:
- removed J11: PIN-CONNECTOR74089, Mother-Board-rev5:PIN-CONNECTOR74089
- removed POWER: SPST-2_5X4, ultrasonic_mount:SPST-2_5X4
- removed U$6: PIC16F676-I/ST, Microchip_By_element14_Batch_1:PIC16F676-I/ST
- added R13: 220, rcl:R-US_R0603
- added R20: 49.9k, rcl:R-US_R0603
- added S1: POWER ON, smd-special:SWS001
- added U$12: DEBUG_CON, range_cape:DEBUG_CON
- PL5: device Son_of_Dark_Powersch:555X-2H -> con-molex-2:555X-2H
- R1: value 0 ohm -> (none)
- U$5: value LOGO-IEEE -> MSP430F20X3; device Son_of_Dark_Powersch:LOGO-IEEE -> TIparts:MSP430F20X3
Connections:
- removed net +3V3: C21.1, C22.1, IC2.VOUT, J11.P$1, J11.P$2, R11.2, R12.2, U$6.VDD
- removed net BB_PWR_SW: U$1P9.PWR_BUT, U$6.RC5
- removed net ICSPCLK: J11.P$3, J11.P$4, U$6.RA1/AN1/CIN-/VREF/ICSPCLK
- removed net ICSPDAT: J11.P$5, J11.P$6, U$6.RA0/AN0/CIN+/ICSPDAT
- removed net N$15: U$6.RC1/AN5
- removed net N$16: U$6.RC0/AN4
- removed net POWER_SIG: SPDT.C1, U$6.RC3/AN7
- removed net VPP/MCLR: J11.P$7, J11.P$8, R14.2, U$6.RA3/~MCLR/VPP
- new net LDS_RX: U$1P9.GPIO_15
- new net LDS_TX: U$1P9.GPIO_14
- new net LIDAR_DIR: U$1P9.GPIO_49
- new net LIDAR_PWM: U$1P9.GPIO_2
- new net POWER_EN: Q2.G, S1.2
- new net RESET: C20.1, R12.1, R13.2, U$5.RTS
- new net SCL: U$1P9.I2C2_SCL
- new net SDA: U$1P9.I2C2_SDA
- new net SIMO: U$1P9.GPIO_122
- new net SOMI: U$1P9.GPIO_121
- new net SPI_CLK: U$1P9.GPIO_120
- new net SPI_SL0: U$1P9.GPIO_123
- new net SPI_SL1: U$1P9.GPIO_7
- new net TCK: U$12.7, U$5.P1.4
- new net TDI/VPP: U$12.3, U$5.P1.6
- new net TDO/TDI: U$12.1, U$5.P1.7
- new net TEST/VPP: U$5.TEST
- new net TMS: U$12.5, U$5.P1.5
- net +5V: now also C23.1, IC2.CE, IC2.VIN
- net EN: now also R20.2, SPDT.C1, U$5.P2.7; no longer Q2.G, U$6.RC4
- net GND: now also R20.1, S1.1, U$12.9, U$5.VSS; no longer J11.P$10, J11.P$9, POWER.P$2, U$1P9.DGND@3, U$1P9.DGND@4, U$1P9.DGND@5, U$1P9.DGND@6, U$6.VSS
- net N$11: now also C21.1, C22.1, IC2.VOUT, R11.2, R12.2, R14.2, U$5.VCC; no longer POWER.P$1, U$6.RA4/~T1G/OSC2/AN3/CLKOUT
- net N$5: now also R13.1, U$12.10, U$12.11, U$12.12; no longer U$6.RC2/AN6
- net N$6: now also U$12.4; no longer C20.1, R12.1
- net N$8: now also U$5.P1.3; no longer U$6.RA2/AN2/COUT/T0CKI/INT
- net N$9: now also U$5.P2.6; no longer U$6.RA5/T1CKI/OSC1/CLKIN
- net VCC: no longer C23.1, IC2.CE, IC2.VIN
Other:
- note added: "NOT Installed"
- note removed: "ICSP"
- moved on the sheet: C20, LED5, R12, R14, R15, R16, R17
