File: designs/Son_of_Dark_Power/Son_of_Dark_Power.sch (EAGLE design)
At the start: 72 parts, among them IC2 TS5205, J1 22-05-7048-04, J11 PIN-CONNECTOR74089, J2 22-05-7028-02, J3 22-05-7028-02, J4 22-05-7028-02, J5 22-05-7028-02, J6 22-05-7028-02, J7 22-05-7028-02, J8 22-05-7028-02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

Commit message: Remaing Files
Parts:
- added U$5: LOGO-IEEE, Son_of_Dark_Powersch:LOGO-IEEE
- PL5: device con-molex-2:555X-2H -> Son_of_Dark_Powersch:555X-2H
Changed lines of the file:
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@@
 <part name="FRAME5" library="frames" deviceset="FRAME_A_L" device=""/>
 <part name="J1" library="con-molex" deviceset="22-?-04" device="05-7048"/>
-<part name="PL5" library="con-molex-2" deviceset="555X-2" device="H"/>
+<part name="PL5" library="Son_of_Dark_Powersch" deviceset="555X-2" device="H"/>
 <part name="J2" library="con-molex" deviceset="22-?-02" device="05-7028"/>
 <part name="J3" library="con-molex" deviceset="22-?-02" device="05-7028"/>
@@
 <part name="POWER" library="ultrasonic_mount" deviceset="SPST-2_5X4" device=""/>
 <part name="GND8" library="supply1" deviceset="GND" device=""/>
+<part name="U$5" library="Son_of_Dark_Powersch" deviceset="LOGO-IEEE" device=""/>
 </parts>
 <sheets>
@@
 <instance part="GND6" gate="1" x="142.24" y="45.72"/>
 <instance part="GND7" gate="1" x="81.28" y="45.72"/>
+<instance part="U$5" gate="G$1" x="215.9" y="170.18"/>
 </instances>
 <busses>
