File: designs/Son_of_Dark_Power_Rev2/Son_of_Dark_Powersch.brd (EAGLE design)
At the start: 89.4 x 55.5 mm, 71 parts, among them IC2 TS5205, J1 22-05-7048-04, J11 PIN-CONNECTOR74089, J2 22-05-7028-02, J3 22-05-7028-02, J4 22-05-7028-02, J5 22-05-7028-02, J6 22-05-7028-02, J7 22-05-7028-02, J8 22-05-7028-02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

Commit message: Update to the BOM
Parts:
- C21: value (none) -> 0.1uF
- C22, C23: value (none) -> 1uF
Changed lines of the file:
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@@
 <attribute name="NAME" x="81.5071" y="53.8211" size="1.016" layer="25" ratio="10" rot="R270"/>
 </element>
-<element name="C21" library="rcl" package="C0603" value="" x="22.352" y="31.496" smashed="yes" rot="MR0">
+<element name="C21" library="rcl" package="C0603" value="0.1uF" x="22.352" y="31.496" smashed="yes" rot="MR0">
 <attribute name="NAME" x="23.241" y="32.131" size="0.8128" layer="26" rot="MR0"/>
 <attribute name="VALUE" x="22.987" y="29.591" size="1.27" layer="28" rot="MR0"/>
 </element>
-<element name="C22" library="rcl" package="C0603" value="" x="22.352" y="35.306" smashed="yes" rot="MR0">
+<element name="C22" library="rcl" package="C0603" value="1uF" x="22.352" y="35.306" smashed="yes" rot="MR0">
 <attribute name="NAME" x="23.749" y="35.941" size="0.8128" layer="26" rot="MR0"/>
 <attribute name="VALUE" x="22.987" y="33.401" size="1.27" layer="28" rot="MR0"/>
@@
 <attribute name="NAME" x="24.765" y="29.337" size="0.8128" layer="26" rot="MR270"/>
 </element>
-<element name="C23" library="rcl" package="C0603" value="" x="22.352" y="24.511" smashed="yes" rot="MR0">
+<element name="C23" library="rcl" package="C0603" value="1uF" x="22.352" y="24.511" smashed="yes" rot="MR0">
 <attribute name="NAME" x="23.368" y="22.987" size="0.8128" layer="26" rot="MR0"/>
 <attribute name="VALUE" x="22.987" y="22.606" size="1.27" layer="28" rot="MR0"/>
