File: designs/Son_of_Dark_Power_Rev2/Son_of_Dark_Powersch.sch (EAGLE design)
At the start: 71 parts, among them IC2 TS5205, J1 22-05-7048-04, J11 PIN-CONNECTOR74089, J2 22-05-7028-02, J3 22-05-7028-02, J4 22-05-7028-02, J5 22-05-7028-02, J6 22-05-7028-02, J7 22-05-7028-02, J8 22-05-7028-02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

Commit message: Update to the BOM
Parts:
- C21: value (none) -> 0.1uF
- C22, C23: value (none) -> 1uF
Changed lines of the file:
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@@
 <part name="J8" library="con-molex" deviceset="22-?-02" device="05-7028"/>
 <part name="J9" library="con-molex" deviceset="22-?-02" device="05-7028"/>
-<part name="C21" library="rcl" deviceset="C-US" device="C0603"/>
-<part name="C22" library="rcl" deviceset="C-US" device="C0603"/>
+<part name="C21" library="rcl" deviceset="C-US" device="C0603" value="0.1uF"/>
+<part name="C22" library="rcl" deviceset="C-US" device="C0603" value="1uF"/>
 <part name="GND1" library="supply1" deviceset="GND" device=""/>
 <part name="R16" library="rcl" deviceset="R-US_" device="R0603" value="1.24k"/>
@@
 <part name="IC2" library="v-reg" deviceset="TS5205" device=""/>
 <part name="GND2" library="SparkFun-Aesthetics" deviceset="GND" device=""/>
-<part name="C23" library="rcl" deviceset="C-US" device="C0603"/>
+<part name="C23" library="rcl" deviceset="C-US" device="C0603" value="1uF"/>
 <part name="+3V4" library="supply1" deviceset="+3V3" device=""/>
 <part name="P+2" library="supply1" deviceset="+5V" device=""/>
