File: EagleClass/PowerSystem.brd (EAGLE design)
At the start: 29 parts, among them Q2 BSS123, Q3 BSS123

Commit message: Updating servo cape
Parts:
- added LED1: (no value), Parts4Class:SMARTLED-TTW
- added U$1: BEAGLE_BONE_BLACK_CAPE, Parts4Class:BEAGLE_BONE_BLACK_CAPE
- added U1: PIC18F46K22-I/PT, Parts4Class:QFP80P1200X1200X120-44N
- moved C16 55.4 mm to (88.6, -23.0)
- moved LED2 55.4 mm to (97.5, -25.2)
- moved LED4 55.4 mm to (97.5, -39.7)
- moved R10 55.4 mm to (97.5, -19.2)
- moved R4 55.4 mm to (97.5, -33.7)
- moved C5 55.4 mm to (88.6, -37.5)
- moved C8 55.4 mm to (62.9, -40.0)
- moved R3 55.4 mm to (51.8, -40.0)
- moved U$2 55.4 mm to (56.9, -37.5)
- moved C14 55.4 mm to (58.2, -23.9)
- moved C15 55.4 mm to (56.9, -19.2)
- moved C17 55.4 mm to (55.3, -23.9)
- moved C18 55.4 mm to (52.5, -23.9)
- moved C19 55.4 mm to (62.9, -25.5)
- moved C2 55.4 mm to (58.2, -38.4)
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Connections:
- new net N$5: LED1.A@1, U1.1
- new net SCL: U$1.P9.19, U1.20
- new net SDA: U$1.P9.20, U1.19
- net +5V: now also U1.28, U1.7
- net EN: now also U1.5
- net GND: now also LED1.C@1, U$1.P9.1, U1.29, U1.6
Routing:
- net SDA: track 0.00 -> 113.0 mm, vias 0 -> 1
- net SCL: track 0.00 -> 109.6 mm
- net N$5: track 0.00 -> 30.9 mm, vias 0 -> 1
- net +5V: track 36.2 -> 54.5 mm
- net GND: track 27.3 -> 35.5 mm, vias 10 -> 11
Other:
- board outline added: 150.4 x 57.4 mm
