File: EagleClass/PowerSystem.sch (EAGLE design)
At the start: 29 parts, among them Q2 BSS123, Q3 BSS123

Commit message: Updating servo cape
Parts:
- added LED1: (no value), Parts4Class:LED
- added U$1: BEAGLE_BONE_BLACK_CAPE, Parts4Class:BEAGLE_BONE_BLACK_CAPE
- added U1: PIC18F46K22-I/PT, Parts4Class:PIC18F46K22-I/PT
Connections:
- new net N$5: LED1.A, U1.RC7
- new net SCL: U$1P9.I2C2_SCL, U1.RA1
- new net SDA: U$1P9.I2C2_SDA, U1.RA0
- net +5V: now also U1.VDD, U1.VDD_2
- net EN: now also U1.RD7
- net GND: now also LED1.C, U$1P9.DGND@1, U1.VSS, U1.VSS_2
Changed lines of the file:
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@@
 <layer number="112" name="tSilk" color="7" fill="1" visible="no" active="yes"/>
 <layer number="113" name="IDFDebug" color="7" fill="1" visible="no" active="yes"/>
+<layer number="114" name="FRNTMAAT1" color="7" fill="1" visible="yes" active="yes"/>
+<layer number="115" name="FRNTMAAT2" color="7" fill="1" visible="yes" active="yes"/>
 <layer number="116" name="Patch_BOT" color="9" fill="4" visible="yes" active="yes"/>
+<layer number="117" name="BACKMAAT1" color="7" fill="1" visible="yes" active="yes"/>
 <layer number="118" name="Rect_Pads" color="7" fill="1" visible="no" active="no"/>
+<layer number="119" name="KAP_TEKEN" color="7" fill="1" visible="yes" active="yes"/>
+<layer number="120" name="KAP_MAAT1" color="7" fill="1" visible="yes" active="yes"/>
 <layer number="121" name="_tsilk" color="7" fill="1" visible="yes" active="yes"/>
 <layer number="122" name="_bsilk" color="7" fill="1" visible="yes" active="yes"/>
@@
 <part name="P+2" library="supply1" deviceset="+5V" device=""/>
 <part name="S1" library="smd-special" deviceset="SWS001" device="" value="POWER ON"/>
+<part name="U$1" library="Parts4Class" deviceset="BEAGLE_BONE_BLACK_CAPE" device=""/>
+<part name="U1" library="Parts4Class" deviceset="PIC18F46K22-I/PT" device=""/>
+<part name="LED1" library="Parts4Class" deviceset="LED" device=""/>
 </parts>
 <sheets>
@@
 <instance part="FRAME1" gate="G$1" x="0" y="0"/>
 <instance part="FRAME1" gate="G$2" x="172.72" y="0"/>
+<instance part="U$1" gate="P8" x="243.84" y="91.44"/>
+<instance part="U$1" gate="P9" x="160.02" y="88.9"/>
+<instance part="U1" gate="A" x="40.64" y="165.1"/>
+<instance part="LED1" gate="G$1" x="81.28" y="175.26"/>
 </instances>
 <busses>
 </busses>
 <nets>
+<net name="GND" class="0">
+<segment>
+<pinref part="U$1" gate="P9" pin="DGND@1"/>
+<wire x1="139.7" y1="114.3" x2="129.54" y2="114.3" width="0.1524" layer="91"/>
+<wire x1="129.54" y1="114.3" x2="129.54" y2="111.76" width="0.1524" layer="91"/>
+<label x="129.54" y="111.76" size="1.778" layer="95"/>
+</segment>
+<segment>
+<pinref part="LED1" gate="G$1" pin="C"/>
+<wire x1="81.28" y1="170.18" x2="81.28" y2="165.1" width="0.1524" layer="91"/>
+<label x="81.28" y="165.1" size="1.778" layer="95"/>
+</segment>
+<segment>
+<pinref part="U1" gate="A" pin="VSS_2"/>
+<wire x1="22.86" y1="127" x2="7.62" y2="127" width="0.1524" layer="91"/>
+<wire x1="7.62" y1="127" x2="7.62" y2="124.46" width="0.1524" layer="91"/>
+<pinref part="U1" gate="A" pin="VSS"/>
+<wire x1="7.62" y1="124.46" x2="7.62" y2="119.38" width="0.1524" layer="91"/>
+<wire x1="22.86" y1="124.46" x2="7.62" y2="124.46" width="0.1524" layer="91"/>
+<junction x="7.62" y="124.46"/>
+<label x="7.62" y="119.38" size="1.778" layer="95"/>
+</segment>
+</net>
+<net name="SCL" class="0">
+<segment>
+<pinref part="U$1" gate="P9" pin="I2C2_SCL"/>
+<wire x1="139.7" y1="91.44" x2="129.54" y2="91.44" width="0.1524" layer="91"/>
+<label x="127" y="91.44" size="1.778" layer="95"/>
+</segment>
+<segment>
+<pinref part="U1" gate="A" pin="RA1"/>
+<wire x1="22.86" y1="182.88" x2="17.78" y2="182.88" width="0.1524" layer="91"/>
+<label x="12.7" y="182.88" size="1.778" layer="95"/>
+</segment>
+</net>
+<net name="SDA" class="0">
+<segment>
+<pinref part="U$1" gate="P9" pin="I2C2_SDA"/>
+<wire x1="180.34" y1="91.44" x2="190.5" y2="91.44" width="0.1524" layer="91"/>
+<label x="190.5" y="91.44" size="1.778" layer="95"/>
+</segment>
+<segment>
+<pinref part="U1" gate="A" pin="RA0"/>
+<wire x1="22.86" y1="185.42" x2="17.78" y2="185.42" width="0.1524" layer="91"/>
+<label x="17.78" y="185.42" size="1.778" layer="95"/>
+</segment>
+</net>
+<net name="+5V" class="0">
+<segment>
+<pinref part="U1" gate="A" pin="VDD"/>
+<wire x1="22.86" y1="195.58" x2="7.62" y2="195.58" width="0.1524" layer="91"/>
+<wire x1="7.62" y1="195.58" x2="7.62" y2="198.12" width="0.1524" layer="91"/>
+<pinref part="U1" gate="A" pin="VDD_2"/>
+<wire x1="7.62" y1="198.12" x2="7.62" y2="205.74" width="0.1524" layer="91"/>
+<wire x1="22.86" y1="198.12" x2="7.62" y2="198.12" width="0.1524" layer="91"/>
+<junction x="7.62" y="198.12"/>
+<label x="7.62" y="205.74" size="1.778" layer="95"/>
+</segment>
+</net>
+<net name="N$5" class="0">
+<segment>
+<pinref part="U1" gate="A" pin="RC7"/>
+<pinref part="LED1" gate="G$1" pin="A"/>
+<wire x1="58.42" y1="180.34" x2="81.28" y2="180.34" width="0.1524" layer="91"/>
+<wire x1="81.28" y1="180.34" x2="81.28" y2="177.8" width="0.1524" layer="91"/>
+</segment>
+</net>
+<net name="EN" class="0">
+<segment>
+<pinref part="U1" gate="A" pin="RD7"/>
+<wire x1="58.42" y1="157.48" x2="66.04" y2="157.48" width="0.1524" layer="91"/>
+<label x="66.04" y="157.48" size="1.778" layer="95"/>
+</segment>
+</net>
 </nets>
 </sheet>
