File: designs/Motherboard/MotherboardRev1.brd (EAGLE design)
At the start: 94 parts, among them IC1 PIC24FJ64GB202, J1 Servo 2, J2 Servo 1, J3 Servo 3, J4 Servo 4, J5 Servo 5, J6 Servo 6, Q1 BSS123, Q2 BSS123, Q3 BSS123, Q4 BSS123, U1 TPS5450DDAR, U2 TPS5450DDAR, U3 LMS8117AMP-3.3

Commit message: added QFN PIC
Parts:
- removed IC1: PIC24FJ64GB202, microchip:DIL28-3
- removed PROGRAMMING: Jtag, Mother-Board-rev5:MOTHER-BOARD-REV5_10-PIN-SMD
- added IC3: PIC18F26J53ML, microchip:QFN28-ML_6X6MM
- added J10, J11, J12, J7, J8, J9: 22-05-7028-02, Son_of_Dark_Power:7395-02
- added J13: 22-05-7048-04, Son_of_Dark_Power:7395-04
- added PROG.: (no value), con-molex:22-23-2061
- moved R19 133.4 mm to (-26.8, 58.6)
- moved R20 129.4 mm to (-30.9, 58.8)
- moved U$7 129.0 mm to (-30.7, 51.2)
- moved U$6 126.6 mm to (-20.1, 51.1)
- moved C21 120.1 mm to (-48.3, 62.0)
- moved U$5 117.8 mm to (-47.8, 55.3)
- moved LED5 116.7 mm to (-15.5, 62.3)
- moved LED6 116.7 mm to (-17.6, 62.3)
- moved R14 116.7 mm to (-50.7, 77.4)
- moved R21 116.7 mm to (-15.3, 67.5)
- moved R22 116.7 mm to (-17.6, 67.5)
- moved R23 116.7 mm to (-19.6, 67.5)
- moved LED7 116.7 mm to (-19.7, 62.3)
- moved LED8 116.7 mm to (-21.7, 62.3)
- moved LED9 116.7 mm to (-23.7, 62.3)
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Connections:
- removed net 6V_INPUT1: C28.1, J4.2, J5.2, J6.2
- removed net 6V_INPUT2: C27.1, J1.2, J2.2, J3.2
- removed net IO1: IC1.9, R19.1, U$6.P$2, U$6.P$3
- removed net IO2: IC1.2, R20.1, U$7.P$2, U$7.P$3
- removed net LOGIC_5V: C6.1, L1.2, R2.2, R4.2
- removed net VOUT_SERVOSRIGHT: C18.1, L2.2, R1.2, R6.2
- new net LVP: PROG..6
- new net N$25: IC3.8
- new net N$31: IC3.14
- new net SWITCH_1: IC3.27, R19.1, U$6.P$2, U$6.P$3
- new net SWITCH_2: IC3.6, R20.1, U$7.P$2, U$7.P$3
- new net VOUT_LOGIC: C12.1, L3.2, R10.2, R8.2
- new net VOUT_SERVORIGHT: C21'.1, C27.1, J1.2, J2.2, J3.2, L4.2, R12.2, R7.2
- net 3.3V: now also IC3.10, IC3.25, PROG..2; no longer IC1.13, IC1.28, PROGRAMMING.1, PROGRAMMING.2
- net GND: now also C21.2, C25.2, C26.2, IC3.24, IC3.5, J13.1, J13.4, LED5.C, LED6.C, LED7.C, LED8.C, LED9.C, PROG..3, R19.2, R20.2, U$5.P$1, U$5.P$4
- net IO3: now also IC3.7; no longer IC1.15
- net IO4: now also IC3.9; no longer IC1.3
- net IO5: now also IC3.11; no longer IC1.10
- net IO6: now also IC3.12; no longer IC1.14
- net IO7: now also IC3.13; no longer IC1.16
- net IO8: now also IC3.28; no longer IC1.17
- net MCLR: now also PROG..1; no longer PROGRAMMING.7, PROGRAMMING.8
- net MCLR': now also IC3.26; no longer IC1.1
- net OC1: now also IC3.23; no longer IC1.25
- net OC2: now also IC3.22; no longer IC1.26
- net OC3: now also IC3.21; no longer IC1.24
- net OC4: now also IC3.19; no longer IC1.22
- net OC5: now also IC3.18; no longer IC1.21
- net OC6: now also IC3.15; no longer IC1.18
- net PGC1: now also IC3.2, PROG..5; no longer IC1.5, PROGRAMMING.3, PROGRAMMING.4
- net PGD1: now also IC3.1, PROG..4; no longer IC1.4, PROGRAMMING.5, PROGRAMMING.6
- net SCL: now also IC3.4; no longer IC1.7
- net SDA: now also IC3.3; no longer IC1.6
- net VOUT_MOTOR: now also C18.1, J13.2, J13.3, L2.2, R1.2, R6.2; no longer C21'.1, L4.2, R12.2, R7.2
- net VOUT_SERVOLEFT: now also C28.1, C6.1, J4.2, J5.2, J6.2, L1.2, R2.2, R4.2; no longer C12.1, L3.2, R10.2, R8.2
- net VSS: no longer C21.2, C25.2, C26.2, IC1.27, IC1.8, LED5.C, LED6.C, LED7.C, LED8.C, LED9.C, PROGRAMMING.10, PROGRAMMING.9, R19.2, R20.2, U$5.P$1, U$5.P$4
Routing:
- net 3.3V: track 223.9 -> 0.00 mm, vias 1 -> 0
- net MCLR: track 77.7 -> 0.00 mm, vias 2 -> 0
- net IO2: track 75.8 -> 0.00 mm, vias 2 -> 0
- net IO1: track 67.8 -> 0.00 mm, vias 3 -> 0
- net VOUT_MOTOR: track 42.3 -> 0.00 mm, vias 3 -> 0
- net VOUT_SERVOLEFT: track 42.3 -> 0.00 mm, vias 3 -> 0
- net OC2: track 41.7 -> 0.00 mm, vias 1 -> 0
- net OC6: track 40.2 -> 0.00 mm, vias 1 -> 0
- net 6V_INPUT1: track 39.7 -> 0.00 mm
- net OC5: track 39.2 -> 0.00 mm, vias 1 -> 0
- net OC1: track 38.5 -> 0.00 mm, vias 1 -> 0
- net VOUT_SERVOSRIGHT: track 36.7 -> 0.00 mm, vias 3 -> 0
- net OC4: track 36.5 -> 0.00 mm, vias 1 -> 0
- net OC3: track 35.5 -> 0.00 mm, vias 1 -> 0
- net IO4: track 33.9 -> 0.00 mm, vias 1 -> 0
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- added copper zone on layer 1, net VOUT_SERVORIGHT
- removed copper zone on layer 1, net 6V_INPUT1
- removed copper zone on layer 1, net 6V_INPUT2
- removed copper zone on layer 1, net LOGIC_5V
- removed copper zone on layer 1, net N$11
- removed copper zone on layer 1, net VOUT_SERVOSRIGHT
- removed copper zone on layer 1, net VSS
- removed copper zone on layer 16, net VSS
Other:
- board outline added: 100 x 100 mm

Commit message: last commit of rev 1
Parts:
- added IC1: PIC18F26J53ML, microchip:QFN28-ML_6X6MM
- added IC2: (no value), ic-package:DIL16
- moved J10 133.5 mm to (5.11, 21.6), turned to 270 degrees
- moved J9 126.1 mm to (4.98, 27.7), turned to 270 degrees
- moved J8 119.2 mm to (4.93, 33.5), turned to 270 degrees
- moved U$5 109.7 mm to (57.0, 87.6)
- moved J11 106.9 mm to (5.19, 16.0), turned to 270 degrees
- moved U$7 102.6 mm to (65.3, 87.5)
- moved U$6 100.6 mm to (73.6, 87.5)
- moved J7 30.3 mm to (21.7, 94.8)
- moved J12 16.7 mm to (27.5, 94.8)
- moved D5 10.5 mm to (47.2, 56.1)
- moved D6 10.5 mm to (46.9, 74.1)
- moved IC3 10.5 mm to (64.7, 65.5)
- moved R16 10.5 mm to (51.5, 72.5)
- moved C23 10.5 mm to (47.0, 70.9)
- moved C24 10.5 mm to (47.3, 59.7)
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Connections:
- new net 1,2EN: IC2.1
- new net 1A: IC2.2
- new net 1Y: IC2.3
- new net 2A: IC2.7
- new net 2Y: IC2.6
- new net 3,4EN: IC2.9
- new net 3A: IC2.10
- new net 3Y: IC2.11
- new net 4A: IC2.15
- new net 4Y: IC2.14
- new net IO3(1): IC1.7
- new net IO5(1): IC1.11
- new net IO7(1): IC1.13
- new net IO8(1): IC1.28
- new net MCLR'(1): IC1.26
- new net N$19: IC2.8
- new net N$20: IC2.16
- new net OC4(1): IC1.19
- new net OC5(1): IC1.18
- new net OC6(1): IC1.15
- new net PGC1(1): IC1.2
- new net PGD1(1): IC1.1
- net 3.3V: now also IC1.10, IC1.25
- net GND: now also IC1.24, IC1.5, IC2.12, IC2.13, IC2.4, IC2.5
- net IO4: now also IC1.9
- net IO6: now also IC1.12
- net N$25: now also IC1.8
- net N$31: now also IC1.14
- net OC1: now also IC1.23
- net OC2: now also IC1.22
- net OC3: now also IC1.21
- net SCL: now also IC1.4
- net SDA: now also IC1.3
Other:
- board text removed: "Servo 1"
- board text removed: "Servo 6"
