File: designs/Motherboard/MotherboardRev1.sch (EAGLE design)
At the start: 94 parts, among them IC1 PIC24FJ64GB202, J1 Servo 2, J2 Servo 1, J3 Servo 3, J4 Servo 4, J5 Servo 5, J6 Servo 6, Q1 BSS123, Q2 BSS123, Q3 BSS123, Q4 BSS123, U1 TPS5450DDAR, U2 TPS5450DDAR, U3 LMS8117AMP-3.3

Commit message: added QFN PIC
Parts:
- removed IC1: PIC24FJ64GB202, microchip:ENC28J60SP
- removed PROGRAMMING: Jtag, Mother-Board-rev5:MOTHER-BOARD-REV5_PIN-CONNECTOR74089
- added IC3: PIC18F26J53ML, microchip:PIC18F26J53ML
- added J10, J11, J12, J7, J8, J9: 22-05-7028-02, Son_of_Dark_Power:22-05-7028-02
- added J13: 22-05-7048-04, Son_of_Dark_Power:22-05-7048-04
- added PROG.: (no value), con-molex:22-23-2061
Connections:
- removed net 6V_INPUT1: C28.1, J4-2.S, J5-2.S, J6-2.S
- removed net 6V_INPUT2: C27.1, J1-2.S, J2-2.S, J3-2.S
- removed net IO1: IC1.!CS, R19.1, U$6.P2, U$6.P3
- removed net IO2: IC1.VSS, R20.1, U$7.P2, U$7.P3
- removed net LOGIC_5V: C6.+, L1.2, R2.2, R4.2
- removed net VOUT_SERVOSRIGHT: C18.+, L2.2, R1.2, R6.2
- new net LVP: PROG.-6.S
- new net N$25: IC3.RC0/T1OSO/T1CKI/RP11
- new net N$31: IC3.RC6/CCP9/TX1/CK1/RP17
- new net SWITCH_1: IC3.RA0/AN0/C1INA/ULPWU/RP0, R19.1, U$6.P2, U$6.P3
- new net SWITCH_2: IC3.OSC1/CLKI/RA7, R20.1, U$7.P2, U$7.P3
- new net VOUT_LOGIC: C12.+, L3.2, R10.2, R8.2
- new net VOUT_SERVORIGHT: C21'.+, C27.1, J1-2.S, J2-2.S, J3-2.S, L4.2, R12.2, R7.2
- net 3.3V: now also IC3.RB7/CCP7/KBI3/PGD/RP10, IC3.RC2/AN11/C2IND/CTPLS/RP13, PROG.-2.S; no longer IC1.TPIN+, IC1.VDD, PROGRAMMING.P$1, PROGRAMMING.P$2
- net GND: now also C21.2, C25.2, C26.2, IC3.RB6/CCP6/KBI2/PGC/RP9, IC3.VSS1, J13-1.S, J13-4.S, LED5.C, LED6.C, LED7.C, LED8.C, LED9.C, PROG.-3.S, R19.2, R20.2, U$5.P1, U$5.P4
- net IO3: now also IC3.OSC2/CLKO/RA6; no longer IC1.VDDTX
- net IO4: now also IC3.RC1/CCP8/T1OSI/!UOE!/RP12; no longer IC1.CLKOUT
- net IO5: now also IC3.VUSB; no longer IC1.!RESET
- net IO6: now also IC3.RC4/D-/VM; no longer IC1.RBIAS
- net IO7: now also IC3.RC5/D+/VP; no longer IC1.TPOUT-
- net IO8: now also IC3.RA1/AN1/C2INA/VBG/RP1; no longer IC1.TPOUT+
- net MCLR: now also PROG.-1.S; no longer PROGRAMMING.P$7, PROGRAMMING.P$8
- net MCLR': now also IC3.!MCLR; no longer IC1.VCAP
- net OC1: now also IC3.RB5/CCP5/KBI1/SDI1/SDA1/RP8; no longer IC1.VDDOSC
- net OC2: now also IC3.RB4/CCP4/KBI0/SCK1/SCL1/RP7; no longer IC1.LEDB
- net OC3: now also IC3.RB3/AN9/C3INA/CTED2/VPO/RP6; no longer IC1.OSC2
- net OC4: now also IC3.RB1/AN10/C3INC/RTCC/RP4; no longer IC1.VSSOSC
- net OC5: now also IC3.RB0/AN12/C3IND/INT0/RP3; no longer IC1.VSSPLL
- net OC6: now also IC3.RC7/CCP10/RX1/DT1/SDO1/RP18; no longer IC1.VSSTX
- net PGC1: now also IC3.RA3/AN3/C1INB/VREF+, PROG.-5.S; no longer IC1.NC*, PROGRAMMING.P$3, PROGRAMMING.P$4
- net PGD1: now also IC3.RA2/AN2/C2INB/C1IND/C3INB/VREF-/CVREF, PROG.-4.S; no longer IC1.!INT, PROGRAMMING.P$5, PROGRAMMING.P$6
- net SCL: now also IC3.RA5/AN4/C1INC/!SS1!/HLVDIN/RCV/RP2; no longer IC1.SI
- net SDA: now also IC3.VDDCORE/VCAP; no longer IC1.SO
- net VOUT_MOTOR: now also C18.+, J13-2.S, J13-3.S, L2.2, R1.2, R6.2; no longer C21'.+, L4.2, R12.2, R7.2
- net VOUT_SERVOLEFT: now also C28.1, C6.+, J4-2.S, J5-2.S, J6-2.S, L1.2, R2.2, R4.2; no longer C12.+, L3.2, R10.2, R8.2
- net VSS: no longer C21.2, C25.2, C26.2, IC1.LEDA, IC1.SCK, LED5.C, LED6.C, LED7.C, LED8.C, LED9.C, PROGRAMMING.P$10, PROGRAMMING.P$9, R19.2, R20.2, U$5.P1, U$5.P4

Commit message: last commit of rev 1
Parts:
- added IC1: PIC18F26J53ML, microchip:PIC18F26J53ML
- added IC2: (no value), ic-package:DIL16
Connections:
- new net 1,2EN: IC2.1
- new net 1A: IC2.2
- new net 1Y: IC2.3
- new net 2A: IC2.7
- new net 2Y: IC2.6
- new net 3,4EN: IC2.9
- new net 3A: IC2.10
- new net 3Y: IC2.11
- new net 4A: IC2.15
- new net 4Y: IC2.14
- new net IO3(1): IC1.OSC2/CLKO/RA6
- new net IO5(1): IC1.VUSB
- new net IO7(1): IC1.RC5/D+/VP
- new net IO8(1): IC1.RA1/AN1/C2INA/VBG/RP1
- new net MCLR'(1): IC1.!MCLR
- new net N$19: IC2.8
- new net N$20: IC2.16
- new net OC4(1): IC1.RB1/AN10/C3INC/RTCC/RP4
- new net OC5(1): IC1.RB0/AN12/C3IND/INT0/RP3
- new net OC6(1): IC1.RC7/CCP10/RX1/DT1/SDO1/RP18
- new net PGC1(1): IC1.RA3/AN3/C1INB/VREF+
- new net PGD1(1): IC1.RA2/AN2/C2INB/C1IND/C3INB/VREF-/CVREF
- net 3.3V: now also IC1.RB7/CCP7/KBI3/PGD/RP10, IC1.RC2/AN11/C2IND/CTPLS/RP13
- net GND: now also IC1.RB6/CCP6/KBI2/PGC/RP9, IC1.VSS1, IC2.12, IC2.13, IC2.4, IC2.5
- net IO4: now also IC1.RC1/CCP8/T1OSI/!UOE!/RP12
- net IO6: now also IC1.RC4/D-/VM
- net N$25: now also IC1.RC0/T1OSO/T1CKI/RP11
- net N$31: now also IC1.RC6/CCP9/TX1/CK1/RP17
- net OC1: now also IC1.RB5/CCP5/KBI1/SDI1/SDA1/RP8
- net OC2: now also IC1.RB4/CCP4/KBI0/SCK1/SCL1/RP7
- net OC3: now also IC1.RB3/AN9/C3INA/CTED2/VPO/RP6
- net SCL: now also IC1.RA5/AN4/C1INC/!SS1!/HLVDIN/RCV/RP2
- net SDA: now also IC1.VDDCORE/VCAP
Other:
- moved on the sheet: C23, C24, D5, D6, R15, R16, U3
