File: designs/Motherboard/Motor-Board/Motor-Board.sch (EAGLE design)
At the start: 71 parts, among them IC1 DRV8814, IC2 DRV8814, IC3 PIC24FJ64GA004, J1 22-05-7028-02, J13 22-05-7048-04, J2 22-05-7028-02, J3 22-05-7048-04, J7 22-05-7028-02, J8 22-05-7028-02, U1 DRV8811PWP, U2 DRV8811PWP

Commit message: Done with left side of mother board
Parts:
- removed IC3: PIC24FJ64GA004, microchip:PIC24FJ64GA004
- added C33: 10uF, rcl:C-USC0805
- added C34, C37, C38, C39: 4.7uF, 5v:GRM31CR71H475KA12L
- added C35: 10nF, 5v:C0805C103K5RACTU
- added C36: 330uF, 5v:10SVP330MX
- added C40: .1uF, rcl:C-USC0402
- added C41, C42: 0.47uF, rcl:C-USC0402
- added D2: PDS760-13, 5v:PDS760-13
- added IC4: PIC24FJ256GB106, microchip:PIC24FJ256GB106
- added L1: (no value), WE-HCC:WE-HCC-7443331000_1090
- added LED4, POWER_ON: (no value), led:LEDCHIP-LED0603
- added MOTIN1, MOTIN2, MOTIN3, MOTIN4: 22-05-7048-04, Son_of_Dark_Power:22-05-7048-04
- added PROGRAMMING: Jtag, Mother-Board-rev5:MOTHER-BOARD-REV5_PIN-CONNECTOR74089
- added PWR_IN(2): (no value), Son_of_Dark_Powersch:555X-2H
- added R27, R29, R31, R32, R33, R34: 10k, rcl:R-US_R0402
- added R28: (no value), rcl:R-US_R0402
- added R30: 100, rcl:R-US_R0402
- added SERVO_1, SERVO_2, SERVO_3: 22-05-7038-03, con-molex:22-05-7038-03
- added TP1, TP2: PTR1B1,27, testpad:PTR1B1,27
- added U$2: TPS5450DDAR, 5v:TPS5450DDAR
- added U$5: Switch3, Parts4Class:MC32882_SW
- C1, C23, C24, C25, C26, C3: value (none) -> 0.01uF
- C10, C14, C15, C16, C8, C9: value (none) -> 0.22uF
- C11, C12, C5, C6: value (none) -> 1nF
- C13: value (none) -> .1uF
- C17, C18, C19, C2, C20, C21, C22, C28, C29, C4, C7: value (none) -> 0.1uF
- C27: value (none) -> 1uF
- R1, R6: value (none) -> 1M
- R10, R5: value (none) -> 30k
- R11, R12, R19, R20: value (none) -> 0.1
- R13, R14, R21, R22: value (none) -> 47k
- R15, R16, R17, R18, R23, R24, R25, R26, R4, R9: value (none) -> 10k
- R2, R3, R7, R8: value (none) -> 0.2
- renumbered J1 to MOTOR4, J13 to STEP2, J2 to MOTOR3, J3 to STEP1, J7 to MOTOR2, J8 to MOTOR1
Connections:
- removed net M1-NFAULT: IC1.NFAULT
- removed net M2-NFAULT: IC2.NFAULT
- removed net MCLR: IC3.!MCLR
- removed net PGC1: IC3.RB1
- removed net PGD1: IC3.RB0
- new net BOOT_VM: C35.1, U$2.BOOT
- new net CHANNEL_A_1: IC4.RG6, MOTIN1-4.S
- new net CHANNEL_A_2: IC4.RB9, MOTIN2-3.S
- new net CHANNEL_A_3: IC4.RB7, MOTIN3-3.S
- new net CHANNEL_A_4: IC4.RG9, MOTIN4-3.S
- new net CHANNEL_B_1: IC4.RG7, MOTIN1-3.S
- new net CHANNEL_B_2: IC4.RB8, MOTIN2-4.S
- new net CHANNEL_B_3: IC4.RB6, MOTIN3-4.S
- new net CHANNEL_B_4: IC4.RG8, MOTIN4-4.S
- new net M_MCLR: C40.1, PROGRAMMING.P$7, PROGRAMMING.P$8, R30.2, R31.1, U$5.P2, U$5.P3
- new net M_MCLR': IC4.!MCLR, R30.1
- new net M_PGC1: IC4.RB1, PROGRAMMING.P$3, PROGRAMMING.P$4
- new net M_PGD1: IC4.RB0, PROGRAMMING.P$5, PROGRAMMING.P$6
- new net N$25: LED4.A, R29.1
- new net N$29: C41.1, IC1.V3V3OUT, R32.2, R4.2
- new net N$31: IC1.NFAULT, R32.1
- new net N$35: IC2.NFAULT, R33.1
- new net N$37: C42.1, IC2.V3V3OUT, R33.2, R9.2
- new net N$38: POWER_ON.A, R34.1
- new net OC1: IC4.RF3, SERVO_1-1.S
- new net OC2: IC4.RF5, SERVO_2-1.S
- new net OC3: IC4.RF4, SERVO_3-1.S
- new net PH_VM: C35.2, D2.K, L1.1, U$2.PH
- new net VCC: C34.2, C37.2, C38.2, C39.2, PWR_IN(2)-2.S, R34.2, U$2.VIN
- new net VSNS_VM: R27.1, R28.2, U$2.VSNS
- net +3V3: now also IC4.VDD@1, IC4.VDD@2, IC4.VDD@3, PROGRAMMING.P$1, PROGRAMMING.P$2, R31.2; no longer IC1.V3V3OUT, IC2.V3V3OUT, IC3.AVDD, IC3.VDD@1, IC3.VDD@2, R4.2, R9.2
- net +7V: now also C33.1, C36.+, H2.MOUNT, L1.2, MOTIN1-2.S, MOTIN2-2.S, MOTIN3-2.S, MOTIN4-2.S, R27.2, R29.2, SERVO_1-2.S, SERVO_2-2.S, SERVO_3-2.S
- net GND: now also C33.2, C34.1, C36.-, C37.1, C38.1, C39.1, C40.2, C41.2, C42.2, D2.A_2, IC4.VSS@1, IC4.VSS@2, IC4.VSS@3, LED4.C, MOTIN1-1.S, MOTIN2-1.S, MOTIN3-1.S, MOTIN4-1.S, POWER_ON.C, PROGRAMMING.P$10, PROGRAMMING.P$9, PWR_IN(2)-1.S, R28.1, SERVO_1-3.S, SERVO_2-3.S, SERVO_3-3.S, U$2.GND_2, U$2.PWPD, U$5.P1, U$5.P4; no longer IC3.AVSS, IC3.VSS@1, IC3.VSS@2
- net M-DECAY: now also IC4.RD1; no longer IC3.TCK
- net M-I0: now also IC4.RD10; no longer IC3.RC8
- net M-I1: now also IC4.RC15; no longer IC3.RC7
- net M-NSLEEP: now also IC4.RF0; no longer IC3.RB14
- net M-RESET: now also IC4.RE0; no longer IC3.RB15
- net M1-AENBL: now also IC4.RC13; no longer IC3.RB11
- net M1-APHASE: now also IC4.RC14; no longer IC3.RB13
- net M1-BENBL: now also IC4.RD0; no longer IC3.RB10
- net M1-BHPASE: now also IC4.RD11; no longer IC3.RC9
- net M2-AENBL: now also IC4.RC12; no longer IC3.RB9
- net M2-APHASE: now also IC4.RD9; no longer IC3.RC6
- net M2-BENBL: now also IC4.RG2; no longer IC3.RB8
- net M2-BHPASE: now also IC4.RD8; no longer IC3.RB7
- net S-SRN: now also IC4.RF1; no longer IC3.TDO
- net S1-DIR: now also IC4.RE4; no longer IC3.RB6
- net S1-ENABLEN: now also IC4.RD7; no longer IC3.TDI
- net S1-HOME: now also IC4.RE3; no longer IC3.RB5
- net S1-STEP: now also IC4.RD5; no longer IC3.RC3
- net S2-DIR: now also IC4.RD6; no longer IC3.RA2
- net S2-ENABLEN: now also IC4.RD3; no longer IC3.RC2
- net S2-HOME: now also IC4.RD4; no longer IC3.RA3
- net S2-STEP: now also IC4.RD2; no longer IC3.RC1
- net SCL: now also IC4.RE6, TP1.TP; no longer IC3.RB3
- net SDA: now also IC4.RE7, TP2.TP; no longer IC3.RB2
- net USM0: now also IC4.RE2; no longer IC3.RC5
- net USM1: now also IC4.RE1; no longer IC3.RC4
