File: designs/Motherboard/Motor-Board/Motor-Board.sch (EAGLE design)
At the start: 106 parts, among them IC1 DRV8814, IC2 DRV8814, IC4 PIC24FJ256GB106, U1 DRV8811PWP, U2 DRV8811PWP

Commit message: Motor board
Parts:
- removed C33: 10uF, rcl:C-USC0805
- removed C34, C37, C38, C39: 4.7uF, 5v:GRM31CR71H475KA12L
- removed C40: .1uF, rcl:C-USC0402
- removed MOTOR4: 22-05-7028-02, Son_of_Dark_Power:22-05-7028-02
- removed R30: 100, rcl:R-US_R0402
- removed R31: 10k, rcl:R-US_R0402
- added C100, C105: 0.01uF, rcl:C-USC0402
- added C101, C106, C132, C137: 0.1uF, rcl:C-USC0402
- added C117: 4.7uF, rcl:C-USC0805
- added C120, C129, C131: 1nF, rcl:C-USC0402
- added C123, C124, C125: 0.22uF, rcl:C-USC0402
- added C128: 10uF, rcl:C-USC0402
- added IC101: DRV8814, Motor-Board:DRV8818PWPR
- added MOTOR101: 22-05-7028-02, Son_of_Dark_Power:22-05-7028-02
- added R106: 1M, rcl:R-US_R0402
- added R108: 0.2, rcl:R-US_R0402
- C1: value 0.01uF -> .1uF
- C10, C8, C9: value 0.22uF -> 4.7uF; device rcl:C-USC0402 -> rcl:C-USC0805
- C11: value 1nF -> 10uF; device rcl:C-USC0402 -> rcl:C-USC0805
- C138: value 1uF -> .1uF
- C2: value 0.1uF -> 10uF
- C3: value 0.01uF -> 0.1uF
- C5, C6: value 1nF -> 0.1uF
- IC1: value DRV8814 -> MCP1703CB; device Motor-Board:DRV8818PWPR -> linear:MCP1703CB
- R1: value 1M -> 10k
- R2: value 0.2 -> 100
- renumbered C12 to C119, C13 to C121, C14 to C114, C15 to C112, C16 to C113, C17 to C111, C18 to C115, C19 to C127, C20 to C126, C21 to C130, C22 to C118, C23 to C107, C24 to C108, C25 to C103, C26 to C102, C27 to C138, C28 to C134, C29 to C135, C30 to C122, C31 to C136, C32 to C110, C35 to C116, C36 to C133, C41 to C109, C42 to C104, D2 to D100, IC2 to IC100, IC4 to IC102, L1 to L100, LED4 to LED100, MOTIN1 to MOTIN100, MOTIN2 to MOTIN103, MOTIN3 to MOTIN101, MOTIN4 to MOTIN102, MOTOR3 to MOTOR100, R10 to R105, R11 to R123, R12 to R125, R13 to R124, R14 to R128, R15 to R127, R16 to R130, R17 to R129, R18 to R126, R19 to R115, R20 to R120, R21 to R116, R22 to R117, R23 to R119, R24 to R122, R25 to R121, R26 to R118, R27 to R113, R28 to R114, R29 to R131, R3 to R109, R32 to R110, R33 to R104, R34 to R101, R4 to R112, R5 to R111, R6 to R100, R7 to R102, R8 to R103, R9 to R107, SERVO_1 to SERVO_102, SERVO_2 to SERVO_101, SERVO_3 to SERVO_100, TP1 to SCL, TP2 to SDA, U$2 to U$101, U$5 to U$100, U1 to U101, U2 to U100
Connections:
- new net N$39: C128.1, IC102.VDDCORE
- net +3V3: now also C137.1, C2.1, C3.1, C5.1, C6.1, C7.1, IC1.VO, IC102.AVDD, IC102.VUSB, R1.2; no longer R31.2
- net +7V: now also C101.2, C106.2, C11.1, C125.1, C4.1, IC1.VI, IC101.VMA, IC101.VMB, R106.2; no longer C10.1, C2.2, C33.1, C4.2, H2.MOUNT, IC1.VMA, IC1.VMB, R1.2
- net GND: now also C1.2, C10.1, C117.1, C120.2, C123.2, C128.2, C129.2, C131.2, C132.2, C137.2, C2.2, C3.2, C4.2, C8.1, C9.1, IC101.GND, IC102.AVSS, IC102.ENVREG, R108.2; no longer C33.2, C34.1, C37.1, C38.1, C39.1, C40.2, C9.2, R2.2
- net M-DECAY: now also IC101.DECAY; no longer IC1.DECAY
- net M-I0: now also IC101.AI0, IC101.BI0; no longer IC1.AI0, IC1.BI0
- net M-I1: now also IC101.AI1, IC101.BI1; no longer IC1.AI1, IC1.BI1
- net M-NSLEEP: now also IC101.NSLEEP; no longer IC1.NSLEEP
- net M-RESET: now also IC101.NRESET; no longer IC1.NRESET
- net M1-AENBL: now also IC101.AENBL; no longer IC1.AENBL
- net M1-APHASE: now also IC101.APHASE; no longer IC1.APHASE
- net M1-BENBL: now also IC101.BENBL; no longer IC1.BENBL
- net M1-BHPASE: now also IC101.BHPASE; no longer IC1.BHPASE
- net M1-MAOUT1: now also IC101.AOUT1, MOTOR1-1.S; no longer IC1.AOUT1, MOTOR2-1.S
- net M1-MAOUT2: now also IC101.AOUT2, MOTOR1-2.S; no longer IC1.AOUT2, MOTOR2-2.S
- net M1-MBOUT1: now also IC101.BOUT1, MOTOR101-1.S; no longer IC1.BOUT1, MOTOR1-1.S
- net M1-MBOUT2: now also IC101.BOUT2, MOTOR101-2.S; no longer IC1.BOUT2, MOTOR1-2.S
- net M2-MAOUT1: now also MOTOR2-1.S; no longer MOTOR4-1.S
- net M2-MAOUT2: now also MOTOR2-2.S; no longer MOTOR4-2.S
- net M_MCLR: now also C1.1, R1.1, R2.2; no longer C40.1, R30.2, R31.1
- net M_MCLR': now also R2.1; no longer R30.1
- net N$1: now also C105.2, IC101.CP2; no longer C1.2, IC1.CP2
- net N$10: now also IC101.ISENB; no longer IC1.ISENB
- net N$12: now also IC101.AVREV, IC101.BVREF; no longer IC1.AVREV, IC1.BVREF
- net N$17: now also C120.1; no longer C11.1
- net N$18: now also C131.1; no longer C5.1
- net N$19: now also C129.1; no longer C6.1
- net N$2: now also C105.1, IC101.CP1; no longer C1.1, IC1.CP1
- net N$26: now also C132.1; no longer C7.1
- net N$29: now also IC101.V3V3OUT; no longer IC1.V3V3OUT
- net N$3: now also C106.1, IC101.VCP, R106.1; no longer C2.1, IC1.VCP, R1.1
- net N$31: now also IC101.NFAULT; no longer IC1.NFAULT
- net N$32: now also C124.1; no longer C8.1
- net N$33: now also C124.2; no longer C8.2
- net N$34: now also C123.1; no longer C9.1
- net N$36: now also C125.2; no longer C10.2
- net N$4: now also IC101.ISENA, R108.1; no longer IC1.ISENA, R2.1
- net N$5: now also C100.2; no longer C3.2
- net N$6: now also C100.1; no longer C3.1
- net N$7: now also C101.1; no longer C4.1
- net VCC: now also C10.2, C117.2, C8.2, C9.2; no longer C34.2, C37.2, C38.2, C39.2
