File: designs/Motherboard/MotherboardRev2/MotherboardRev2.sch (EAGLE design)
At the start: 102 parts, among them IC1 PIC24FJ64GB202, IC2 PIC18F26J53SO, J1 Servo 2, J2 Servo 1, J3 Servo 3, J4 Servo 4, J5 Servo 5, J6 Servo 6, Q1 BSS123, Q2 BSS123, Q3 BSS123, Q4 BSS123, U3 LMS8117AMP-3.3

Commit message: More work done on motherboard
Parts:
- removed IC2: PIC18F26J53SO, microchip:PIC18F26J53SO
- removed J1: Servo 2, con-molex:22-05-7038-03
- removed J2: Servo 1, con-molex:22-05-7038-03
- removed J3: Servo 3, con-molex:22-05-7038-03
- removed J4: Servo 4, con-molex:22-05-7038-03
- removed J5: Servo 5, con-molex:22-05-7038-03
- removed J6: Servo 6, con-molex:22-05-7038-03
- added 3.3V, 3.3V(2), 5V, 5V(2): 22-05-7028-02, Son_of_Dark_Powersch:22-05-7028-02
- added C33: 10uF, rcl:C-USC0805
- added C34, C35, C36: .1uF, rcl:C-USC0805
- added C37: .1uF, 3-3_fixed:C3216X5R1A106K
- added C38: 10uF, SparkFun-Capacitors:10UF-16V-10%(TANT)
- added D7: 3_3V_PWR, SparkFun-LED:LED-FKIT-1206
- added D8: 6V_Pwr, SparkFun-LED:LED-FKIT-1206
- added IC3: PIC24FJ64GB202, microchip:PIC18F26J53ML
- added LED10, LED11, LED12: (no value), motherboard_i_autoroute:LED_LEDCHIPLED_1206
- added MOTOR_PWR: 22-05-7048-04, Son_of_Dark_Powersch:22-05-7048-04
- added PWR_IN, PWR_IN(2): (no value), Son_of_Dark_Powersch:555X-2H
- added R18: 470, rcl:R-US_R0805
- added R26: 10k, rcl:R-US_R0805
- added R27, R28: 4.7k, rcl:R-US_R0805
- added R29, R30, R31: (no value), rcl:R-US_M0805
- added R32: 0 ohm, rcl:R-US_R1206
- added R33: 4.7K, rcl:R-US_R0805
- added R34, R35: (no value), rcl:R-US_R0805W
- added SERVO_1, SERVO_10, SERVO_2, SERVO_3, SERVO_4, SERVO_5, SERVO_6, SERVO_7, SERVO_8, SERVO_9: 22-05-7038-03, con-molex:22-05-7038-03
- added START_SWITCH: (no value), con-lstb:MA03-1
- added U$10: Switch3, Parts4Class:MC32882_SW
- added U$11, U$13, U$14: Switch1, Parts4Class:MC32882_SW
- added U$12: Switch2, Parts4Class:MC32882_SW
- added U1: LMS8117AMP-3.3, NSC-LMS8117AMP:LMS8117AMP-3.3
- C29: value .1uF -> 10uF; device 3-3_fixed:C3216X5R1A106K -> SparkFun-Capacitors:10UF-16V-10%(TANT)
- IC1: device microchip:ENC28J60SP -> microchip:PIC18F26J53ML
- R17: value 0 ohm -> 4.7K; device rcl:R-US_R1206 -> rcl:R-US_R0805
Connections:
- removed net 6V_INPUT1: C28.1, J4-2.S, J5-2.S, J6-2.S
- removed net 6V_INPUT2: C27.1, J1-2.S, J2-2.S, J3-2.S
- removed net BB_PWR_SW: U$3P9.PWR_BUT
- removed net IO1: IC1.!CS, R19.1, U$6.P2, U$6.P3
- removed net IO2: IC1.VSS, R20.1, U$7.P2, U$7.P3
- removed net VSS: C21.2, C23.-, C24.-, C25.2, C26.2, C27.2, C28.2, D5.C, D6.C, IC1.LEDA, IC1.SCK, J1-3.S, J2-3.S, J3-3.S, J4-3.S, J5-3.S, J6-3.S, LED5.C, LED6.C, LED7.C, LED8.C, LED9.C, PROGRAMMING.P$10, PROGRAMMING.P$9, R19.2, R20.2, U$5.P1, U$5.P4, U3.GND
- new net BB_PWR_BUTTON: U$13.P2, U$13.P3, U$1P9.PWR_BUT
- new net BB_SYS_RESET: U$14.P2, U$14.P3, U$1P9.SYS_RESET!N
- new net IO3(1): IC1.OSC2/CLKO/RA6, R29.2
- new net IO4(1): IC1.RC1/CCP8/T1OSI/!UOE!/RP12, R30.2
- new net IO5(1): IC1.VUSB, R31.2
- new net MCLR'(1): IC1.!MCLR, R18.1
- new net MCLR(1): C36.1, R18.2, R26.1, U$10.P2, U$10.P3
- new net N$15: LED10.A, R29.1
- new net N$16: LED11.A, R30.1
- new net N$17: LED12.A, R31.1
- new net N$18: C37.1, R32.1, U$1P9.VDD_5V@1, U$1P9.VDD_5V@2
- new net N$21: D8.A, R35.1
- new net N$25: IC3.RC0/T1OSO/T1CKI/RP11
- new net N$31: IC3.RC6/CCP9/TX1/CK1/RP17
- new net OC1(1): IC1.RB5/CCP5/KBI1/SDI1/SDA1/RP8, SERVO_9-1.S
- new net OC2(1): IC1.RB4/CCP4/KBI0/SCK1/SCL1/RP7, SERVO_8-1.S
- new net OC3(1): IC1.RB3/AN9/C3INA/CTED2/VPO/RP6, SERVO_10-1.S
- new net OC4(1): IC1.RB1/AN10/C3INC/RTCC/RP4, SERVO_7-1.S
- new net START_LEFT: START_SWITCH.3, U$1P9.GPIO_60
- new net START_RIGHT: START_SWITCH.1, U$1P9.GPIO_30
- new net SWITCH_1: IC3.RA0/AN0/C1INA/ULPWU/RP0, R19.1, U$6.P2, U$6.P3
- new net SWITCH_2: IC3.OSC1/CLKI/RA7, R20.1, U$7.P2, U$7.P3
- new net SWITCH_3: IC1.OSC1/CLKI/RA7, R27.1, U$11.P2, U$11.P3
- new net SWITCH_4: IC1.RA0/AN0/C1INA/ULPWU/RP0, R28.1, U$12.P2, U$12.P3
- new net VOUT5: 3.3V(2)-1.S, 3.3V-1.S, C38.+, R34.1, U1.VOUT
- net +5V: now also R32.2; no longer C23.+, R16.2, R17.2, U3.IN
- net 3.3V: now also C34.1, C35.1, IC1.RB7/CCP7/KBI3/PGD/RP10, IC1.RC2/AN11/C2IND/CTPLS/RP13, IC3.RB7/CCP7/KBI3/PGD/RP10, IC3.RC2/AN11/C2IND/CTPLS/RP13, R17.2, R26.2, R33.2, START_SWITCH.2, U$11.P1, U$11.P4, U$12.P1, U$12.P4; no longer IC1.TPIN+, IC1.VDD
- net GND: now also 3.3V(2)-2.S, 3.3V-2.S, 5V(2)-2.S, 5V-2.S, C21.2, C23.-, C24.-, C25.2, C26.2, C27.2, C28.2, C29.-, C33.2, C34.2, C35.2, C36.2, C37.2, C38.-, D5.C, D6.C, D7.C, D8.C, IC1.RB6/CCP6/KBI2/PGC/RP9, IC1.VSS1, IC3.RB6/CCP6/KBI2/PGC/RP9, IC3.VSS1, LED10.C, LED11.C, LED12.C, LED5.C, LED6.C, LED7.C, LED8.C, LED9.C, MOTOR_PWR-1.S, MOTOR_PWR-4.S, PROGRAMMING.P$10, PROGRAMMING.P$9, PWR_IN(2)-1.S, PWR_IN-1.S, R19.2, R20.2, R27.2, R28.2, SERVO_1-3.S, SERVO_10-3.S, SERVO_2-3.S, SERVO_3-3.S, SERVO_4-3.S, SERVO_5-3.S, SERVO_6-3.S, SERVO_7-3.S, SERVO_8-3.S, SERVO_9-3.S, U$10.P1, U$10.P4, U$13.P1, U$13.P4, U$14.P1, U$14.P4, U$5.P1, U$5.P4, U1.GND, U3.GND; no longer C29.2
- net IO3: now also IC3.OSC2/CLKO/RA6; no longer IC1.VDDTX
- net IO4: now also IC3.RC1/CCP8/T1OSI/!UOE!/RP12; no longer IC1.CLKOUT
- net IO5: now also IC3.VUSB; no longer IC1.!RESET
- net IO6: now also IC3.RC4/D-/VM; no longer IC1.RBIAS
- net IO7: now also IC3.RC5/D+/VP; no longer IC1.TPOUT-
- net IO8: now also IC1.RA1/AN1/C2INA/VBG/RP1, IC3.RA1/AN1/C2INA/VBG/RP1; no longer IC1.TPOUT+
- net MCLR': now also IC3.!MCLR
- net N$11: now also D7.A, R34.2; no longer C29.1, R17.1, U$3P9.VDD_5V@1, U$3P9.VDD_5V@2
- net OC1: now also IC3.RB5/CCP5/KBI1/SDI1/SDA1/RP8, SERVO_1-1.S; no longer IC1.VDDOSC, J2-1.S
- net OC2: now also IC3.RB4/CCP4/KBI0/SCK1/SCL1/RP7, SERVO_2-1.S; no longer IC1.LEDB, J1-1.S
- net OC3: now also IC3.RB3/AN9/C3INA/CTED2/VPO/RP6, SERVO_3-1.S; no longer IC1.OSC2, J3-1.S
- net OC4: now also IC3.RB1/AN10/C3INC/RTCC/RP4, SERVO_4-1.S; no longer IC1.VSSOSC, J4-1.S
- net OC5: now also IC3.RB0/AN12/C3IND/INT0/RP3, SERVO_5-1.S; no longer IC1.VSSPLL, J5-1.S
- net OC6: now also IC3.RC7/CCP10/RX1/DT1/SDO1/RP18, SERVO_6-1.S; no longer IC1.VSSTX, J6-1.S
- net PGC1: now also IC1.RA3/AN3/C1INB/VREF+, IC3.RA3/AN3/C1INB/VREF+; no longer IC1.NC*
- net PGD1: now also IC1.RA2/AN2/C2INB/C1IND/C3INB/VREF-/CVREF, IC3.RA2/AN2/C2INB/C1IND/C3INB/VREF-/CVREF; no longer IC1.!INT
- net SCL: now also IC1.RA5/AN4/C1INC/!SS1!/HLVDIN/RCV/RP2, IC3.RA5/AN4/C1INC/!SS1!/HLVDIN/RCV/RP2, R33.1; no longer IC1.SI
- net SDA: now also IC1.VDDCORE/VCAP, IC3.VDDCORE/VCAP, R17.1; no longer IC1.SO
- net VCC: now also PWR_IN(2)-2.S, PWR_IN-2.S
- net VOUT1: now also 5V(2)-1.S, 5V-1.S, C23.+, C29.+, R16.2, R35.2, U1.IN, U3.IN
- net VOUT2: now also C27.1, SERVO_1-2.S, SERVO_2-2.S, SERVO_3-2.S, SERVO_7-2.S
- net VOUT3: now also C28.1, C33.1, SERVO_10-2.S, SERVO_4-2.S, SERVO_5-2.S, SERVO_6-2.S, SERVO_8-2.S, SERVO_9-2.S
- net VOUT4: now also MOTOR_PWR-2.S, MOTOR_PWR-3.S
Other:
- note added: "LDO for 3.3V output"
- note added: "LDO for on board 3.3V"
- note added: "Regulator for 5 Volt Output"
- note added: "Regulator for Left Servo Line ~ 6V"
- note added: "Regulator for Motor Power ~ 6 Volt"
- note added: "Regulator for Right Servo Line ~ 6V"

Commit message: Running traces on motherboard
Connections:
- removed net +5V: R32.2
- net VOUT1: now also R32.2
- net VOUT2: now also C28.1, SERVO_4-2.S, SERVO_5-2.S; no longer SERVO_7-2.S
- net VOUT3: now also SERVO_7-2.S; no longer C28.1, SERVO_4-2.S, SERVO_5-2.S
Changed lines of the file:
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@@
 </variantdefs>
 <classes>
-<class number="0" name="default" width="0.2032" drill="0.508">
+<class number="0" name="default" width="0.2032" drill="0.3302">
 <clearance class="0" value="0.254"/>
 </class>
@@
 </segment>
 </net>
-<net name="+5V" class="0">
+<net name="VOUT1" class="0">
 <segment>
 <pinref part="R32" gate="G$1" pin="2"/>
@@
 </segment>
 <segment>
-<wire x1="231.14" y1="111.76" x2="231.14" y2="93.98" width="0.1524" layer="91"/>
-<pinref part="SERVO_7" gate="-2" pin="S"/>
-<wire x1="238.76" y1="93.98" x2="231.14" y2="93.98" width="0.1524" layer="91"/>
-<label x="233.68" y="109.22" size="1.778" layer="95"/>
-</segment>
-</net>
-<net name="VOUT3" class="0">
-<segment>
 <wire x1="139.7" y1="142.24" x2="139.7" y2="124.46" width="0.1524" layer="91"/>
 <pinref part="SERVO_4" gate="-2" pin="S"/>
@@
 <junction x="139.7" y="124.46"/>
 <label x="142.24" y="139.7" size="1.778" layer="95"/>
-<pinref part="SERVO_6" gate="-2" pin="S"/>
-<wire x1="147.32" y1="53.34" x2="139.7" y2="53.34" width="0.1524" layer="91"/>
 <wire x1="139.7" y1="124.46" x2="139.7" y2="88.9" width="0.1524" layer="91"/>
-<wire x1="139.7" y1="88.9" x2="139.7" y2="53.34" width="0.1524" layer="91"/>
 <pinref part="SERVO_5" gate="-2" pin="S"/>
 <wire x1="147.32" y1="88.9" x2="139.7" y2="88.9" width="0.1524" layer="91"/>
-<junction x="139.7" y="88.9"/>
 <pinref part="C28" gate="G$1" pin="1"/>
 <wire x1="139.7" y1="124.46" x2="127" y2="124.46" width="0.1524" layer="91"/>
 <wire x1="127" y1="124.46" x2="127" y2="116.84" width="0.1524" layer="91"/>
 </segment>
+</net>
+<net name="VOUT3" class="0">
 <segment>
 <wire x1="193.04" y1="142.24" x2="193.04" y2="124.46" width="0.1524" layer="91"/>
@@
 <wire x1="200.66" y1="53.34" x2="193.04" y2="53.34" width="0.1524" layer="91"/>
 <wire x1="193.04" y1="124.46" x2="193.04" y2="88.9" width="0.1524" layer="91"/>
-<wire x1="193.04" y1="88.9" x2="193.04" y2="53.34" width="0.1524" layer="91"/>
+<wire x1="193.04" y1="88.9" x2="193.04" y2="68.58" width="0.1524" layer="91"/>
 <pinref part="SERVO_8" gate="-2" pin="S"/>
+<wire x1="193.04" y1="68.58" x2="193.04" y2="53.34" width="0.1524" layer="91"/>
 <wire x1="200.66" y1="88.9" x2="193.04" y2="88.9" width="0.1524" layer="91"/>
 <junction x="193.04" y="88.9"/>
@@
 <wire x1="193.04" y1="124.46" x2="180.34" y2="124.46" width="0.1524" layer="91"/>
 <wire x1="180.34" y1="124.46" x2="180.34" y2="116.84" width="0.1524" layer="91"/>
-</segment>
-</net>
+<pinref part="SERVO_6" gate="-2" pin="S"/>
+<wire x1="147.32" y1="53.34" x2="139.7" y2="53.34" width="0.1524" layer="91"/>
+<wire x1="139.7" y1="53.34" x2="139.7" y2="68.58" width="0.1524" layer="91"/>
+<wire x1="139.7" y1="68.58" x2="193.04" y2="68.58" width="0.1524" layer="91"/>
+<junction x="193.04" y="68.58"/>
+</segment>
+<segment>
+<wire x1="231.14" y1="111.76" x2="231.14" y2="93.98" width="0.1524" layer="91"/>
+<pinref part="SERVO_7" gate="-2" pin="S"/>
+<wire x1="238.76" y1="93.98" x2="231.14" y2="93.98" width="0.1524" layer="91"/>
+<label x="233.68" y="109.22" size="1.778" layer="95"/>
+</segment>
+</net>

Commit message: Final Motherboard
Parts:
- removed C19, C30, C31, C32: 4.7uF, 5v:GRM31CR71H475KA12L
- removed C20: 10nF, 5v:C0805C103K5RACTU
- removed C22: 330uF, 5v:10SVP330MX
- removed C33: 10uF, rcl:C-USC0805
- removed C34, C35, C36: .1uF, rcl:C-USC0805
- removed D4: PDS760-13, 5v:PDS760-13
- removed D6, D8: 6V_Pwr, SparkFun-LED:LED-FKIT-1206
- removed IC1: PIC24FJ64GB202, microchip:PIC18F26J53ML
- removed L4: (no value), WE-HCC:WE-HCC-7443331000_1090
- removed LED10, LED11, LED12: (no value), motherboard_i_autoroute:LED_LEDCHIPLED_1206
- removed LED3: (no value), led:LEDSML1206
- removed MOTOR_PWR: 22-05-7048-04, Son_of_Dark_Powersch:22-05-7048-04
- removed PWR_IN(2): (no value), Son_of_Dark_Powersch:555X-2H
- removed Q4: BSS123, transistor-small-signal:BSS123
- removed R12: 10k, rcl:R-US_R1206
- removed R16, R35: (no value), rcl:R-US_R0805W
- removed R18: 470, rcl:R-US_R0805
- removed R26: 10k, rcl:R-US_R0805
- removed R27, R28: 4.7k, rcl:R-US_R0805
- removed R29, R30, R31: (no value), rcl:R-US_M0805
- removed SERVO_10, SERVO_7, SERVO_8, SERVO_9: 22-05-7038-03, con-molex:22-05-7038-03
- removed U$10: Switch3, Parts4Class:MC32882_SW
- removed U$11: Switch1, Parts4Class:MC32882_SW
- removed U$12: Switch2, Parts4Class:MC32882_SW
- removed U$3: BEAGLE_BONE_BLACK_CAPE, SparkFun-Boards:BEAGLE_BONE_BLACK_CAPE
- removed U$9: TPS5450DDAR, 5v:TPS5450DDAR
- added 3.3V(2)1, 3.3V1, 5V(2)1, 5V1: 22-05-7028-02, Son_of_Dark_Powersch:22-05-7028-02
- C1, C10, C11, C12, C13, C16, C17, C18, C2, C6, C7, C8: device 5v:GRM31CR71H475KA12L -> rcl:C-USC0805
- C21, C25, C26: device rcl:C-USC0805 -> rcl:C-USC0402
- C37: device 3-3_fixed:C3216X5R1A106K -> rcl:C-USC0402
- LED5, LED6, LED7, LED8, LED9: device motherboard_i_autoroute:LED_LEDCHIPLED_1206 -> led:LEDCHIPLED-0603-TTW
- R10: value 10k -> (none); device rcl:R-US_R1206 -> rcl:R-US_R0402
- R11, R32: device rcl:R-US_R1206 -> rcl:R-US_R0402
- R13, R14, R17, R19, R20, R33: device rcl:R-US_R0805 -> rcl:R-US_R0402
- R21, R22, R23, R24, R25: device rcl:R-US_M0805 -> rcl:R-US_R0402
Connections:
- removed net BOOT4: C20.1, U$9.BOOT
- removed net EN4: Q4.G
- removed net ENA_4: Q4.D, U$9.ENA
- removed net IO3(1): IC1.OSC2/CLKO/RA6, R29.2
- removed net IO4(1): IC1.RC1/CCP8/T1OSI/!UOE!/RP12, R30.2
- removed net IO5(1): IC1.VUSB, R31.2
- removed net MCLR'(1): IC1.!MCLR, R18.1
- removed net MCLR(1): C36.1, R18.2, R26.1, U$10.P2, U$10.P3
- removed net N$12: U$3P8.GPIO_66
- removed net N$13: D6.A, R16.1
- removed net N$14: U$3P8.GPIO_67
- removed net N$15: LED10.A, R29.1
- removed net N$16: LED11.A, R30.1
- removed net N$17: LED12.A, R31.1
- removed net N$21: D8.A, R35.1
- removed net N$4: LED3.A, R12.1
- removed net OC1(1): IC1.RB5/CCP5/KBI1/SDI1/SDA1/RP8, SERVO_9-1.S
- removed net OC2(1): IC1.RB4/CCP4/KBI0/SCK1/SCL1/RP7, SERVO_8-1.S
- removed net OC3(1): IC1.RB3/AN9/C3INA/CTED2/VPO/RP6, SERVO_10-1.S
- removed net OC4(1): IC1.RB1/AN10/C3INC/RTCC/RP4, SERVO_7-1.S
- removed net PH4: C20.2, D4.K, L4.1, U$9.PH
- removed net SWITCH_3: IC1.OSC1/CLKI/RA7, R27.1, U$11.P2, U$11.P3
- removed net SWITCH_4: IC1.RA0/AN0/C1INA/ULPWU/RP0, R28.1, U$12.P2, U$12.P3
- removed net VOUT4: C22.+, L4.2, MOTOR_PWR-2.S, MOTOR_PWR-3.S, R10.2, R12.2
- removed net VSNS4: R10.1, R11.2, U$9.VSNS
- net 3.3V: no longer C34.1, C35.1, IC1.RB7/CCP7/KBI3/PGD/RP10, IC1.RC2/AN11/C2IND/CTPLS/RP13, R26.2, U$11.P1, U$11.P4, U$12.P1, U$12.P4
- net GND: now also 3.3V(2)1-2.S, 3.3V1-2.S, 5V(2)1-2.S, 5V1-2.S, R10.1; no longer C19.1, C22.-, C30.1, C31.1, C32.1, C33.2, C34.2, C35.2, C36.2, D4.A_2, D6.C, D8.C, IC1.RB6/CCP6/KBI2/PGC/RP9, IC1.VSS1, LED10.C, LED11.C, LED12.C, LED3.C, MOTOR_PWR-1.S, MOTOR_PWR-4.S, PWR_IN(2)-1.S, Q4.S, R27.2, R28.2, SERVO_10-3.S, SERVO_7-3.S, SERVO_8-3.S, SERVO_9-3.S, U$10.P1, U$10.P4, U$3P8.DGND@1, U$3P8.DGND@2, U$3P9.DGND@1, U$3P9.DGND@2, U$3P9.DGND@3, U$3P9.DGND@4, U$3P9.DGND@5, U$3P9.DGND@6, U$9.GND_2, U$9.PWPD
- net IO3: now also R25.2; no longer R21.2
- net IO4: now also R24.2; no longer R25.2
- net IO5: now also R23.2; no longer R24.2
- net IO7: now also R21.2; no longer R23.2
- net IO8: no longer IC1.RA1/AN1/C2INA/VBG/RP1
- net OC1: now also SERVO_6-1.S; no longer SERVO_1-1.S
- net OC2: now also SERVO_5-1.S; no longer SERVO_2-1.S
- net OC3: now also SERVO_4-1.S; no longer SERVO_3-1.S
- net OC4: now also SERVO_3-1.S; no longer SERVO_4-1.S
- net OC5: now also SERVO_2-1.S; no longer SERVO_5-1.S
- net OC6: now also SERVO_1-1.S; no longer SERVO_6-1.S
- net PGC1: no longer IC1.RA3/AN3/C1INB/VREF+
- net PGD1: no longer IC1.RA2/AN2/C2INB/C1IND/C3INB/VREF-/CVREF
- net SCL: no longer IC1.RA5/AN4/C1INC/!SS1!/HLVDIN/RCV/RP2
- net SDA: no longer IC1.VDDCORE/VCAP
- net START_LEFT: now also R10.2
- net START_RIGHT: now also R11.2
- net VCC: no longer C19.2, C30.2, C31.2, C32.2, PWR_IN(2)-2.S, U$9.VIN
- net VOUT1: now also 5V(2)1-1.S, 5V1-1.S; no longer R16.2, R35.2
- net VOUT2: now also SERVO_6-2.S; no longer C27.1, SERVO_1-2.S, SERVO_2-2.S, SERVO_3-2.S
- net VOUT3: now also C27.1, SERVO_1-2.S, SERVO_2-2.S, SERVO_3-2.S; no longer C33.1, SERVO_10-2.S, SERVO_6-2.S, SERVO_7-2.S, SERVO_8-2.S, SERVO_9-2.S
- net VOUT5: now also 3.3V(2)1-1.S, 3.3V1-1.S
Other:
- note removed: "Regulator for Motor Power ~ 6 Volt"

Commit message: final commit of motherboard
Parts:
- added C19, C22, C51, C52, C53, C54: 0.01uF, rcl:C-USC0402
- added C20, C30, C33, C45, C46, C47, C48, C49, C50, C56, C57: 0.1uF, rcl:C-USC0402
- added C31, C32, C39, C40: 1nF, rcl:C-USC0402
- added C34, C35, C36, C42, C43, C44: 0.22uF, rcl:C-USC0402
- added C41, C68: .1uF, rcl:C-USC0402
- added C55: 1uF, rcl:C-USC0402
- added C58, C59, C60: (no value), rcl:CPOL-US153CLV-0605
- added C61: 10uF, rcl:C-USC0805
- added C62, C65, C66, C67: 4.7uF, 5v:GRM31CR71H475KA12L
- added C63: 10nF, 5v:C0805C103K5RACTU
- added C64: 330uF, 5v:10SVP330MX
- added C69, C70: 0.47uF, rcl:C-USC0402
- added D4: PDS760-13, 5v:PDS760-13
- added IC1, IC2: DRV8814, Motor-Board:DRV8818PWPR
- added IC4: PIC24FJ256GB106, microchip:PIC24FJ256GB106
- added L4: (no value), WE-HCC:WE-HCC-7443331000_1090
- added LED10, LED11, LED12, LED13, LED16, LED17, LED18, LED19, LED20, LED3, POWER_ON: (no value), led:LEDCHIP-LED0603
- added MOTIN1, MOTIN2, MOTIN3, MOTIN4, STEP1, STEP2: 22-05-7048-04, Son_of_Dark_Power:22-05-7048-04
- added MOTOR1, MOTOR2, MOTOR3, MOTOR4: 22-05-7028-02, Son_of_Dark_Power:22-05-7028-02
- added PROGRAMMING1: Jtag, Mother-Board-rev5:MOTHER-BOARD-REV5_PIN-CONNECTOR74089
- added PWR_IN(2): (no value), Son_of_Dark_Powersch:555X-2H
- added R12, R28: 1M, rcl:R-US_R0402
- added R16, R18, R29, R30: 0.2, rcl:R-US_R0402
- added R26, R31, R40, R41, R42, R43, R48, R49, R50, R51, R52, R54, R56, R57, R58, R59, R61, R62, R63, R64: 10k, rcl:R-US_R0402
- added R27, R35: 30k, rcl:R-US_R0402
- added R36, R37, R44, R45: 0.1, rcl:R-US_R0402
- added R38, R39, R46, R47: 47k, rcl:R-US_R0402
- added R53, R67, R68, R69, R70, R71: (no value), rcl:R-US_R0402
- added R55: 100, rcl:R-US_R0402
- added R60: (no value), rcl:R-US_R0805
- added SERVO_7, SERVO_8, SERVO_9: 22-05-7038-03, con-molex:22-05-7038-03
- added U$10: LOGO, logo:LOGO
- added U$3: TPS5450DDAR, 5v:TPS5450DDAR
- added U$9: Switch3, Parts4Class:MC32882_SW
- added U2, U4: DRV8811PWP, Texas Instruments_By_element14_Batch_1:DRV8811PWP
- LED1, LED2, LED4: device led:LEDSML1206 -> led:LEDCHIP-LED0603
- LED5, LED6, LED7, LED8, LED9: device led:LEDCHIPLED-0603-TTW -> led:LEDCHIP-LED0603
- R32: device rcl:R-US_R0402 -> rcl:R-US_R0805
- R4, R6, R9: device rcl:R-US_R1206 -> rcl:R-US_R0402
Connections:
- new net +7V: C20.2, C30.2, C36.1, C44.1, C45.1, C46.1, C47.1, C48.1, C51.1, C52.1, C53.1, C54.1, C58.+, C59.+, C60.+, C61.1, C64.+, H4.MOUNT, IC1.VMA, IC1.VMB, IC2.VMA, IC2.VMB, L4.2, MOTIN1-2.S, MOTIN2-2.S, MOTIN3-2.S, MOTIN4-2.S, R12.2, R28.2, R52.2, R54.2, R64.2, SERVO_7-2.S, SERVO_8-2.S, SERVO_9-2.S, U2.VMA, U2.VMB, U4.VMA, U4.VMB
- new net BOOT_VM: C63.1, U$3.BOOT
- new net CHANNEL_A_1: IC4.RG6, MOTIN1-4.S
- new net CHANNEL_A_2: IC4.RB9, MOTIN2-3.S
- new net CHANNEL_A_3: IC4.RB7, MOTIN3-3.S
- new net CHANNEL_A_4: IC4.RG9, MOTIN4-3.S
- new net CHANNEL_B_1: IC4.RG7, MOTIN1-3.S
- new net CHANNEL_B_2: IC4.RB8, MOTIN2-4.S
- new net CHANNEL_B_3: IC4.RB6, MOTIN3-4.S
- new net CHANNEL_B_4: IC4.RG8, MOTIN4-4.S
- new net GPIO23: R70.2, U$1P8.GPIO_23
- new net GPIO45: R69.2, U$1P8.GPIO_45
- new net GPIO47: R71.2, U$1P8.GPIO_47
- new net GPIO66: R67.2, U$1P8.GPIO_66
- new net GPIO69: R68.2, U$1P8.GPIO_69
- new net M-DECAY: IC1.DECAY, IC2.DECAY, IC4.RD1
- new net M-I0: IC1.AI0, IC1.BI0, IC2.AI0, IC2.BI0, IC4.RD10
- new net M-I1: IC1.AI1, IC1.BI1, IC2.AI1, IC2.BI1, IC4.RC15
- new net M-NSLEEP: IC1.NSLEEP, IC2.NSLEEP, IC4.RF0, U2.SLEEPN, U4.SLEEPN
- new net M-RESET: IC1.NRESET, IC2.NRESET, IC4.RE0, U2.RESETN, U4.RESETN
- new net M1-AENBL: IC1.AENBL, IC4.RC13
- new net M1-APHASE: IC1.APHASE, IC4.RC14
- new net M1-BENBL: IC1.BENBL, IC4.RD0
- new net M1-BHPASE: IC1.BHPASE, IC4.RD11
- new net M1-MAOUT1: IC1.AOUT1, MOTOR2-1.S
- new net M1-MAOUT2: IC1.AOUT2, MOTOR2-2.S
- new net M1-MBOUT1: IC1.BOUT1, MOTOR1-1.S
- new net M1-MBOUT2: IC1.BOUT2, MOTOR1-2.S
- new net M2-AENBL: IC2.AENBL, IC4.RC12
- new net M2-APHASE: IC2.APHASE, IC4.RD9
- new net M2-BENBL: IC2.BENBL, IC4.RG2
- new net M2-BHPASE: IC2.BHPASE, IC4.RD8
- new net M2-MAOUT1: IC2.AOUT1, MOTOR4-1.S
- new net M2-MAOUT2: IC2.AOUT2, MOTOR4-2.S
- new net M2-MBOUT1: IC2.BOUT1, MOTOR3-1.S
- new net M2-MBOUT2: IC2.BOUT2, MOTOR3-2.S
- new net M_MCLR: C68.1, PROGRAMMING1.P$7, PROGRAMMING1.P$8, R55.2, R56.1, U$9.P2, U$9.P3
- new net M_MCLR': IC4.!MCLR, R55.1
- new net M_PGC1: IC4.RB1, PROGRAMMING1.P$3, PROGRAMMING1.P$4
- new net M_PGD1: IC4.RB0, PROGRAMMING1.P$5, PROGRAMMING1.P$6
- new net N$12: C19.1, IC1.CP1
- new net N$13: C20.1, IC1.VCP, R12.1
- new net N$14: IC1.ISENA, R16.1
- new net N$15: IC1.ISENB, R18.1
- new net N$16: IC1.AVREV, IC1.BVREF, R26.1, R27.1
- new net N$17: C22.2, IC2.CP2
- new net N$20: C22.1, IC2.CP1
- new net N$21: C30.1, IC2.VCP, R28.1
- new net N$22: IC2.ISENA, R29.1
- new net N$23: IC2.ISENB, R30.1
- new net N$24: IC2.AVREV, IC2.BVREF, R31.1, R35.1
- new net N$26: IC1.NFAULT, R57.1
- new net N$27: R37.1, U2.ISENB
- new net N$28: R36.1, U2.ISENA
- new net N$29: C69.1, IC1.V3V3OUT, R26.2, R57.2
- new net N$30: C31.1, R38.1, U2.RCA
- new net N$32: C32.1, R39.1, U2.RCB
- new net N$33: C33.1, R40.2, R41.1, U2.DECAY
- new net N$34: R42.1, R43.2, U2.VREF
- new net N$35: IC2.NFAULT, R58.1
- new net N$36: C34.1, U2.CP1
- new net N$37: C70.1, IC2.V3V3OUT, R31.2, R58.2
- new net N$38: C34.2, U2.CP2
- new net N$39: C35.1, U2.VGD
- new net N$4: C19.2, IC1.CP2
- new net N$40: C36.2, U2.VCP
- new net N$41: R45.1, U4.ISENB
- new net N$42: R44.1, U4.ISENA
- new net N$43: C39.1, R46.1, U4.RCA
- new net N$44: C40.1, R47.1, U4.RCB
- new net N$45: C41.1, R48.2, R49.1, U4.DECAY
- new net N$46: R50.1, R51.2, U4.VREF
- new net N$47: C42.1, U4.CP1
- new net N$48: C42.2, U4.CP2
- new net N$49: C43.1, U4.VGD
- new net N$50: C44.2, U4.VCP
- new net N$51: LED3.A, R54.1
- new net N$52: POWER_ON.A, R59.1
- new net N$55: LED16.A, R67.1
- new net N$56: LED17.A, R68.1
- new net N$57: LED18.A, R69.1
- new net N$58: LED19.A, R70.1
- new net N$59: LED20.A, R71.1
- new net N$60: LED10.A, R61.1
- new net N$61: LED11.A, R62.1
- new net N$62: LED12.A, R63.1
- new net N$63: LED13.A, R64.1
- new net OC1': IC4.RF3, SERVO_7-1.S
- new net OC2': IC4.RF5, SERVO_8-1.S
- new net OC3': IC4.RF4, SERVO_9-1.S
- new net PH_VM: C63.2, D4.K, L4.1, U$3.PH
- new net S-SRN: IC4.RF1, U2.SRN, U4.SRN
- new net S1-AOUT1: STEP1-4.S, U2.AOUT1
- new net S1-AOUT2: STEP1-1.S, U2.AOUT2
- new net S1-BOUT1: STEP1-3.S, U2.BOUT1
- new net S1-BOUT2: STEP1-2.S, U2.BOUT2
- new net S1-DIR: IC4.RE4, U2.DIR
- new net S1-ENABLEN: IC4.RD7, U2.ENABLEN
- new net S1-HOME: IC4.RE3, U2.HOME
- new net S1-STEP: IC4.RD5, U2.STEP
- new net S2-AOUT1: STEP2-4.S, U4.AOUT1
- new net S2-AOUT2: STEP2-1.S, U4.AOUT2
- new net S2-BOUT1: STEP2-3.S, U4.BOUT1
- new net S2-BOUT2: STEP2-2.S, U4.BOUT2
- new net S2-DIR: IC4.RD6, U4.DIR
- new net S2-ENABLEN: IC4.RD3, U4.ENABLEN
- new net S2-HOME: IC4.RD4, U4.HOME
- new net S2-STEP: IC4.RD2, U4.STEP
- new net USM0: IC4.RE2, U2.USM0, U4.USM0
- new net USM1: IC4.RE1, U2.USM1, U4.USM1
- new net VSNS_VM: R52.1, R53.2, U$3.VSNS
- net 3.3V: now also C49.1, C50.1, C55.1, C56.1, C57.1, IC4.VDD@1, IC4.VDD@2, IC4.VDD@3, PROGRAMMING1.P$1, PROGRAMMING1.P$2, R40.1, R43.1, R48.1, R51.1, R56.2, R60.1, R60.2, U2.VCC, U4.VCC
- net GND: now also C31.2, C32.2, C33.2, C35.2, C39.2, C40.2, C41.2, C43.2, C45.2, C46.2, C47.2, C48.2, C49.2, C50.2, C51.2, C52.2, C53.2, C54.2, C55.2, C56.2, C57.2, C58.-, C59.-, C60.-, C61.2, C62.1, C64.-, C65.1, C66.1, C67.1, C68.2, C69.2, C70.2, D4.A_2, IC1.GND, IC2.GND, IC4.VSS@1, IC4.VSS@2, IC4.VSS@3, LED10.C, LED11.C, LED12.C, LED13.C, LED16.C, LED17.C, LED18.C, LED19.C, LED20.C, LED3.C, MOTIN1-1.S, MOTIN2-1.S, MOTIN3-1.S, MOTIN4-1.S, POWER_ON.C, PROGRAMMING1.P$10, PROGRAMMING1.P$9, PWR_IN(2)-1.S, R16.2, R18.2, R27.2, R29.2, R30.2, R35.2, R36.2, R37.2, R38.2, R39.2, R41.2, R42.2, R44.2, R45.2, R46.2, R47.2, R49.2, R50.2, R53.1, SERVO_7-3.S, SERVO_8-3.S, SERVO_9-3.S, U$3.GND_2, U$3.PWPD, U$9.P1, U$9.P4, U2.EP, U2.GND, U2.GND_2, U4.EP, U4.GND, U4.GND_2
- net SCL: now also IC4.RE6
- net SDA: now also IC4.RE7
- net VCC: now also C62.2, C65.2, C66.2, C67.2, PWR_IN(2)-2.S, R59.2, U$3.VIN
- net VOUT1: now also R63.2
- net VOUT2: now also R61.2
- net VOUT3: now also R62.2
