File: designs/Motherboard/MotherboardRev2/MotherboardRev2.sch (EAGLE design)
At the start: 227 parts, among them IC1 DRV8814, IC2 DRV8814, IC3 PIC24FJ64GB202, IC4 PIC24FJ256GB106, Q1 BSS123, Q2 BSS123, Q3 BSS123, U1 LMS8117AMP-3.3, U2 DRV8811PWP, U3 LMS8117AMP-3.3, U4 DRV8811PWP

Commit message: Done with Motherboard
Parts:
- added C71: 0.1uF, rcl:C-USC0402
- added MOTIN5: 22-05-7048-04, Son_of_Dark_Power:22-05-7048-04
- R10, R11: value (none) -> 10K
- R13: value 470 -> 100
- R19, R20: value 4.7k -> 10K
- R21, R22, R23, R24, R25: value (none) -> 330
- R67, R68, R69, R70, R71: value (none) -> 1K
Connections:
- net +7V: now also MOTIN5-2.S, MOTIN5-3.S
- net 3.3V: now also C71.1, IC4.AVDD
- net GND: now also C71.2, IC4.AVSS, MOTIN5-1.S, MOTIN5-4.S
Changed lines of the file:
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@@
 <part name="GND3" library="Son_of_Dark_Powersch" deviceset="GND" device=""/>
 <part name="FRAME2" library="frames" deviceset="DINA5_L" device="" value="Microcontroller"/>
-<part name="R13" library="rcl" deviceset="R-US_" device="R0402" value="470"/>
+<part name="R13" library="rcl" deviceset="R-US_" device="R0402" value="100"/>
 <part name="R14" library="rcl" deviceset="R-US_" device="R0402" value="10k"/>
 <part name="C21" library="rcl" deviceset="C-US" device="C0402" value=".1uF"/>
@@
 <part name="U$6" library="Parts4Class" deviceset="MC32882_SW" device="" value="Switch1"/>
 <part name="U$7" library="Parts4Class" deviceset="MC32882_SW" device="" value="Switch2"/>
-<part name="R19" library="rcl" deviceset="R-US_" device="R0402" value="4.7k"/>
-<part name="R20" library="rcl" deviceset="R-US_" device="R0402" value="4.7k"/>
+<part name="R19" library="rcl" deviceset="R-US_" device="R0402" value="10K"/>
+<part name="R20" library="rcl" deviceset="R-US_" device="R0402" value="10K"/>
 <part name="LED5" library="led" deviceset="LED" device="CHIP-LED0603"/>
 <part name="LED6" library="led" deviceset="LED" device="CHIP-LED0603"/>
@@
 <part name="LED8" library="led" deviceset="LED" device="CHIP-LED0603"/>
 <part name="LED9" library="led" deviceset="LED" device="CHIP-LED0603"/>
-<part name="R21" library="rcl" deviceset="R-US_" device="R0402"/>
-<part name="R22" library="rcl" deviceset="R-US_" device="R0402"/>
-<part name="R23" library="rcl" deviceset="R-US_" device="R0402"/>
-<part name="R24" library="rcl" deviceset="R-US_" device="R0402"/>
-<part name="R25" library="rcl" deviceset="R-US_" device="R0402"/>
+<part name="R21" library="rcl" deviceset="R-US_" device="R0402" value="330"/>
+<part name="R22" library="rcl" deviceset="R-US_" device="R0402" value="330"/>
+<part name="R23" library="rcl" deviceset="R-US_" device="R0402" value="330"/>
+<part name="R24" library="rcl" deviceset="R-US_" device="R0402" value="330"/>
+<part name="R25" library="rcl" deviceset="R-US_" device="R0402" value="330"/>
 <part name="C27" library="rcl" deviceset="C-US" device="C0805" value="10uF"/>
 <part name="C28" library="rcl" deviceset="C-US" device="C0805" value="10uF"/>
@@
 <part name="3.3V1" library="Son_of_Dark_Powersch" deviceset="22-?-02" device="05-7028" value=""/>
 <part name="3.3V(2)1" library="Son_of_Dark_Powersch" deviceset="22-?-02" device="05-7028" value=""/>
-<part name="R10" library="rcl" deviceset="R-US_" device="R0402"/>
-<part name="R11" library="rcl" deviceset="R-US_" device="R0402"/>
+<part name="R10" library="rcl" deviceset="R-US_" device="R0402" value="10K"/>
+<part name="R11" library="rcl" deviceset="R-US_" device="R0402" value="10K"/>
 <part name="GND10" library="supply1" deviceset="GND" device=""/>
 <part name="GND11" library="supply1" deviceset="GND" device=""/>
@@
 <part name="LED19" library="led" deviceset="LED" device="CHIP-LED0603"/>
 <part name="LED20" library="led" deviceset="LED" device="CHIP-LED0603"/>
-<part name="R67" library="rcl" deviceset="R-US_" device="R0402"/>
-<part name="R68" library="rcl" deviceset="R-US_" device="R0402"/>
-<part name="R69" library="rcl" deviceset="R-US_" device="R0402"/>
-<part name="R70" library="rcl" deviceset="R-US_" device="R0402"/>
-<part name="R71" library="rcl" deviceset="R-US_" device="R0402"/>
+<part name="R67" library="rcl" deviceset="R-US_" device="R0402" value="1K"/>
+<part name="R68" library="rcl" deviceset="R-US_" device="R0402" value="1K"/>
+<part name="R69" library="rcl" deviceset="R-US_" device="R0402" value="1K"/>
+<part name="R70" library="rcl" deviceset="R-US_" device="R0402" value="1K"/>
+<part name="R71" library="rcl" deviceset="R-US_" device="R0402" value="1K"/>
 <part name="GND29" library="supply1" deviceset="GND" device=""/>
+<part name="MOTIN5" library="Son_of_Dark_Power" deviceset="22-?-04" device="05-7048"/>
+<part name="C71" library="rcl" deviceset="C-US" device="C0402" value="0.1uF"/>
 </parts>
 <sheets>
@@
 <instance part="GND23" gate="1" x="474.98" y="78.74" rot="R90"/>
 <instance part="GND24" gate="1" x="411.48" y="50.8" rot="R90"/>
-<instance part="+3V7" gate="G$1" x="373.38" y="43.18" rot="R90"/>
+<instance part="+3V7" gate="G$1" x="358.14" y="43.18" rot="R90"/>
 <instance part="+3V8" gate="G$1" x="309.88" y="99.06" rot="R180"/>
 <instance part="+3V9" gate="G$1" x="477.52" y="66.04" rot="R270"/>
@@
 <instance part="+3V11" gate="G$1" x="551.18" y="121.92"/>
 <instance part="GND28" gate="1" x="508" y="76.2"/>
+<instance part="MOTIN5" gate="-1" x="332.74" y="5.08"/>
+<instance part="MOTIN5" gate="-2" x="332.74" y="0"/>
+<instance part="MOTIN5" gate="-3" x="332.74" y="-5.08"/>
+<instance part="MOTIN5" gate="-4" x="332.74" y="-10.16"/>
+<instance part="C71" gate="G$1" x="396.24" y="35.56" rot="R90"/>
 </instances>
 <busses>
@@
 <wire x1="406.4" y1="50.8" x2="408.94" y2="50.8" width="0.1524" layer="91"/>
 <wire x1="401.32" y1="43.18" x2="406.4" y2="43.18" width="0.1524" layer="91"/>
-<wire x1="406.4" y1="43.18" x2="406.4" y2="50.8" width="0.1524" layer="91"/>
+<wire x1="406.4" y1="43.18" x2="406.4" y2="48.26" width="0.1524" layer="91"/>
 <junction x="406.4" y="50.8"/>
 <pinref part="IC4" gate="G$1" pin="VSS@2"/>
+<pinref part="C71" gate="G$1" pin="2"/>
+<wire x1="406.4" y1="48.26" x2="406.4" y2="50.8" width="0.1524" layer="91"/>
+<wire x1="401.32" y1="35.56" x2="406.4" y2="35.56" width="0.1524" layer="91"/>
+<wire x1="406.4" y1="35.56" x2="406.4" y2="43.18" width="0.1524" layer="91"/>
+<junction x="406.4" y="43.18"/>
+<pinref part="IC4" gate="G$1" pin="AVSS"/>
+<wire x1="373.38" y1="76.2" x2="373.38" y2="48.26" width="0.1524" layer="91"/>
+<wire x1="373.38" y1="48.26" x2="406.4" y2="48.26" width="0.1524" layer="91"/>
+<junction x="406.4" y="48.26"/>
 </segment>
 <segment>
@@
 <pinref part="GND27" gate="1" pin="GND"/>
 </segment>
+<segment>
+<pinref part="MOTIN5" gate="-4" pin="S"/>
+<wire x1="330.2" y1="-10.16" x2="320.04" y2="-10.16" width="0.1524" layer="91"/>
+<label x="320.04" y="-10.16" size="1.778" layer="95" rot="R180"/>
+</segment>
+<segment>
+<pinref part="MOTIN5" gate="-1" pin="S"/>
+<wire x1="330.2" y1="5.08" x2="320.04" y2="5.08" width="0.1524" layer="91"/>
+<label x="320.04" y="5.08" size="1.778" layer="95" rot="R180"/>
+</segment>
 </net>
 <net name="3.3V" class="0">
 <segment>
 <pinref part="+3V7" gate="G$1" pin="+3V3"/>
-<wire x1="375.92" y1="43.18" x2="388.62" y2="43.18" width="0.1524" layer="91"/>
+<wire x1="360.68" y1="43.18" x2="370.84" y2="43.18" width="0.1524" layer="91"/>
+<wire x1="370.84" y1="43.18" x2="388.62" y2="43.18" width="0.1524" layer="91"/>
 <wire x1="388.62" y1="43.18" x2="388.62" y2="76.2" width="0.1524" layer="91"/>
 <pinref part="C57" gate="G$1" pin="1"/>
@@
 <junction x="388.62" y="43.18"/>
 <pinref part="IC4" gate="G$1" pin="VDD@2"/>
+<pinref part="C71" gate="G$1" pin="1"/>
+<wire x1="393.7" y1="35.56" x2="388.62" y2="35.56" width="0.1524" layer="91"/>
+<wire x1="388.62" y1="35.56" x2="388.62" y2="43.18" width="0.1524" layer="91"/>
+<pinref part="IC4" gate="G$1" pin="AVDD"/>
+<wire x1="370.84" y1="76.2" x2="370.84" y2="43.18" width="0.1524" layer="91"/>
+<junction x="370.84" y="43.18"/>
 </segment>
 <segment>
@@
 <pinref part="SUPPLY9" gate="G$1" pin="+7V"/>
 </segment>
+<segment>
+<pinref part="MOTIN5" gate="-2" pin="S"/>
+<wire x1="330.2" y1="0" x2="320.04" y2="0" width="0.1524" layer="91"/>
+<label x="320.04" y="0" size="1.778" layer="95" rot="R180"/>
+</segment>
+<segment>
+<pinref part="MOTIN5" gate="-3" pin="S"/>
+<wire x1="330.2" y1="-5.08" x2="320.04" y2="-5.08" width="0.1524" layer="91"/>
+<label x="320.04" y="-5.08" size="1.778" layer="95" rot="R180"/>
+</segment>
 </net>

Commit message: Added values for some of the capactiors
Parts:
- removed Q1, Q2, Q3: BSS123, transistor-small-signal:BSS123
- added C72: 4.7uF, rcl:C-USC0402
- added LED14: (no value), led:LEDCHIP-LED0603
- added LIDAR: (no value), con-lstb:MA04-1
- added R65: 10k, rcl:R-US_R0402
- C58, C59, C60: value (none) -> 100uf
Connections:
- removed net EN1: Q2.G
- removed net EN2: Q1.G
- removed net EN3: Q3.G
- removed net ENA_1: Q2.D, U$2.ENA
- removed net ENA_2: Q1.D, U$4.ENA
- removed net ENA_3: Q3.D, U$8.ENA
- new net N$19: LED14.A, R65.1
- new net UART_RX: LIDAR.2, U$1P9.GPIO_2
- new net UART_TX: LIDAR.3, U$1P9.GPIO_3
- net 3.3V: now also C72.1, LIDAR.4
- net GND: now also C72.2, LED14.C, LIDAR.1; no longer Q1.S, Q2.S, Q3.S
- net VCC: now also R65.2

Commit message: final
Parts:
- removed C21: .1uF, rcl:C-USC0402
- removed C55: 1uF, rcl:C-USC0402
- removed C56, C57, C71: 0.1uF, rcl:C-USC0402
- removed C61: 10uF, rcl:C-USC0805
- removed C62, C65, C66: 4.7uF, 5v:GRM31CR71H475KA12L
- removed C72: 4.7uF, rcl:C-USC0402
- removed D5, D7: 3_3V_PWR, SparkFun-LED:LED-FKIT-1206
- removed LED16, LED17, LED18, LED19, LED20: (no value), led:LEDCHIP-LED0603
- removed MOTOR4: 22-05-7028-02, Son_of_Dark_Power:22-05-7028-02
- removed R24, R25: 330, rcl:R-US_R0402
- removed R33: 4.7K, rcl:R-US_R0402
- removed R34: (no value), rcl:R-US_R0805W
- removed R60: (no value), rcl:R-US_R0805
- removed R61, R62, R63, R64: 10k, rcl:R-US_R0402
- removed R67, R68, R69, R70, R71: 1K, rcl:R-US_R0402
- removed U$10: LOGO, logo:LOGO
- removed U$6: Switch1, Parts4Class:MC32882_SW
- removed U$7: Switch2, Parts4Class:MC32882_SW
- added C104: 0.01uF, rcl:C-USC0402
- added C108, C110, C112: 10nF, 5v:C0805C103K5RACTU
- added C109, C111, C113: 4.7uF, rcl:C-USC0805
- added C125, C126, C127: 330uF, 5v:10SVP330MX
- added D101, D102: PDS760-13, 5v:PDS760-13
- added LED100, LED101, LED102, LED103, LED104: (no value), led:LEDCHIP-LED0603
- added MOTOR101: 22-05-7028-02, Son_of_Dark_Power:22-05-7028-02
- added R104, R106, R108, R133, R134, R135: 10k, rcl:R-US_R0402
- added R105, R107: 2.55k, rcl:R-US_R0402
- added R109: 3.23K, rcl:R-US_R0402
- added R113: 1M, rcl:R-US_R0402
- added R121, R122: 0.2, rcl:R-US_R0402
- added R136, R138: 330, rcl:R-US_R0402
- added U$102: Switch3, Parts4Class:MC32882_SW
- added U$105, U$107: TPS5450DDAR, 5v:TPS5450DDAR
- C1, C2: value 4.7uF -> 0.1uF; device rcl:C-USC0805 -> rcl:C-USC0402
- C14: value 10nF -> 4.7uF; device 5v:C0805C103K5RACTU -> rcl:C-USC0805
- C15: value 330uF -> 4.7uF; device 5v:10SVP330MX -> rcl:C-USC0805
- C19: value 0.01uF -> 10uF; device rcl:C-USC0402 -> rcl:C-USC0805
- C3: value 10nF -> 1uF; device 5v:C0805C103K5RACTU -> rcl:C-USC0402
- C4: value 10nF -> 0.1uF; device 5v:C0805C103K5RACTU -> rcl:C-USC0402
- C5: value 330uF -> 4.7uF; device 5v:10SVP330MX -> rcl:C-USC0402
- C6, C7, C8: device rcl:C-USC0805 -> 5v:GRM31CR71H475KA12L
- C9: value 330uF -> .1uF; device 5v:10SVP330MX -> rcl:C-USC0402
- D1, D2: value PDS760-13 -> 3_3V_PWR; device 5v:PDS760-13 -> led:LEDCHIP-LED0603
- R1: value 10k -> 0; device rcl:R-US_R1206 -> rcl:R-US_R0805
- R10, R11: value 10K -> 1K
- R12: value 1M -> 1K
- R124: value (none) -> 2.55k
- R13: value 100 -> 10K
- R14: value 10k -> 330
- R15: value (none) -> 330; device rcl:R-US_R0805W -> rcl:R-US_R0402
- R16, R18: value 0.2 -> 330
- R17: value 4.7K -> 330
- R2: device rcl:R-US_R1206 -> rcl:R-US_R0402
- R20: value 10K -> 100
- R21: value 330 -> 10k
- R22, R23: value 330 -> 10K
- R3, R5: value (none) -> 10k; device rcl:R-US_R1206 -> rcl:R-US_R0402
- R6: value 10k -> 1K
- R7: value 10k -> 1K; device rcl:R-US_R1206 -> rcl:R-US_R0402
- R8: value (none) -> 4.7K; device rcl:R-US_R1206 -> rcl:R-US_R0402
- R9: value 10k -> 4.7K
- U$1: value BEAGLE_BONE_BLACK_CAPE -> LOGO; device Son_of_Dark_Powersch:BEAGLE_BONE_BLACK_CAPE -> logo:LOGO
- U$3: value TPS5450DDAR -> Switch2; device 5v:TPS5450DDAR -> Parts4Class:MC32882_SW
- U$4: value TPS5450DDAR -> Switch1; device 5v:TPS5450DDAR -> Parts4Class:MC32882_SW
- U$5: value Switch3 -> BEAGLE_BONE_BLACK_CAPE; device Parts4Class:MC32882_SW -> Son_of_Dark_Powersch:BEAGLE_BONE_BLACK_CAPE
- renumbered C20 to C105, C22 to C100, C23 to C136, C24 to C137, C25 to C128, C26 to C129, C27 to C143, C28 to C144, C29 to C145, C30 to C101, C31 to C149, C32 to C148, C33 to C150, C34 to C141, C35 to C139, C36 to C140, C37 to C114, C38 to C151, C39 to C133, C40 to C132, C41 to C134, C42 to C122, C43 to C120, C44 to C121, C45 to C119, C46 to C123, C47 to C142, C48 to C138, C49 to C147, C50 to C131, C51 to C106, C52 to C117, C53 to C107, C54 to C102, C58 to C152, C59 to C135, C60 to C124, C63 to C118, C64 to C146, C67 to C130, C68 to C115, C69 to C116, C70 to C103, D3 to D100, D4 to D103, IC1 to IC101, IC2 to IC100, IC3 to IC102, IC4 to IC103, L1 to L102, L2 to L101, L3 to L100, L4 to L103, MOTIN1 to MOTIN100, MOTIN2 to MOTIN102, MOTIN3 to MOTIN103, MOTIN4 to MOTIN104, MOTIN5 to MOTIN101, MOTOR3 to MOTOR100, PROGRAMMING1 to PROGRAMMING100, R26 to R118, R27 to R120, R28 to R102, R29 to R103, R30 to R114, R31 to R111, R32 to R115, R35 to R112, R36 to R137, R37 to R139, R38 to R141, R39 to R140, R40 to R144, R41 to R145, R42 to R143, R43 to R142, R44 to R132, R45 to R125, R46 to R127, R47 to R126, R48 to R131, R49 to R129, R50 to R128, R51 to R130, R52 to R123, R53 to R124, R54 to R146, R55 to R116, R56 to R117, R57 to R119, R58 to R110, R59 to R101, R65 to R100, SERVO_1 to SERVO_103, SERVO_2 to SERVO_104, SERVO_3 to SERVO_105, SERVO_4 to SERVO_106, SERVO_5 to SERVO_107, SERVO_6 to SERVO_108, SERVO_7 to SERVO_102, SERVO_8 to SERVO_101, SERVO_9 to SERVO_100, U$13 to U$101, U$14 to U$100, U$2 to U$106, U$8 to U$104, U$9 to U$103, U1 to U103, U2 to U102, U3 to U101, U4 to U100
Connections:
- net +7V: now also C19.1, H1.MOUNT, R113.2, R2.2; no longer C61.1, H4.MOUNT, R12.2, R64.2
- net 3.3V: now also C1.1, C2.1, C3.1, C4.1, C5.1, R1.1, R1.2, R136.1, R21.2, R8.2, R9.2, U$3.P1, U$3.P4, U$4.P1, U$4.P4; no longer C55.1, C56.1, C57.1, C71.1, C72.1, R14.2, R15.1, R17.2, R33.2, R60.1, R60.2, U$6.P1, U$6.P4, U$7.P1, U$7.P4
- net BB_PWR_BUTTON: now also U$5P9.PWR_BUT; no longer U$1P9.PWR_BUT
- net BB_SYS_RESET: now also U$5P9.SYS_RESET!N; no longer U$1P9.SYS_RESET!N
- net BOOT1: now also C112.1; no longer C4.1
- net BOOT2: now also C110.1, U$105.BOOT; no longer C3.1, U$4.BOOT
- net BOOT3: now also C108.1; no longer C14.1
- net BOOT_VM: now also U$107.BOOT; no longer U$3.BOOT
- net GND: now also C1.2, C109.1, C111.1, C113.1, C125.-, C126.-, C127.-, C14.1, C15.1, C19.2, C2.2, C3.2, C4.2, C5.2, C9.2, D1.C, D101.A_2, D102.A_2, D2.C, LED100.C, LED101.C, LED102.C, LED103.C, LED104.C, R105.1, R107.1, R109.1, R121.2, R122.2, R13.1, R19.1, R22.2, R23.2, U$102.P1, U$102.P4, U$105.GND_2, U$105.PWPD, U$107.GND_2, U$107.PWPD, U$5P8.DGND@1, U$5P8.DGND@2, U$5P9.DGND@1, U$5P9.DGND@2, U$5P9.DGND@3, U$5P9.DGND@4, U$5P9.DGND@5, U$5P9.DGND@6; no longer C1.1, C15.-, C2.1, C21.2, C5.-, C55.2, C56.2, C57.2, C61.2, C62.1, C65.1, C66.1, C71.2, C72.2, C9.-, D1.A_2, D2.A_2, D5.C, D7.C, LED16.C, LED17.C, LED18.C, LED19.C, LED20.C, R10.1, R11.1, R16.2, R18.2, R19.2, R20.2, R3.1, R5.1, R8.1, U$1P8.DGND@1, U$1P8.DGND@2, U$1P9.DGND@1, U$1P9.DGND@2, U$1P9.DGND@3, U$1P9.DGND@4, U$1P9.DGND@5, U$1P9.DGND@6, U$3.GND_2, U$3.PWPD, U$4.GND_2, U$4.PWPD, U$5.P1, U$5.P4
- net GPIO23: now also R7.2, U$5P8.GPIO_23; no longer R70.2, U$1P8.GPIO_23
- net GPIO45: now also R10.2, U$5P8.GPIO_45; no longer R69.2, U$1P8.GPIO_45
- net GPIO47: now also R6.2, U$5P8.GPIO_47; no longer R71.2, U$1P8.GPIO_47
- net GPIO66: now also R12.2, U$5P8.GPIO_66; no longer R67.2, U$1P8.GPIO_66
- net GPIO69: now also R11.2, U$5P8.GPIO_69; no longer R68.2, U$1P8.GPIO_69
- net IO3: now also R18.2; no longer R25.2
- net IO4: now also R17.2; no longer R24.2
- net IO5: now also R16.2; no longer R23.2
- net IO6: now also R14.2; no longer R22.2
- net IO7: now also R15.2; no longer R21.2
- net M1-MAOUT1: now also MOTOR1-1.S; no longer MOTOR2-1.S
- net M1-MAOUT2: now also MOTOR1-2.S; no longer MOTOR2-2.S
- net M1-MBOUT1: now also MOTOR101-1.S; no longer MOTOR1-1.S
- net M1-MBOUT2: now also MOTOR101-2.S; no longer MOTOR1-2.S
- net M2-MAOUT1: now also MOTOR2-1.S; no longer MOTOR4-1.S
- net M2-MAOUT2: now also MOTOR2-2.S; no longer MOTOR4-2.S
- net MCLR: now also C9.1, R20.2, R21.1, U$102.P2, U$102.P3; no longer C21.1, R13.2, R14.1, U$5.P2, U$5.P3
- net MCLR': now also R20.1; no longer R13.1
- net N$1: now also LED103.A, R135.1; no longer LED4.A, R4.1
- net N$10: now also D2.A, R136.2; no longer D5.A, R15.2
- net N$11: now also D1.A, R138.2; no longer D7.A, R34.2
- net N$12: now also C104.1; no longer C19.1
- net N$13: now also R113.1; no longer R12.1
- net N$14: now also R121.1; no longer R16.1
- net N$15: now also R122.1; no longer R18.1
- net N$18: now also U$5P9.VDD_5V@1, U$5P9.VDD_5V@2; no longer U$1P9.VDD_5V@1, U$1P9.VDD_5V@2
- net N$19: now also LED100.A; no longer LED14.A
- net N$2: now also LED102.A, R134.1; no longer LED1.A, R6.1
- net N$3: now also LED101.A, R133.1; no longer LED2.A, R9.1
- net N$4: now also C104.2; no longer C19.2
- net N$5: now also LED10.A, R15.1; no longer LED5.A, R21.1
- net N$51: now also LED104.A; no longer LED3.A
- net N$55: now also LED9.A, R12.1; no longer LED16.A, R67.1
- net N$56: now also LED8.A, R11.1; no longer LED17.A, R68.1
- net N$57: now also LED7.A, R10.1; no longer LED18.A, R69.1
- net N$58: now also LED6.A, R7.1; no longer LED19.A, R70.1
- net N$59: now also LED5.A, R6.1; no longer LED20.A, R71.1
- net N$6: now also LED11.A, R14.1; no longer LED6.A, R22.1
- net N$60: now also LED3.A, R4.1; no longer LED10.A, R61.1
- net N$61: now also LED4.A, R5.1; no longer LED11.A, R62.1
- net N$62: now also LED2.A, R3.1; no longer LED12.A, R63.1
- net N$63: now also LED1.A, R2.1; no longer LED13.A, R64.1
- net N$7: now also LED12.A, R16.1; no longer LED7.A, R23.1
- net N$8: now also LED13.A, R17.1; no longer LED8.A, R24.1
- net N$9: now also LED14.A, R18.1; no longer LED9.A, R25.1
- net PH1: now also C112.2, D102.K; no longer C4.2, D2.K
- net PH2: now also C110.2, D101.K, U$105.PH; no longer C3.2, D1.K, U$4.PH
- net PH3: now also C108.2; no longer C14.2
- net PH_VM: now also U$107.PH; no longer U$3.PH
- net SCL: now also R9.1, U$5P9.I2C2_SCL; no longer R33.1, U$1P9.I2C2_SCL
- net SDA: now also R8.1, U$5P9.I2C2_SDA; no longer R17.1, U$1P9.I2C2_SDA
- net START_LEFT: now also R19.2, U$5P9.GPIO_60; no longer R10.2, U$1P9.GPIO_60
- net START_RIGHT: now also R13.2, U$5P9.GPIO_30; no longer R11.2, U$1P9.GPIO_30
- net SWITCH_1: now also R23.1, U$4.P2, U$4.P3; no longer R19.1, U$6.P2, U$6.P3
- net SWITCH_2: now also R22.1, U$3.P2, U$3.P3; no longer R20.1, U$7.P2, U$7.P3
- net UART_RX: now also U$5P9.GPIO_2; no longer U$1P9.GPIO_2
- net UART_TX: now also U$5P9.GPIO_3; no longer U$1P9.GPIO_3
- net VCC: now also C109.2, C111.2, C113.2, C14.2, C15.2, U$105.VIN, U$107.VIN; no longer C1.2, C2.2, C62.2, C65.2, C66.2, U$3.VIN, U$4.VIN
- net VOUT1: now also C127.+, R108.2, R135.2, R3.2; no longer C5.+, R2.2, R4.2, R63.2
- net VOUT2: now also C126.+, R106.2, R134.2, R4.2; no longer C9.+, R1.2, R6.2, R61.2
- net VOUT3: now also C125.+, R104.2, R133.2, R5.2; no longer C15.+, R62.2, R7.2, R9.2
- net VOUT5: now also R138.1; no longer R34.1
- net VSNS1: now also R108.1, R109.2; no longer R2.1, R3.2
- net VSNS2: now also R106.1, R107.2, U$105.VSNS; no longer R1.1, R5.2, U$4.VSNS
- net VSNS3: now also R104.1, R105.2; no longer R7.1, R8.2
- net VSNS_VM: now also U$107.VSNS; no longer U$3.VSNS
