File: designs/RPLidar_Interface_pic/RPLidar_interface.brd (EAGLE design)
At the start: 74.9 x 54.6 mm, 75 parts, among them IC1 TS5205, J1 PIN-CONNECTOR74089, J2 PIN-CONNECTOR74089, J3 PIN-CONNECTOR74089, J4 22-05-7028-02, J5 PIN-CONNECTOR74089, U1 PIC24FJ32GB002-I/ML, U2 PIC24FJ32GB002-I/ML, X1 22-23-2071

Commit message: cleaning up
Parts:
- removed C1, C18, C4: .1uF, rcl:C0402
- removed J1, J2, J5: PIN-CONNECTOR74089, Mother-Board-rev5:10-PIN-SMD
- removed R12, R14, R3: 100, resistor:R0402
- removed R19, R4, R6: 10k, resistor:R0402
- added RESET: EVQQ2, adafruit:EVQ-Q2
- added SV11: (no value), con-lstb:MA04-2
- moved R11 7.32 mm to (38.5, 17.4), flipped to the bottom
- moved J4 3.43 mm to (16.5, 14.1)
- moved C3 1.26 mm to (58.8, 32.1)
Connections:
- removed net ICSPCLK_A: J5.3, J5.4, U$2.24
- removed net ICSPCLK_P: J2.3, J2.4, U2.2
- removed net ICSPCLK_U: J1.3, J1.4, U$1.24
- removed net ICSPDAT_A: J5.5, J5.6, U$2.25
- removed net ICSPDAT_P: J2.5, J2.6, U2.1
- removed net ICSPDAT_U: J1.5, J1.6, U$1.25
- removed net MCLR_A: C18.1, J5.7, J5.8, R14.2, R19.1
- removed net MCLR_P: C4.1, J2.7, J2.8, R12.2, R6.1
- removed net MCLR_U: C1.1, J1.7, J1.8, R3.2, R4.1
- removed net N$7: U2.23
- removed net N$8: U2.22
- new net N$11: R11.1, SV11.2, SV11.4, SV11.6, SV11.8
- new net P8.11: U$3.P8.11, U2.23
- new net P8.12: U$3.P8.12, U2.22
- new net RPLIDAR_EN: U1.23, X1.2
- net +3V3: no longer J1.1, J1.2, J2.1, J2.2, R4.2, R6.2
- net 5V: no longer J5.1, J5.2, R19.2, X1.2
- net GND: now also RESET.A, RESET.A'; no longer C1.2, C18.2, C4.2, J1.10, J1.9, J2.10, J2.9, J5.10, J5.9
- net ICSPCLK: now also U$1.24, U$2.24, U2.2
- net ICSPDAT: now also U$1.25, U$2.25, U2.1
- net MCLR/VPP_A: now also SV11.3; no longer R14.1
- net MCLR/VPP_P: now also SV11.1; no longer R12.1
- net MCLR/VPP_U: now also SV11.5; no longer R3.1
- net MCLR_LIDAR: now also RESET.B, RESET.B'
- net VPP/MCLR: now also SV11.7; no longer R11.1
Routing:
- net ICSPDAT: track 7.75 -> 81.5 mm, vias 0 -> 4
- net ICSPCLK: track 8.00 -> 79.3 mm, vias 0 -> 5
- net P8.12: track 0.00 -> 54.4 mm, vias 0 -> 2
- net P8.11: track 0.00 -> 51.8 mm, vias 0 -> 2
- net VPP/MCLR: track 8.52 -> 36.2 mm
- net MCLR/VPP_A: track 3.59 -> 29.3 mm, vias 0 -> 4
- net +3V3: track 151.0 -> 126.7 mm, vias 11 -> 10
- net MCLR_LIDAR: track 10.3 -> 34.0 mm, vias 0 -> 2
- net MCLR/VPP_U: track 3.47 -> 27.0 mm, vias 0 -> 2
- net N$11: track 0.00 -> 21.3 mm, vias 0 -> 2
- net RPLIDAR_EN: track 0.00 -> 15.2 mm
- net ICSPCLK_P: track 14.9 -> 0.00 mm
- net ICSPDAT_P: track 13.7 -> 0.00 mm
- net MCLR_P: track 11.6 -> 0.00 mm
- net ICSPCLK_A: track 11.5 -> 0.00 mm
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Other:
- board text added: "Lidar"
- board text added: "Piolt"
- board text added: "US"
- board text removed: "Pilot"
- board text removed: "RPLIDAR"
- board text removed: "Ultrasonic"
