File: designs/RPLidar_Interface_pic/RPLidar_interface.sch (EAGLE design)
At the start: 75 parts, among them IC1 TS5205, J1 PIN-CONNECTOR74089, J2 PIN-CONNECTOR74089, J3 PIN-CONNECTOR74089, J4 22-05-7028-02, J5 PIN-CONNECTOR74089, U1 PIC24FJ32GB002-I/ML, U2 PIC24FJ32GB002-I/ML, X1 22-23-2071

Commit message: cleaning up
Parts:
- removed C1, C18, C4: .1uF, rcl:C-EUC0402
- removed J1, J2, J5: PIN-CONNECTOR74089, Mother-Board-rev5:PIN-CONNECTOR74089
- removed R12, R14, R3: 100, resistor:R-US_R0402
- removed R19, R4, R6: 10k, resistor:R-US_R0402
- added RESET: EVQQ2, adafruit:EVQQ2
- added SV11: (no value), con-lstb:MA04-2
Connections:
- removed net ICSPCLK_A: J5.P$3, J5.P$4, U$2.RB6/PGC
- removed net ICSPCLK_P: J2.P$3, J2.P$4, U2.RB1
- removed net ICSPCLK_U: J1.P$3, J1.P$4, U$1.RB6/PGC
- removed net ICSPDAT_A: J5.P$5, J5.P$6, U$2.RB7/PGD
- removed net ICSPDAT_P: J2.P$5, J2.P$6, U2.RB0
- removed net ICSPDAT_U: J1.P$5, J1.P$6, U$1.RB7/PGD
- removed net MCLR_A: C18.1, J5.P$7, J5.P$8, R14.2, R19.1
- removed net MCLR_P: C4.1, J2.P$7, J2.P$8, R12.2, R6.1
- removed net MCLR_U: C1.1, J1.P$7, J1.P$8, R3.2, R4.1
- removed net N$7: U2.RB15
- removed net N$8: U2.RB14
- new net N$11: R11.1, SV11.2, SV11.4, SV11.6, SV11.8
- new net P8.11: U$3P8.GPIO_45, U2.RB15
- new net P8.12: U$3P8.GPIO_44, U2.RB14
- new net RPLIDAR_EN: U1.RB15, X1-2.S
- net +3V3: no longer J1.P$1, J1.P$2, J2.P$1, J2.P$2, R4.2, R6.2
- net 5V: no longer J5.P$1, J5.P$2, R19.2, X1-2.S
- net GND: now also RESET.P, RESET.P1; no longer C1.2, C18.2, C4.2, J1.P$10, J1.P$9, J2.P$10, J2.P$9, J5.P$10, J5.P$9
- net ICSPCLK: now also U$1.RB6/PGC, U$2.RB6/PGC, U2.RB1
- net ICSPDAT: now also U$1.RB7/PGD, U$2.RB7/PGD, U2.RB0
- net MCLR/VPP_A: now also SV11.3; no longer R14.1
- net MCLR/VPP_P: now also SV11.1; no longer R12.1
- net MCLR/VPP_U: now also SV11.5; no longer R3.1
- net MCLR_LIDAR: now also RESET.S, RESET.S1
- net VPP/MCLR: now also SV11.7; no longer R11.1
Other:
- moved on the sheet: C14, C15, C16, C2, R5, R7
