File: designs/Pi3_Analog_hat/Pi3_Analog_hat.sch (EAGLE design)
At the start: 65 parts, among them IC1 TS5205, J3 PIN-CONNECTOR74089, J4 22-05-7028-02, U1 PIC24FJ32GB002-I/ML, U2 PIC24FJ32GB002-I/ML, X1 22-23-2071

Commit message: Add part for Pi3 hats
Parts:
- removed 3.3V, 5V, USER_LED1, USER_LED2, USER_LED5, USER_LED6: (no value), led:LEDCHIP-LED0603
- removed C10, C100, C101, C15, C3, C6: 0.1uF, rcl:C-EUC0402
- removed C11, C16: .01uF, rcl:C-EUC0402
- removed C13: 10uF, rcl:C-EUC0402
- removed C14, C5: 1uF, rcl:C-EUC0402
- removed C17, C2, C7: .1uF, rcl:C-EUC0402
- removed IC1: TS5205, v-reg:TS5205
- removed J3: PIN-CONNECTOR74089, Mother-Board-rev5:PIN-CONNECTOR74089
- removed R10: 10k, resistor:R-US_R0402
- removed R100, R101, R102, R13, R5, R7: 0, resistor:R-US_R0402
- removed R11: 100, resistor:R-US_R0402
- removed R15, R16: 1K, resistor:R-US_R0402
- removed R17, R18: 330, resistor:R-US_R0402
- removed RESET: EVQQ2, adafruit:EVQQ2
- removed SV11: (no value), con-lstb:MA04-2
- removed U$1: PIC16F73-I/ML, Microchip_By_element14_Batch_1:PIC16F73-I/ML
- removed U$3: BEAGLE_BONE_BLACK_CAPE, SparkFun-Boards:BEAGLE_BONE_BLACK_CAPE
- removed U1, U2: PIC24FJ32GB002-I/ML, Microchip-PIC24:PIC24FJ32GB002-I/ML
- R1: value 300 -> 4.7k
- R2: value 330 -> 4.7k
- X1: value 22-23-2071 -> RASPI_BOARD_B+#_HD; device con-molex:22-23-2071 -> Pi3_Power_hat_Rev1:RASPI_BOARD_B+#_HD
Connections:
- removed net !SS: U$3P9.GPIO_4, U1.RB10
- removed net MCLR/VPP_P: SV11.1, U2.MCLR*
- removed net MCLR/VPP_U: SV11.5, U$1.~MCLR/VPP
- removed net MCLR_LIDAR: C7.1, J3.P$7, J3.P$8, R10.1, R11.2, RESET.S, RESET.S1
- removed net MISO: U$3P9.GPIO_3, U1.RB13
- removed net MOSI: U$3P9.GPIO_5, U1.RB11
- removed net N$11: R11.1, SV11.2, SV11.4, SV11.6, SV11.8
- removed net N$5: R17.1, USER_LED5.A
- removed net N$6: R18.1, USER_LED6.A
- removed net P8.11: U$3P8.GPIO_45, U2.RB15
- removed net P8.12: U$3P8.GPIO_44, U2.RB14
- removed net P8.27: U$1.RB5, U$3P8.GPIO_86
- removed net P8.28: U$1.RB4, U$3P8.GPIO_88
- removed net P8.29: U$1.RB3/PGM, U$3P8.GPIO_87
- removed net P8.30: U$1.RB2, U$3P8.GPIO_89
- removed net P8.31: U$1.RB1, U$3P8.GPIO_10
- removed net P8.32: U$1.RB0/INT, U$3P8.GPIO_11
- removed net P8.33: U$1.RC7/RX/DT, U$3P8.GPIO_9
- removed net P8.34: U$1.RC6/TX/CK, U$3P8.GPIO_81
- removed net P8.35: U$1.RC5/SDO, U$3P8.GPIO_8
- removed net P8.36: U$1.RC2/CCP1, U$3P8.GPIO_80
- removed net P8.37: U$1.RC1/T1OSI/CCP2, U$3P8.GPIO_78
- removed net P8.38: U$1.RC0/T1OSO/T1CKI, U$3P8.GPIO_79
- removed net P8.39: U$1.OSC2/CLKO, U$3P8.GPIO_76
- removed net P8.40: U$1.OSC1/CLKI, U$3P8.GPIO_77
- removed net P8.41: U$1.RA5/AN4/~SS, U$3P8.GPIO_74
- removed net P8.42: U$1.RA4/T0CKI, U$3P8.GPIO_75
- removed net P8.43: U$1.RA3/AN3/VREF, U$3P8.GPIO_72
- removed net P8.44: U$1.RA2/AN2, U$3P8.GPIO_73
- removed net P8.45: U$1.RA1/AN1, U$3P8.GPIO_70
- removed net P8.46: U$1.RA0/AN0, U$3P8.GPIO_71
- removed net P9.24: U$3P9.GPIO_15
- removed net P9.25: U$3P9.GPIO_117, U2.RB4
- removed net P9.26: U$3P9.GPIO_14
- removed net P9.27: U$3P9.GPIO_125, U2.TDI
- removed net P9.28: U$3P9.GPIO_123, U2.TCK
- removed net P9.29: U$3P9.GPIO_121, U2.TDO
- removed net P9.30: U$3P9.GPIO_122, U2.RB10
- removed net P9.31: U$3P9.GPIO_120, U2.RB11
- removed net RPLIDAR_EN: U1.RB15, X1-2.S
- removed net SCLK: U$3P9.GPIO_2, U1.RB14
- removed net UART_RX: U1.RA0, X1-5.S
- removed net UART_TX: U1.RA1, X1-6.S
- removed net USER1: R1.2, U1.TCK
- removed net USER2: R2.2, U1.TDO
- removed net USER3: R18.2, U2.RA1
- removed net USER4: R17.2, U2.RA0
- removed net VBUS: R7.1, U1.VBUS
- removed net VBUS_P: R102.1, U2.VBUS
- removed net VDDCORE: C2.1, U1.VDDCORE
- removed net VDDCORE_P: C17.1, U2.VDDCORE
- removed net VPP/MCLR: SV11.7, U1.MCLR*
- removed net VUSB: R5.1, U1.VUSB
- removed net VUSB_P: R13.1, U2.VUSB
- new net SPI_CE: U$2.RA5/AN4/~SS, X1.SPI_CE0
- new net SPI_MISO: U$2.RB2, X1.SPI_MISO
- new net SPI_MOSI: U$2.RB3/PGM, X1.SPI_MOSI
- new net SPI_SCLK: U$2.RB1, X1.SPI_SCLK
- net +3V3: now also R1.2, R2.2, X1.3V3A; no longer C10.1, C100.1, C101.1, C11.1, C14.1, C15.1, C16.1, C3.1, C5.1, C6.1, IC1.VOUT, J3.P$1, J3.P$2, R10.2, R100.1, R101.1, R16.2, U$1.VDD, U1.VDD1, U1.VDD2, U2.VDD1, U2.VDD2
- net 5V: no longer C13.1, IC1.CE, IC1.VIN, R15.2, X1-1.S, X1-4.S
- net CH1: now also U$2.RC7/RX/DT; no longer U$2.RA0/AN0
- net CH10: now also U$2.RA0/AN0; no longer U$2.RC6/TX/CK
- net CH2: now also U$2.RC6/TX/CK; no longer U$2.RA1/AN1
- net CH3: now also U$2.RC5/SDO; no longer U$2.RA2/AN2
- net CH4: now also U$2.RC4/SDI/SDA; no longer U$2.RA3/AN3/VREF
- net CH5: now also U$2.RC3/SCK/SCL; no longer U$2.RA5/AN4/~SS
- net CH7: now also U$2.RA3/AN3/VREF; no longer U$2.RC3/SCK/SCL
- net CH8: now also U$2.RA2/AN2; no longer U$2.RC4/SDI/SDA
- net CH9: now also U$2.RA1/AN1; no longer U$2.RC5/SDO
- net GND: now also X1.GND_A, X1.GND_B, X1.GND_C, X1.GND_D, X1.GND_E, X1.GND_F, X1.GND_G, X1.GND_H; no longer 3.3V.C, 5V.C, C10.2, C100.2, C101.2, C11.2, C13.2, C14.2, C15.2, C16.2, C17.2, C2.2, C3.2, C5.2, C6.2, C7.2, IC1.GND, J3.P$10, J3.P$9, R102.2, R13.2, R5.2, R7.2, RESET.P, RESET.P1, U$1.EPAD, U$1.VSS, U$1.VSS_2, U$3P8.DGND@1, U$3P8.DGND@2, U$3P9.DGND@1, U$3P9.DGND@2, U1.DISVREG, U1.EP, U1.VSS1, U1.VSS2, U2.DISVREG, U2.EP, U2.VSS1, U2.VSS2, USER_LED1.C, USER_LED2.C, USER_LED5.C, USER_LED6.C, X1-3.S, X1-7.S
- net ICSPCLK: no longer J3.P$3, J3.P$4, U$1.RB6/PGC, U1.RB1, U2.RB1
- net ICSPDAT: no longer J3.P$5, J3.P$6, U$1.RB7/PGD, U1.RB0, U2.RB0
- net MCLR/VPP_A: no longer SV11.3
- net N$1: now also X1.5V0A, X1.5V0B; no longer 3.3V.A, R16.1
- net N$2: now also U$2.RA4/T0CKI; no longer R1.1, USER_LED1.A
- net N$3: now also U$2.RB4; no longer R2.1, USER_LED2.A
- net N$4: now also U$2.RB5; no longer 5V.A, R15.1
- net SCL: now also R2.1, X1.SCL; no longer R101.2, U$1.RC3/SCK/SCL, U$3P9.I2C2_SCL, U1.RB3, U2.RB3
- net SDA: now also R1.1, X1.SDA; no longer R100.2, U$1.RC4/SDI/SDA, U$3P9.I2C2_SDA, U1.RB2, U2.RB2
- net USER5: no longer U$2.RC7/RX/DT
Other:
- note removed: "BeagleBone Header"
- note removed: "ICSP"

Commit message: update
Parts:
- added +3.3V, +5V: (no value), led:LEDCHIP-LED0603
- added C1: 5uF, rcl:C-EUC0402
- added R3, R4, R5: 500, resistor:R-US_R0402
- added U$1: SN74CB3T3125PW, SN74CB3T3125PW:SN74CB3T3125PW
- renumbered USER_LED3 to USR3, USER_LED4 to USR1
Connections:
- removed net N$4: U$2.RB5
- new net CE: R4.2, U$1.3B, U$2.RA5/AN4/~SS
- new net CE_EN: U$1.3QE, X1.GPIO24
- new net MISO: U$1.2B, U$2.RB2
- new net MOSI: U$1.1B, U$2.RB3/PGM
- new net SCLK: U$1.4B, U$2.RB1
- new net SPI_EN: U$1.1QE, U$1.2QE, U$1.4QE, X1.GPIO23
- net +3V3: now also R5.2, U$1.VCC
- net 5V: now also C1.1, R3.2
- net GND: now also +3.3V.C, +5V.C, C1.2, R4.1, U$1.GND
- net N$1: now also +5V.A, R3.1; no longer X1.5V0A, X1.5V0B
- net N$3: now also +3.3V.A, R5.1; no longer U$2.RB4
- net SPI_CE: now also U$1.3A; no longer U$2.RA5/AN4/~SS
- net SPI_MISO: now also U$1.2A; no longer U$2.RB2
- net SPI_MOSI: now also U$1.1A; no longer U$2.RB3/PGM
- net SPI_SCLK: now also U$1.4A; no longer U$2.RB1
- net USER5: now also U$2.RB4
- net USER6: now also U$2.RB5; no longer U$2.RB0/INT
