File: designs/IR Interface Board/IR Interface Board.brd (EAGLE design)
At the start: 67 parts, among them IC2 PIC16F1517/19PT, IC4 REG1118

Commit message: Fix Resistor values
Parts:
- R13, R15, R16, R21, R3, R6, R7: value 10K -> 500
- R2: value 330 -> 500
Changed lines of the file:
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@@
 <?xml version="1.0" encoding="utf-8"?>
 <!DOCTYPE eagle SYSTEM "eagle.dtd">
-<eagle version="7.4.0">
+<eagle version="7.6.0">
 <drawing>
 <settings>
@@
 <element name="LED2" library="interface_board-rev13" package="SML0603" value="" x="11.43" y="-59.69"/>
 <element name="LED3" library="interface_board-rev13" package="SML0603" value="" x="17.78" y="-59.69"/>
-<element name="R6" library="rcl" package="R1206" value="10K" x="-10.16" y="-53.34"/>
-<element name="R7" library="rcl" package="R1206" value="10K" x="-5.08" y="-53.34"/>
+<element name="R6" library="rcl" package="R1206" value="500" x="-10.16" y="-53.34"/>
+<element name="R7" library="rcl" package="R1206" value="500" x="-5.08" y="-53.34"/>
 <element name="C5" library="rcl" package="C0805" value="0.1uF" x="-3.81" y="-46.99"/>
 <element name="C6" library="rcl" package="C0805" value="0.1uF" x="2.54" y="-46.99"/>
@@
 <element name="C20" library="rcl" package="C0805" value="0.1uF" x="21.59" y="-46.99"/>
 <element name="LED4" library="interface_board-rev13" package="SML0603" value="" x="24.13" y="-59.69"/>
-<element name="R21" library="rcl" package="R1206" value="10K" x="0" y="-59.69"/>
+<element name="R21" library="rcl" package="R1206" value="500" x="0" y="-59.69"/>
 <element name="JP11" library="pinhead" package="1X06/90" value="" x="-2.54" y="-38.1"/>
 <element name="R9" library="rcl" package="R1206" value="100" x="5.08" y="-53.34"/>
@@
 <element name="TOUCH_RESET" library="power_lib" package="MC32882_FINAL" value="RESET" x="11.43" y="-34.29"/>
 <element name="LED6" library="interface_board-rev13" package="SML0603" value="" x="-3.81" y="-66.04"/>
-<element name="R13" library="rcl" package="R1206" value="10K" x="15.24" y="-53.34"/>
+<element name="R13" library="rcl" package="R1206" value="500" x="15.24" y="-53.34"/>
 <element name="LED8" library="interface_board-rev13" package="SML0603" value="" x="8.89" y="-66.04"/>
-<element name="R15" library="rcl" package="R1206" value="10K" x="25.4" y="-53.34"/>
+<element name="R15" library="rcl" package="R1206" value="500" x="25.4" y="-53.34"/>
 <element name="LED9" library="interface_board-rev13" package="SML0603" value="" x="15.24" y="-66.04"/>
-<element name="R16" library="rcl" package="R1206" value="10K" x="-10.16" y="-59.69"/>
+<element name="R16" library="rcl" package="R1206" value="500" x="-10.16" y="-59.69"/>
 <element name="OUT0" library="pinhead" package="1X04" value="" x="-6.35" y="-100.33"/>
 <element name="OUT1" library="pinhead" package="1X04" value="" x="5.08" y="-100.33"/>
@@
 </element>
 <element name="R1" library="resistor" package="R0805" value="1k" x="0" y="-187.96"/>
-<element name="R2" library="resistor" package="R0805" value="330" x="-10.16" y="-187.96"/>
+<element name="R2" library="resistor" package="R0805" value="500" x="-10.16" y="-187.96"/>
 <element name="C8" library="resistor" package="C0805" value="0.1uF" x="-3.81" y="-181.61"/>
 <element name="C9" library="resistor" package="C0805" value="4.7uF" x="2.54" y="-181.61"/>
@@
 <element name="C11" library="rcl" package="C0805" value="4.7 uF" x="-10.16" y="-213.36"/>
 <element name="LED1" library="interface_board-rev13" package="SML0603" value="" x="-10.16" y="-226.06"/>
-<element name="R3" library="rcl" package="R1206" value="10K" x="-10.16" y="-219.71"/>
+<element name="R3" library="rcl" package="R1206" value="500" x="-10.16" y="-219.71"/>
 <element name="OUT20" library="pinhead" package="1X04" value="" x="-6.35" y="-231.14"/>
 <element name="OUT21" library="pinhead" package="1X04" value="" x="-6.35" y="-237.49"/>

Commit message: Fiexd +5 V
Connections:
- removed net BT_VBUS1: BT_FTDI1.8, BT_USB_MICROB1.VBUS, R2.2
- net +5V: now also BT_FTDI1.8, BT_USB_MICROB1.VBUS, R2.2
Changed lines of the file:
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@@
 <contactref element="OUT27" pad="2"/>
 <contactref element="OUT27" pad="4"/>
+<contactref element="R2" pad="2"/>
+<contactref element="BT_USB_MICROB1" pad="VBUS"/>
+<contactref element="BT_FTDI1" pad="8"/>
 <wire x1="-2.54" y1="-243.84" x2="-7.62" y2="-243.84" width="0" layer="19" extent="1-1"/>
 <wire x1="-2.54" y1="-250.19" x2="-2.54" y2="-243.84" width="0" layer="19" extent="1-1"/>
@@
 <wire x1="-11.11" y1="-213.36" x2="-8.738" y2="-219.71" width="0" layer="19" extent="1-1"/>
 <wire x1="-6.5786" y1="-206.3496" x2="-11.11" y2="-213.36" width="0" layer="19" extent="1-1"/>
-<wire x1="-7.62" y1="-157.48" x2="-6.5786" y2="-206.3496" width="0" layer="19" extent="1-1"/>
+<wire x1="-9.21" y1="-187.96" x2="-6.5786" y2="-206.3496" width="0" layer="19" extent="1-1"/>
+<wire x1="-8.92" y1="-171.34" x2="-9.21" y2="-187.96" width="0" layer="19" extent="1-1"/>
+<wire x1="-10.39" y1="-167.4" x2="-8.92" y2="-171.34" width="0" layer="19" extent="1-1"/>
+<wire x1="-7.62" y1="-157.48" x2="-10.39" y2="-167.4" width="0" layer="19" extent="1-1"/>
 <wire x1="-2.54" y1="-157.48" x2="-7.62" y2="-157.48" width="0" layer="19" extent="1-1"/>
 <wire x1="-7.62" y1="-151.13" x2="-7.62" y2="-157.48" width="0" layer="19" extent="1-1"/>
@@
 <wire x1="-11.19" y1="-165.1" x2="-7.62" y2="-171.34" width="0" layer="19" extent="1-1"/>
 </signal>
-<signal name="BT_VBUS1">
-<contactref element="R2" pad="2"/>
-<contactref element="BT_USB_MICROB1" pad="VBUS"/>
-<contactref element="BT_FTDI1" pad="8"/>
-<wire x1="-8.92" y1="-171.34" x2="-9.21" y2="-187.96" width="0" layer="19" extent="1-1"/>
-<wire x1="-10.39" y1="-167.4" x2="-8.92" y2="-171.34" width="0" layer="19" extent="1-1"/>
-</signal>
 <signal name="ADC_16">

Commit message: Finished layout. Kind of rushed. Probably needs a second set of eyes.
Parts:
- removed IC4: REG1118, burr-brown:SOT223
- added H1, H2, H3, H4: MOUNT-PAD-ROUND3.2, holes:3,2-PAD
- added IC1: REG1117, burr-brown:SOT223
- added JP1, JP2: (no value), pinhead:1X02
- C10: value 1 uF -> 10uF
- C11: value 4.7 uF -> 10uF
- moved OUT27 328.6 mm to (27.2, 51.3), turned to 180 degrees
- moved OUT26 326.8 mm to (26.9, 55.9), turned to 180 degrees
- moved OUT25 324.5 mm to (26.9, 59.9), turned to 180 degrees
- moved OUT24 322.3 mm to (26.9, 64.0), turned to 180 degrees
- moved OUT23 320.2 mm to (26.9, 68.3), turned to 180 degrees
- moved OUT22 300.3 mm to (15.7, 55.6), turned to 180 degrees
- moved OUT21 298.5 mm to (15.7, 60.2)
- moved OUT20 297.0 mm to (15.7, 65.0)
- moved LED1 237.1 mm to (7.37, 10.4)
- moved C1 237.1 mm to (12.2, 48.5), turned to 90 degrees
- moved R3 231.1 mm to (11.2, 10.4)
- moved C11 229.8 mm to (26.9, 13.5)
- moved R2 227.0 mm to (3.81, 38.6), turned to 270 degrees
- moved OUT16 226.0 mm to (23.1, 72.9)
- moved RST_JMPR1 224.8 mm to (9.14, 28.7), turned to 180 degrees
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Connections:
- new net VBUS: BT_FTDI1.8, BT_USB_MICROB1.VBUS, JP2.1, R2.2
- net +3V3: now also C11.1, IC1.2; no longer C10.1, IC4.1
- net +5V: now also C10.1, IC1.3, JP1.1; no longer BT_FTDI1.8, BT_USB_MICROB1.VBUS, C11.1, IC4.3, R2.2
- net GND: now also H1.B3,2, H2.B3,2, H3.B3,2, H4.B3,2, IC1.1, JP1.2, JP2.2; no longer IC4.2
Routing:
- net +5V: track 0.00 -> 531.5 mm, vias 0 -> 5
- net +3V3: track 0.00 -> 89.9 mm, vias 0 -> 9
- net MCLR: track 0.00 -> 60.5 mm, vias 0 -> 2
- net ADC_25: track 0.00 -> 56.8 mm, vias 0 -> 3
- net GND: track 0.00 -> 56.3 mm, vias 0 -> 26
- net ADC_12: track 0.00 -> 52.6 mm
- net ADC_11: track 0.00 -> 52.4 mm, vias 0 -> 2
- net ADC_24: track 0.00 -> 50.0 mm, vias 0 -> 4
- net ADC_9: track 0.00 -> 49.0 mm, vias 0 -> 2
- net ADC_14: track 0.00 -> 48.2 mm
- net ADC_17: track 0.00 -> 47.1 mm
- net ADC_7: track 0.00 -> 46.3 mm, vias 0 -> 2
- net ADC_13: track 0.00 -> 46.1 mm
- net ADC_8: track 0.00 -> 46.0 mm, vias 0 -> 2
- net ADC_6: track 0.00 -> 45.7 mm, vias 0 -> 2
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- added copper zone on layer 16, net GND
Other:
- board outline added: 75 x 75 mm

Commit message: Done with Unknown
Parts:
- removed FTDI1: (no value), interface_board-rev13:CHIPLED_1206
- added C12: 10uF, rcl:C0805
- added LED5: (no value), interface_board-rev13:SML0603
- C1, C2, C8, C9: device resistor:C0805 -> rcl:C0805
- C11: value 10uF -> 4.7uF
- C20, C5: value 0.1uF -> 1uF
- C3, C4, C6: value 0.1uF -> 4.7uF
- R10, R13, R15, R16, R21, R3, R6, R7, R9: device rcl:R1206 -> rcl:R0805
- R2: device resistor:R0805 -> rcl:R0805
- moved LED1 67.2 mm to (30.5, 73.5), turned to 180 degrees
- moved R3 65.0 mm to (26.8, 73.5), turned to 180 degrees
- moved JP1 58.1 mm to (21.3, 72.9)
- moved C5 57.4 mm to (15.7, 35.9), flipped to the bottom, turned to 180 degrees
- moved IC1 57.0 mm to (14.2, 66.5), turned to 0 degrees
- moved C10 54.4 mm to (16.6, 60.2), turned to 270 degrees
- moved C3 54.1 mm to (50.9, 30.5), turned to 0 degrees
- moved C6 53.5 mm to (51.2, 15.1), turned to 0 degrees
- moved R10 51.5 mm to (11.4, 2.16), turned to 180 degrees
- moved LED4 51.4 mm to (1.91, 51.9), turned to 0 degrees
- moved JP2 51.3 mm to (16.0, 72.9)
- moved OUT11 50.0 mm to (33.0, 27.9), turned to 0 degrees
- moved C11 49.5 mm to (13.1, 61.0), turned to 180 degrees
- moved R21 47.5 mm to (5.59, 51.9), turned to 0 degrees
- moved OUT13 45.2 mm to (33.0, 33.0), turned to 0 degrees
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Connections:
- removed net GND1: LED6.C
- net +3V3: now also R15.2, R16.2
- net +5V: now also C12.1, JP2.2; no longer R15.2, R16.2
- net ADC_10: now also IC2.11; no longer IC2.14
- net ADC_11: now also IC2.19; no longer IC2.15
- net ADC_12: now also IC2.15; no longer IC2.19
- net ADC_13: now also IC2.21; no longer IC2.20
- net ADC_14: now also IC2.20; no longer IC2.21
- net ADC_15: now also IC2.24; no longer IC2.22
- net ADC_16: now also IC2.22; no longer IC2.24
- net ADC_17: now also IC2.26; no longer IC2.25
- net ADC_18: now also IC2.25; no longer IC2.26
- net ADC_19: now also IC2.36; no longer IC2.27
- net ADC_20: now also IC2.27; no longer IC2.36
- net ADC_21: now also IC2.38; no longer IC2.37
- net ADC_22: now also IC2.37; no longer IC2.38
- net ADC_23: now also IC2.40; no longer IC2.39
- net ADC_24: now also IC2.39; no longer IC2.40
- net ADC_25: now also IC2.42; no longer IC2.41
- net ADC_26: now also IC2.41; no longer IC2.42
- net ADC_27: now also IC2.44; no longer IC2.43
- net ADC_28: now also IC2.43; no longer IC2.44
- net ADC_3: now also IC2.4; no longer IC2.3
- net ADC_4: now also IC2.3; no longer IC2.4
- net ADC_5: now also IC2.8; no longer IC2.5
- net ADC_6: now also IC2.5; no longer IC2.8
- net ADC_7: now also IC2.10; no longer IC2.9
- net ADC_8: now also IC2.9; no longer IC2.10
- net ADC_9: now also IC2.14; no longer IC2.11
- net GND: now also C12.2, LED5.C, LED6.C; no longer FTDI1.C, JP2.2
- net N$12: now also LED5.A; no longer FTDI1.A
Routing:
- net ADC_27: track 34.6 -> 82.3 mm, vias 2 -> 0
- net +3V3: track 89.9 -> 47.5 mm, vias 9 -> 2
- net ADC_23: track 26.2 -> 67.0 mm, vias 4 -> 0
- net ADC_28: track 27.8 -> 68.5 mm, vias 1 -> 0
- net ADC_12: track 52.6 -> 15.4 mm
- net MCLR: track 60.5 -> 24.8 mm, vias 2 -> 0
- net ADC_14: track 48.2 -> 15.6 mm
- net ADC_10: track 45.6 -> 17.6 mm, vias 2 -> 0
- net STATUS_0: track 2.82 -> 28.3 mm, vias 0 -> 2
- net ADC_21: track 33.9 -> 58.9 mm, vias 4 -> 0
- net ADC_11: track 52.4 -> 28.2 mm, vias 2 -> 0
- net ADC_8: track 46.0 -> 22.1 mm, vias 2 -> 0
- net ADC_16: track 40.4 -> 17.1 mm
- net ADC_26: track 38.7 -> 61.0 mm, vias 3 -> 0
- net ADC_2: track 25.8 -> 47.8 mm, vias 3 -> 0
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Other:
- board size 75 x 75 mm -> 58.4 x 75 mm
