File: designs/Pi3_power_hat/Pi3_Power_hat_Rev1.brd (EAGLE design)
At the start: 65.2 x 57.4 mm, 61 parts, among them J1 22-05-7028-02, J2 22-05-7028-02, J3 22-05-7028-02, J4 22-05-7028-02, J5 22-05-7028-02, J6 22-05-7028-02, J7 22-05-7028-02, J8 22-05-7028-02, J9 22-05-7028-02, X1 RASPI_BOARD_B+#_E4P

Commit message: update
Parts:
- C1, C17, C9: value (none) -> .1uF
- C10, C18, C2: value (none) -> 4.7pF
- C11, C13, C15, C19, C21, C23, C3, C5, C7: value (none) -> 1uF
- C12, C20, C4: value (none) -> 47uF
- C14, C22, C6: value (none) -> 10nF
- C16, C24, C8: value (none) -> 4.7uF
- L1: value (none) -> 4.7uH
- L2, L3: value (none) -> 1.5uH
- R1, R5, R9: value (none) -> 1M
- R10: value (none) -> 243k
- R11, R7: value (none) -> 18.2k
- R12, R4, R8: value (none) -> 10k
- R13: value 330 -> 600
- R14: value 330 -> 1.2k
- R18: value 330 -> 500\
- R2: value (none) -> 88.7k
- R3: value (none) -> 41.2K
- R6: value (none) -> 200k

Commit message: Done with Unknown
Connections:
- new net N$26: U$1.14
Changed lines of the file:
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@@
 <wire x1="5.0396" y1="29.8704" x2="5.0396" y2="29.8958" width="0.254" layer="1"/>
+</signal>
+<signal name="N$26">
+<contactref element="U$1" pad="14"/>
 </signal>
 </signals>
