File: designs/UI-interface/UI-interface.brd (EAGLE design)
At the start: 26.8 x 24 mm, 2 parts

Commit message: done with first version of the boards
Parts:
- added D1: 1N4148, adafruit:SOD-323F
- added JP1: (no value), microbuilder:1X06_ROUND_70
- added R5: 10K, microbuilder:0805
- moved H1 10.0 mm to (20.0, 5.00)
- moved H2 10.0 mm to (20.0, 19.0)
Connections:
- new net 3.3V: JP1.2, R5.2
- new net GND: JP1.3
- new net RES_3.3V: D1.A, R5.1
- new net RES_5.0V: D1.C, JP1.4
- new net SCL_5.0V: JP1.5
- new net SDA_5.0V: JP1.6
- new net VIN: JP1.1
Other:
- board size 26.8 x 24 mm -> 33.4 x 26 mm
