File: designs/Unkown Circuit/UnknownSchematic.brd (EAGLE design)
At the start: 160 x 100 mm, 47 parts, among them IC1 REG1118, IC2 PIC16F1517/19PT, U1 0914-0-15-20-77-14-11-0

Commit message: Updated Unknown Circuit Schematic
Parts:
- added C10: 1 uF, rcl:C0805
- added C11: 4.7 uF, rcl:C0805
- added C8, C9: 0.01 uF, rcl:C0805
- added IC3: LF442D, linear:SO08
- added IC4: REG1118, burr-brown:SOT223
- added JP2, JP3, JP4: (no value), pinhead:1X11
- added JP5: (no value), pinhead:1X02
- added LED6, LED7, LED8, LED9: (no value), interface_board-rev13:SML0603
- added R11, R12: 4.7k, rcl:R0805
- added R13, R14, R15, R16: 10K, rcl:R1206
- JP1: device pinhead:1X08 -> pinhead:1X11
- moved JP1 245.2 mm to (-175.3, -261.6)
Connections:
- net AEN_1 renamed NC_6_PIC
- net AEN_2 renamed NC_8_PIC
- net APH_1 renamed NC_2_PIC
- net APH_2 renamed NC_4_PIC
- net BEN_1 renamed NC_7_PIC
- net BEN_2 renamed NC_9_PIC
- net BPH_1 renamed NC_3_PIC
- net BPH_2 renamed NC_5_PIC
- net OUT0 renamed NC_20_PIC
- net SCL renamed NC_19_PIC
- removed net +3V3_KB: BT_FTDI.6, BT_FTDI.7, C37.2, C38.2, C39.2, C40.2, R46.2
- removed net NFAULT_1: IC2.14
- removed net NFAULT_2: IC2.15
- removed net NSLEEP_1: IC2.27, R8.2
- removed net NSLEEP_2: IC2.26, R7.2
- removed net OUT8: IC2.44
- removed net OUT9: IC2.1
- removed net QEIA1_1: IC2.20
- removed net QEIA1_2: IC2.19
- removed net QEIA2_1: IC2.24
- removed net QEIA2_2: IC2.23
- removed net QEIB1_1: IC2.22
- removed net QEIB1_2: IC2.21
- removed net QEIB2_1: IC2.31
- removed net QEIB2_2: IC2.30
- removed net SDA: IC2.32
- removed net STATUS1: IC2.25, R6.2
- new net GND1: LED6.C
- new net N$10: LED8.A, R15.1
- new net N$11: LED9.A, R16.1
- new net N$2: IC3.6, R11.2, R12.1
- new net N$3: LED6.A, R13.1
- new net N$4: LED7.A, R14.1
- new net NC_10_PIC: IC2.14, JP2.3
- new net NC_11_PIC: IC2.15, JP2.4
- new net NC_12_PIC: IC2.19, JP2.8
- new net NC_13_PIC: IC2.20, JP2.9
- new net NC_14_PIC: IC2.22, JP2.11
- new net NC_15_PIC: IC2.23, JP3.1
- new net NC_16_PIC: IC2.30, JP3.8
- new net NC_17_PIC: IC2.31, JP3.9
- new net NC_18_PIC: IC2.32, JP3.10
- new net NC_1_PIC: IC2.1, JP1.1
- new net NC_21_PIC: IC2.44, JP4.11
- new net NC_PIC_19: JP4.2
- new net NC_PIC_20: JP4.3
- new net NC_PIN12: JP2.1
- new net NC_PIN13: JP2.2
- new net NC_PIN33: JP3.11
- new net NC_PIN34: JP4.1
- new net NIC_2_PIC: JP1.2
- new net NIC_3_PIC: JP1.3
- new net NIC_4_PIC: JP1.4
- new net NIC_5_PIC: JP1.5
- new net NIC_6_PIC: JP1.8
- new net NIC_7_PIC: JP1.9
- new net NIC_8_PIC: JP1.10
- new net NIC_9_PIC: JP1.11
- new net STATUS_0: IC2.24, JP3.2, R13.2
- new net STATUS_1: IC2.25, JP3.3, R6.2
- new net STATUS_2: IC2.26, JP3.4, R7.2
- new net STATUS_3: IC2.27, JP3.5, R8.2
- net +3V3: now also BT_FTDI.6, BT_FTDI.7, C10.1, C37.2, C38.2, C39.2, C40.2, IC4.1, R15.2, R16.2, R46.2
- net +5V: now also C11.1, IC3.8, IC4.3, JP1.7, JP3.6; no longer JP1.1
- net ADCP1: now also JP4.5; no longer JP1.3
- net ADCP2: now also JP4.6; no longer JP1.4
- net ADCP3: now also JP4.7; no longer JP1.5
- net ADCP4: now also JP4.8; no longer JP1.6
- net ADCP5: now also JP4.9; no longer JP1.7
- net BUFFEROUTPUT: now also C9.1, IC3.7, JP5.2, R11.1
- net DAC: now also C8.2, IC2.21, IC3.5, JP2.10, JP5.1; no longer JP1.2
- net GND: now also C10.2, C11.2, C8.1, C9.2, IC3.4, IC4.2, JP1.6, JP3.7, LED7.C, R12.2; no longer JP1.8
- net ICDCLK: now also JP2.5
- net ICDDAT: now also JP2.6
- net MCLR: now also JP2.7
- net PROBE0: now also R14.2
- net UART_RX: now also JP4.10, LED9.C
- net UART_TX: now also JP4.4, LED8.C

Commit message: Fiexd +5 V
Parts:
- removed BT_USB_MICROB: USB-MICROB, Mother-Board-rev5:USB-MICROB
- removed C3, C4, C5: 0.1uF, rcl:C0805
- removed FTDI: (no value), interface_board-rev13:CHIPLED_1206
- removed IC3: LF442D, linear:SO08
- removed JP3, JP4: (no value), pinhead:1X11
- added H1, H10, H2, H3, H4, H5, H6, H7, H8, H9: MOUNT-PAD-ROUND3.2, holes:3,2-PAD
- added IC5: UA741D, linear:SO08
- added LED10: (no value), interface_board-rev13:SML0603
- JP2: device pinhead:1X11 -> pinhead:1X04
- R47: value 330 -> 500
- moved JP5 380.3 mm to (152.7, -115.3), turned to 90 degrees
- moved JP2 355.2 mm to (126.2, -80.3), turned to 270 degrees
- moved R12 343.8 mm to (148.8, -115.1), turned to 90 degrees
- moved R2 343.6 mm to (156.7, -100.8), turned to 90 degrees
- moved C9 340.1 mm to (141.0, -110.2), turned to 180 degrees
- moved R11 339.8 mm to (145.0, -110.2)
- moved C8 339.6 mm to (144.8, -122.7), turned to 180 degrees
- moved R3 337.3 mm to (142.5, -136.1), turned to 90 degrees
- moved D2 334.2 mm to (153.2, -97.8), turned to 90 degrees
- moved IC1 334.1 mm to (142.7, -87.9), turned to 270 degrees
- moved C11 331.2 mm to (113.5, -80.0), turned to 270 degrees
- moved LED9 328.3 mm to (104.1, -109.2)
- moved R15 325.9 mm to (109.2, -112.5)
- moved LED8 325.2 mm to (104.1, -112.5)
- moved C1 325.1 mm to (135.4, -86.4), turned to 270 degrees
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Connections:
- removed net BT_VBUS: BT_FTDI.8, BT_USB_MICROB.VBUS, R47.2
- removed net NC_PIC_19: JP4.2
- removed net NC_PIC_20: JP4.3
- removed net NC_PIN12: JP2.1
- removed net NC_PIN13: JP2.2
- removed net NC_PIN33: JP3.11
- removed net NC_PIN34: JP4.1
- removed net NIC_2_PIC: JP1.2
- removed net NIC_3_PIC: JP1.3
- removed net NIC_4_PIC: JP1.4
- removed net NIC_5_PIC: JP1.5
- removed net NIC_6_PIC: JP1.8
- removed net NIC_7_PIC: JP1.9
- removed net NIC_8_PIC: JP1.10
- removed net NIC_9_PIC: JP1.11
- net +5V: now also BT_FTDI.8, IC5.7, JP2.2, R47.2; no longer C3.1, C4.1, C5.1, IC3.8, JP1.7, JP3.6
- net ADCP1: no longer JP4.5
- net ADCP2: no longer JP4.6
- net ADCP3: no longer JP4.7
- net ADCP4: no longer JP4.8
- net ADCP5: no longer JP4.9
- net BT_D+: now also JP2.4; no longer BT_USB_MICROB.D+
- net BT_D-: now also JP2.3; no longer BT_USB_MICROB.D-
- net BUFFEROUTPUT: now also IC5.6; no longer IC3.7
- net DAC: now also IC5.3; no longer IC3.5, JP2.10
- net GND: now also IC5.4, JP2.1, LED10.C; no longer BT_USB_MICROB.GND, BT_USB_MICROB.MT1, BT_USB_MICROB.MT2, C3.2, C4.2, C5.2, FTDI.C, IC3.4, JP1.6, JP3.7
- net ICDCLK: no longer JP2.5
- net ICDDAT: no longer JP2.6
- net MCLR: no longer JP2.7
- net N$2: now also IC5.2; no longer IC3.6
- net N$9: now also LED10.A; no longer FTDI.A
- net NC_10_PIC: no longer JP2.3
- net NC_11_PIC: no longer JP2.4
- net NC_12_PIC: no longer JP2.8
- net NC_13_PIC: no longer JP2.9
- net NC_14_PIC: no longer JP2.11
- net NC_15_PIC: no longer JP3.1
- net NC_16_PIC: no longer JP3.8
- net NC_17_PIC: no longer JP3.9
- net NC_18_PIC: no longer JP3.10
- net NC_1_PIC: no longer JP1.1
- net NC_21_PIC: no longer JP4.11
- net STATUS_0: no longer JP3.2
- net STATUS_1: no longer JP3.3
- net STATUS_2: no longer JP3.4
- net STATUS_3: no longer JP3.5
- net UART_RX: no longer JP4.10
- net UART_TX: no longer JP4.4
Routing:
- added copper zone on layer 16, net GND
Other:
- board size 160 x 100 mm -> 90 x 90 mm

Commit message: Done with Unknow circuit
Parts:
- removed JP1: (no value), pinhead:1X11
- IC1: value REG1118 -> +2.5v
- IC4: value REG1118 -> +3.3v
- moved LED8 9.15 mm to (113.3, -112.3), turned to 180 degrees
- moved LED9 8.92 mm to (113.0, -108.5), turned to 180 degrees
- moved R5 7.96 mm to (88.4, -103.9), turned to 0 degrees
- moved D5 7.41 mm to (87.4, -98.6)
- moved C7 5.34 mm to (86.9, -115.6), turned to 90 degrees
- moved R47 4.75 mm to (132.3, -77.7)
- moved D2 4.57 mm to (148.6, -97.8)
- moved LED10 4.26 mm to (132.3, -73.7)
- moved R2 4.10 mm to (152.7, -101.3)
- moved C20 3.64 mm to (124.7, -142.0), turned to 270 degrees
- moved R13 3.06 mm to (103.9, -143.8)
- moved R6 3.06 mm to (106.9, -143.8)
- moved LED6 3.06 mm to (103.9, -147.8)
- moved LED3 3.05 mm to (106.9, -148.1)
- moved LED4 2.90 mm to (83.6, -89.7)
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Connections:
- removed net GND1: LED6.C
- net ADCP1: now also IC2.42; no longer IC2.38
- net ADCP2: now also IC2.41; no longer IC2.39
- net ADCP4: now also IC2.38; no longer IC2.41
- net ADCP5: now also IC2.39; no longer IC2.42
- net GND: now also H1.B3,2, H10.B3,2, H2.B3,2, H3.B3,2, H4.B3,2, H5.B3,2, H6.B3,2, H7.B3,2, H8.B3,2, H9.B3,2, LED6.C
Routing:
- net PROBE0: track 0.00 -> 252.6 mm, vias 0 -> 4
- net +5V: track 0.00 -> 244.2 mm, vias 0 -> 9
- net BUFFEROUTPUT: track 0.00 -> 216.4 mm, vias 0 -> 7
- net GND: track 0.00 -> 95.1 mm, vias 0 -> 18
- net ADCP1: track 0.00 -> 75.9 mm, vias 0 -> 4
- net ADCP5: track 0.00 -> 68.4 mm, vias 0 -> 2
- net +3V3: track 0.00 -> 60.8 mm, vias 0 -> 2
- net DAC: track 0.00 -> 60.0 mm, vias 0 -> 2
- net ADCP2: track 0.00 -> 55.6 mm, vias 0 -> 2
- net ICDCLK: track 0.00 -> 52.9 mm
- net ICDDAT: track 0.00 -> 52.3 mm
- net UART_RX: track 0.00 -> 41.1 mm, vias 0 -> 2
- net UART_TX: track 0.00 -> 40.6 mm, vias 0 -> 2
- net ADCP4: track 0.00 -> 36.8 mm, vias 0 -> 2
- net MCLR`: track 0.00 -> 31.4 mm
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
Commit message: done with first version of the boards
Parts:
- added R17: 100, rcl:R0805
- added R18: 10K, rcl:R0805
- added U$1: LOGO, IEEE-logo:IEEE-LOGO
- added U2: QRE11131:1, Testing:QRE1113-1:1
- R13, R14, R15, R16, R20, R21, R6, R7, R8: device rcl:R1206 -> rcl:R0805
Connections:
- removed net NC_20_PIC: IC2.36
- new net IR_RANGE: IC2.36, R18.2, U2.3
- new net N$12: R17.1, U2.1
- net +3V3: now also IC4.2; no longer IC4.1
- net +5V: now also R17.2, R18.1
- net GND: now also IC1.1, IC4.1, U2.2, U2.4; no longer IC1.2, IC4.2
- net PROBE0: now also IC1.2; no longer IC1.1
Routing:
- net IR_RANGE: track 0.00 -> 33.2 mm, vias 0 -> 5
- net GND: track 95.1 -> 87.3 mm, vias 18 -> 19
- net +5V: track 244.2 -> 250.1 mm, vias 9 -> 10
- net +3V3: track 60.8 -> 63.9 mm
- net N$12: track 0.00 -> 2.46 mm
- net PROBE0: track 252.6 -> 251.6 mm
Other:
- board text added: "NCSU Robotics Club"
